File: USB_Amp.brd (EAGLE design)
At the start: 5.1 x 8.6 mm, 149 parts, among them CON1 USB-C, CON2 PIC32_CON, CON4 VOLUEME, CON5 SWD, IC1 3.3V, IC10 +12V, IC16 STM32G031F, IC2 PIC32MZEF, IC3 TAS2780, IC4 TAS2780, IC5 1.8V, IC6 1.8V, IC7 +5V, IC8 +5V, IC9 +12V, X1 24.576MHz, X2 22.5792MHz, X3 12MHz

Commit message: 発注
Parts:
- removed CON5: SWD, my_connector:SWD_CON
- removed FB6: FB2012-FB, my_rcl:2012-FB
- removed IC16: STM32G031F, my_ic:TSSOP20
- removed R14, R29: 1k, my_rcl:1608
- removed TP12: IO13, my_connector:TESTPIN
- removed TP13, TP14: GND, my_connector:TESTPIN
- removed TP17: +3V3, my_connector:TESTPIN
- added C69: 10p, my_rcl:1608C
- added C70: 10u, my_rcl:3216
- added C71: 10u, my_rcl:2012
- added C72, C73, C78: 0.1u, my_rcl:1608C
- added C74: DNP, my_rcl:1608C
- added C75, C76: 1000u, my_rcl:E5-10
- added C77: 470u, my_rcl:E5-10
- added C79: 22u, my_rcl:2012
- added C80, C84: 0.47uF, my_rcl:C050
- added C81, C85: 0.47uF, my_rcl:3225-3
- added C82, C83, C86, C87: 1n, my_rcl:1608-2
- added C88: 22u, my_rcl:3225
- added CON3: VOLUEME, my_connector:VOL_CON
- added D3: LED1, my_rcl:D1608
- added DR1, DR2, DR3, DR4: HOLE-3.2, my_connector:HOLE_3.2
- added IC11: STM32G031F, my_ic:TSSOP20
- added IC12: +5V, my_ic:TO220-SOP-DUAL
- added IC13: 3.3V, my_ic:SOT23-5
- added JP1: IO, my_connector:1X05
- added R39: SCK, my_rcl:1608-J
- added R40, R41, R42, R49: 1k, my_rcl:1608
- added R43: DNP, my_rcl:1608
- added R44: 100k, my_rcl:1608
- added R45, R46, R47, R48: 10k, my_rcl:1608
- added TP7, TP8: G, my_connector:TESTPIN
- C1, C42: value 0.1u -> 10u; device my_rcl:1608C -> my_rcl:2012
- C12: value 0.1u -> 22p
- C14: value 22p -> 0.47uF; device my_rcl:1608C -> my_rcl:3225-3
- C15, C17: value 0.1u -> 10n; device my_rcl:1608C -> my_rcl:3216-3
- C16, C43: value 0.1u -> 0.47uF; device my_rcl:1608C -> my_rcl:C050
- C18: value 1u -> 470p
- C19, C39: value (none) -> 10u; device my_rcl:C050 -> my_rcl:3216
- C2, C36: value 0.1u -> 1u
- C20: value 10n -> 10u; device my_rcl:2012 -> my_rcl:3216
- C21: value 10n -> 3.3n; device my_rcl:2012 -> my_rcl:1608C
- C22, C23: value 0.1u -> 470u; device my_rcl:1608C -> my_rcl:E5-10
- C24: value 3.3n -> 10p
- C25: value 470p -> 0.1u
- C26, C29: value 10p -> 0.1u
- C27: value 3.3n -> 1u
- C28: value 470p -> 1u
- C3, C38: value 1u -> 10u; device my_rcl:1608C -> my_rcl:2012
- C30: value 10u -> 0.1u; device my_rcl:2012 -> my_rcl:1608C
- C33: value 0.1u -> 470p
- C34: value 0.1u -> 10n
- C37: value 0.1u -> 3.3n
- C40: value 10n -> 0.1u; device my_rcl:2012 -> my_rcl:1608C
- C41: value 10n -> 10p; device my_rcl:2012 -> my_rcl:1608C
- C44: value 3.3n -> 10n; device my_rcl:1608C -> my_rcl:3216-3
- C45: value 470p -> 0.47uF; device my_rcl:1608C -> my_rcl:3225-3
- C46: value 10p -> 10n; device my_rcl:1608C -> my_rcl:3216-3
- C47: value 3.3n -> 470p
- C48: value 470p -> 10u; device my_rcl:1608C -> my_rcl:3216
- C49: value 10p -> 10u; device my_rcl:1608C -> my_rcl:3216
- C5: value 22u -> 0.1u; device my_rcl:2012 -> my_rcl:1608C
- C50: value 10u -> 3.3n; device my_rcl:2012 -> my_rcl:1608C
- C51, C52: value 10u -> 470u; device my_rcl:2012 -> my_rcl:E5-10
- C53: value DNP -> 10p
- C54: value 1u -> 0.1u
- C55, C58, C59: value 10u -> 0.1u; device my_rcl:3216 -> my_rcl:1608C
- C57: value 10u -> 1u; device my_rcl:3216 -> my_rcl:1608C
- C60, C61: device my_rcl:3216 -> my_rcl:2012
- C62: value 470u -> 470p; device my_rcl:E5-10 -> my_rcl:1608C
- C63: value 470u -> 10n; device my_rcl:E5-10 -> my_rcl:1608C
- C64, C68: value 100u -> 0.1u; device my_rcl:E5-10 -> my_rcl:1608C
- C65: value 100u -> 3.3n; device my_rcl:E5-10 -> my_rcl:1608C
- C66: value 10u -> 1u; device my_rcl:2012 -> my_rcl:1608C
- CON4: value VOLUEME -> SWD; device my_connector:VOL_CON -> my_connector:SWD_CON
- D1: value LED0 -> SBD-E; device my_rcl:D1608 -> my_rcl:SOD523
- D2: value LED1 -> LED0
- D4: value SBD-E -> PWR; device my_rcl:SOD523 -> my_rcl:D1608
- FB5: device my_rcl:1608-J -> my_rcl:2012-FB
- IC10: value +12V -> 1.8V; device my_ic:TO220-SOP-DUAL -> my_ic:SOT23-5
- IC3: value TAS2780 -> +12V; device my_ic:VQFN30 -> my_ic:TO220-SOP-DUAL
- IC4: value TAS2780 -> +5V; device my_ic:VQFN30 -> my_ic:TO220-SOP-DUAL
- IC5: value 1.8V -> TAS2780; device my_ic:SOT23-5 -> my_ic:VQFN30
- IC7: value +5V -> +12V
- IC9: value +12V -> TAS2780; device my_ic:TO220-SOP-DUAL -> my_ic:VQFN30
- L1, L2, L3, L4: value (none) -> 15uH
- R1: value 1k -> 10k
- R10, R22, R37: value 39 -> LRCLK
- R11: value 10 -> DATA; device my_rcl:2012 -> my_rcl:1608-J
- R12, R24: value 10 -> SCK; device my_rcl:2012 -> my_rcl:1608-J
- R13, R26: value DNP -> 1k
- R16, R31: value 1k -> 10; device my_rcl:1608 -> my_rcl:2012
- R17: value DNP -> 10; device my_rcl:1608 -> my_rcl:2012
- R19: value 330 -> 1k
- R2, R4: value 1k -> 5.1k
- R20: value 1k -> DNP
- R21, R36: value 39 -> DATA
- R23, R38: value 39 -> 330; device my_rcl:1608-J -> my_rcl:1608
- R25: value 10 -> 1k; device my_rcl:2012 -> my_rcl:1608
- R28: value 330 -> DNP
- R3, R9: value 39 -> 10k; device my_rcl:1608-J -> my_rcl:1608
- R30: value DNP -> 330
- R32: value 330 -> 10; device my_rcl:1608 -> my_rcl:2012
- R34, R7: value 10k -> 1k
- R35: value 10k -> DNP
- R5: value 5.1k -> 10k
- R6: value 5.1k -> 1k
- TP1: value (none) -> L_P
- TP10: value IO14 -> G
- TP2: value (none) -> L_N
- TP3: value (none) -> R_P
- TP4: value (none) -> R_N
- TP5: value (none) -> VIN+
- TP6: value (none) -> VIN-
- TP9: value IO15 -> G
- X3: device my_rcl:KC3225 -> my_rcl:KC3225-2
- moved FB5 123.7 mm to (47.0, 65.0), turned to 270 degrees
- moved C39 122.4 mm to (35.0, 53.5), turned to 0 degrees
- moved R11 119.5 mm to (63.9, 31.1), turned to 180 degrees
- moved R27 119.3 mm to (30.5, 53.0), flipped to the top, turned to 90 degrees
- moved R12 118.7 mm to (66.8, 30.0)
- moved C41 118.0 mm to (23.0, 50.0), flipped to the bottom, turned to 180 degrees
- moved R28 117.5 mm to (18.7, 56.5), turned to 90 degrees
- moved IC4 116.0 mm to (30.5, 61.0)
- moved C38 114.5 mm to (34.0, 50.0)
- moved R24 114.0 mm to (29.1, 41.5)
- moved R26 112.9 mm to (16.0, 55.5), turned to 180 degrees
- moved C40 112.5 mm to (31.0, 47.0), turned to 0 degrees
- moved C34 111.5 mm to (28.6, 53.0), turned to 90 degrees
- moved R13 109.8 mm to (69.0, 13.5), flipped to the top, turned to 90 degrees
- moved C7 109.2 mm to (69.5, 20.4), turned to 90 degrees
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Connections:
- removed net N$38: IC16.14, TP10.1
- removed net N$39: IC16.16
- removed net N$52: IC16.15, TP9.1
- new net PIC_COM1: IC11.12, IC2.62
- new net PIC_COM2: IC11.13, IC2.64
- new net PIC_COM3: IC11.14, IC2.63
- new net STM_IO16: IC11.16, JP1.2
- new net STM_IO17: IC11.17, JP1.3
- new net STM_IO20: IC11.20, JP1.4
- net +3V3: now also C72.1, C79.1, CON3.1, D4.A, IC11.4, IC13.5, JP1.1, R46.2, R47.2; no longer CON4.1, IC16.4, R34.2, R35.2, TP17.1
- net +3V3D: now also C4.1, C7.1, C88.1, FB2.1, FB3.2, R5.2; no longer C12.1, C5.1, FB5.2, R8.2
- net +5V: now also C28.1, C57.1, C77.+, C78.1, IC10.1, IC10.3, IC12.3, IC12.6, IC13.1, IC13.3; no longer IC5.1, IC5.3
- net AMP_AVDD_L: now also C35.1, C38.1, C39.1, IC5.24-1, IC5.24-2, IC6.5; no longer C22.1, C32.1, C55.1, IC3.24-1, IC3.24-2, IC5.5
- net AMP_AVDD_R: now also C64.1, C67.1, C70.1, IC10.5, IC9.23, IC9.24-1, IC9.24-2; no longer C42.1, C52.1, C57.1, IC4.23, IC4.24-1, IC4.24-2, IC6.5
- net AMP_IOVDD_L: now also C40.1, C42.1, FB3.1, IC5.20; no longer C23.1, C66.1, FB4.1, IC3.20
- net AMP_IOVDD_R: now also C68.1, C71.1, FB4.1, IC9.20; no longer C43.1, C67.1, FB5.1, IC4.20
- net AMP_OUTN_L: now also C26.1, IC5.29, R26.2, R28.1; no longer C6.1, IC3.29, R17.1, R18.2
- net AMP_OUTN_R: now also C55.1, IC9.29, R41.2, R43.1; no longer C33.1, IC4.29, R30.1, R31.2
- net AMP_OUTP_L: now also C25.2, IC5.3, R19.2, R20.1; no longer C7.2, IC3.3, R13.1, R14.2
- net AMP_OUTP_R: now also C54.2, IC9.3, R34.2, R35.1; no longer C34.2, IC4.3, R26.1, R27.2
- net AMP_SDZ: now also IC5.22, IC9.22, R49.1; no longer IC16.3, IC3.22, IC4.22
- net AMP_SNS_N_L: now also C37.2, C41.1, IC5.1-1, IC5.1-2, R25.2, R28.2; no longer C27.2, C29.1, IC3.1-1, IC3.1-2, R17.2, R20.2
- net AMP_SNS_N_R: now also C65.2, C69.1, IC9.1-1, IC9.1-2, R40.2, R43.2; no longer C47.2, C49.1, IC4.1-1, IC4.1-2, R30.2, R33.2
- net AMP_SNS_P_L: now also C21.2, C24.1, IC5.5, R18.2, R20.2; no longer C24.2, C26.1, IC3.5, R13.2, R16.2
- net AMP_SNS_P_R: now also C50.2, C53.1, IC9.5, R33.2, R35.2; no longer C44.2, C46.1, IC4.5, R26.2, R29.2
- net AMP_VDD_1S_L: now also C20.1, C23.+, C30.1, C32.1, IC4.3, IC4.6, IC5.27; no longer C16.1, C31.1, C58.1, C65.+, IC3.27, IC7.3, IC7.6
- net AMP_VDD_1S_R: now also C49.1, C52.+, C61.1, IC9.27; no longer C36.1, C51.1, C63.+, IC4.27
- net AMP_VDD_L: now also C19.1, C22.+, C29.1, C31.1, IC3.3, IC3.6, IC5.28, R27.2; no longer C17.1, C30.1, C60.1, C64.+, FB2.2, IC3.28, IC9.3, IC9.6
- net AMP_VDD_R: now also C48.1, C51.+, C58.1, C60.1, IC7.3, IC7.6, IC9.28, R42.2; no longer C37.1, C50.1, C61.1, C62.+, FB3.2, IC10.3, IC10.6, IC4.28
- net EN_44.1K: now also R9.2
- net EN_48K: now also R8.2
- net EN_DDC: now also IC11.8, R1.1, R3.2; no longer IC16.20, R7.1
- net GND: now also C15.1, C16.1, C19.2, C20.2, C22.-, C23.-, C24.2, C27.2, C28.2, C34.2, C39.2, C40.2, C43.1, C44.1, C45.2, C48.2, C51.-, C52.-, C6.2, C63.2, C64.2, C68.2, C69.2, C7.2, C70.2, C71.2, C72.2, C73.2, C74.2, C75.-, C76.-, C77.-, C78.2, C79.2, C80.1, C81.2, C82.2, C83.1, C84.1, C85.2, C86.2, C87.1, C88.2, CON3.3, D3.K, IC11.5, IC12.2, IC12.5, IC13.2, IC3.5, IC4.5, IC5.23, IC5.25, IC5.7, IC9.25, IC9.7, JP1.5, R2.1, R3.1, R4.1, R44.1, R45.1, R48.1, R8.1, R9.1, TP10.1, TP7.1, TP8.1, TP9.1; no longer C15.2, C16.2, C18.2, C20.1, C21.2, C22.2, C23.2, C26.2, C37.2, C40.1, C43.2, C50.2, C51.2, C52.2, C54.2, C55.2, C62.-, C63.-, C64.-, C65.-, C68.-, CON5.3, D1.K, IC10.5, IC16.5, IC3.23, IC3.25, IC3.7, IC4.25, IC4.7, IC9.5, R5.1, R6.1, TP13.1, TP14.1
- net I2C_SCL: now also IC11.1, IC5.18, IC9.18, R46.1; no longer IC16.1, IC3.18, IC4.18, R34.1
- net I2C_SDA: now also IC11.2, IC5.19, IC9.19, R47.1; no longer IC16.2, IC3.19, IC4.19, R35.1
- net I2S_DATA: now also R11.2, R36.1; no longer R3.1, R37.2
- net I2S_LRCLK: now also R10.2, R37.1; no longer R36.2, R9.1
- net I2S_SCK: now also R12.2, R24.1, R39.1; no longer R10.1, R23.1, R38.2
- net LED0: now also IC2.2, R6.2; no longer IC2.3, R1.2
- net LED1: now also IC2.3, R7.2; no longer IC2.4, R2.2
- net MCLR: now also R5.1; no longer R8.1
- net N$1: now also R2.2; no longer R5.2
- net N$10: now also C33.2, C37.1, R26.1; no longer C27.1, C28.2, R18.1
- net N$11: now also C26.2, IC5.30; no longer C6.2, IC3.30
- net N$12: now also C25.1, IC5.4; no longer C7.1, IC3.4
- net N$13: now also C18.2, C21.1, R19.1; no longer C24.1, C25.2, R14.1
- net N$14: now also C34.1, IC5.26, R27.1; no longer C15.1, FB2.1, IC3.26
- net N$15: now also C27.1, IC5.10; no longer C18.1, IC3.10
- net N$16: now also IC5.13, R21.2; no longer IC3.13, R3.2
- net N$17: now also IC5.14, R22.2; no longer IC3.14, R9.2
- net N$18: now also IC5.15, R24.2; no longer IC3.15, R10.2
- net N$19: now also C33.1, R23.2; no longer C28.1, R19.2
- net N$2: now also R4.2; no longer R6.2
- net N$20: now also C18.1; no longer C25.1
- net N$21: now also C15.2, R16.2; no longer C20.2, R12.2
- net N$22: now also C17.1, R17.1; no longer C21.1, R11.1
- net N$23: now also C55.2, IC9.30; no longer C33.2, IC4.30
- net N$24: now also C54.1, IC9.4; no longer C34.1, IC4.4
- net N$25: now also C63.1, IC9.26, R42.1; no longer C35.1, FB3.1, IC4.26
- net N$26: now also C56.1, IC9.10; no longer C38.1, IC4.10
- net N$27: now also IC9.13, R36.2; no longer IC4.13, R21.2
- net N$28: now also IC9.14, R37.2; no longer IC4.14, R22.2
- net N$29: now also IC9.15, R39.2; no longer IC4.15, R23.2
- net N$30: now also C44.2, R31.2; no longer C40.2, R25.2
- net N$31: now also C46.1, R32.1; no longer C41.1, R24.1
- net N$32: now also C47.2, C50.1, R34.1; no longer C44.1, C45.2, R27.1
- net N$33: now also C47.1, R30.2; no longer C45.1, R28.2
- net N$34: now also C62.2, C65.1, R41.1; no longer C47.1, C48.2, R31.1
- net N$35: now also C62.1, R38.2; no longer C48.1, R32.2
- net N$36: now also D4.K, R48.2; no longer IC16.13, TP12.1
- net N$37: now also IC11.3, R45.2, R49.2; no longer IC16.17
- net N$4: now also D1.A, R1.2; no longer D4.A, R7.2
- net N$40: now also R12.1; no longer R38.1
- net N$41: now also R11.1; no longer R37.1
- net N$42: now also C36.1, IC6.4; no longer C54.1, IC5.4
- net N$43: now also R10.1; no longer R36.1
- net N$44: now also C66.1, IC10.4; no longer C56.1, IC6.4
- net N$5: now also C12.1; no longer C13.1
- net N$6: now also R13.2; no longer R4.2
- net N$7: now also C13.1, R13.1; no longer C14.1, R4.1
- net N$72: now also C74.1, CON3.2, IC11.11, R44.2; no longer C53.1, CON4.2, IC16.7
- net N$8: now also D2.A, R6.1; no longer D1.A, R1.1
- net N$9: now also D3.A, R7.1; no longer D2.A, R2.1
- net NC1: now also IC5.9-1, IC5.9-2; no longer IC3.9-1, IC3.9-2
- net NC2: now also IC5.16-1, IC5.16-2; no longer IC3.16-1, IC3.16-2
- net NC3: now also IC9.9-1, IC9.9-2; no longer IC4.9-1, IC4.9-2
- net NC4: now also IC9.16-1, IC9.16-2; no longer IC4.16-1, IC4.16-2
- net SP_OUTN_L: now also C80.2, C81.1, C83.2, R16.1, R23.1, R25.1; no longer C19.2, R12.1, R19.1, R20.1
- net SP_OUTN_R: now also C43.2, C45.1, C87.2, R31.1, R38.1, R40.1; no longer C39.2, R25.1, R32.1, R33.1
- net SP_OUTP_L: now also C14.1, C16.2, C82.1, R17.2, R18.1; no longer C19.1, R11.2, R16.1
- net SP_OUTP_R: now also C84.2, C85.1, C86.1, R30.1, R32.2, R33.1; no longer C39.1, R24.2, R28.1, R29.1
- net STM_TX: now also CON4.5, IC11.9; no longer CON5.5, IC16.9
- net SWCLK: now also CON4.1, IC11.19; no longer CON5.1, IC16.19
- net SWDIO: now also CON4.4, IC11.18; no longer CON5.4, IC16.18
- net USB_VBUS: now also C1.1, C2.1, D1.K; no longer C3.1, C4.1, D4.K
- net V+: now also C73.1, C75.+, C76.+, FB5.2, IC12.1, IC12.4, IC3.1, IC3.4, IC4.1, IC4.4; no longer C68.+, FB6.2, IC10.1, IC10.4, IC9.1, IC9.4
- net VIN+: now also FB5.1; no longer FB6.1
- net XVCC: now also C3.1, C5.1, C6.1, FB2.2; no longer C1.1, C2.1
Routing:
- net +5V: track 0.00 -> 104.4 mm, vias 0 -> 2
- net +3V3: track 0.00 -> 54.6 mm, vias 0 -> 2
- net +3V3D: track 11.3 -> 65.7 mm, vias 0 -> 16
- net MCLR: track 0.00 -> 33.7 mm, vias 0 -> 1
- net PIC_COM2: track 0.00 -> 29.3 mm, vias 0 -> 2
- net PIC_COM3: track 0.00 -> 29.1 mm, vias 0 -> 2
- net USB_VBUS: track 0.00 -> 28.4 mm, vias 0 -> 2
- net PIC_COM1: track 0.00 -> 27.2 mm, vias 0 -> 2
- net V+: track 81.4 -> 105.4 mm
- net SWCLK: track 0.00 -> 21.7 mm
- net STM_IO16: track 0.00 -> 21.1 mm
- net STM_IO17: track 0.00 -> 20.0 mm
- net STM_IO20: track 0.00 -> 19.8 mm
- net UART_TX: track 5.46 -> 24.9 mm, vias 0 -> 1
- net XVCC: track 0.00 -> 18.9 mm
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- added copper zone on layer 1, net +3V3D
- added copper zone on layer 15, net +3V3D
- added copper zone on layer 1, net AMP_OUTN_L
- added copper zone on layer 1, net AMP_OUTN_R
- added copper zone on layer 1, net AMP_OUTP_L
- added copper zone on layer 1, net AMP_OUTP_R
- added copper zone on layer 1, net GND
- added copper zone on layer 15, net GND
- added copper zone on layer 16, net GND
- added copper zone on layer 2, net GND
- added copper zone on layer 1, net V+
Other:
- board size 5.1 x 8.6 mm -> 80 x 72 mm
- board text added: "USB Audio Amp"

Commit message: 微修正
Parts:
- added C89: 0.1u, my_rcl:1608C
- C22, C23, C51, C52, C77: device my_rcl:E5-10 -> my_rcl:E5-10-DUAL
Connections:
- net +3V3D: now also C89.1, IC2.34
- net GND: now also C22.--, C23.--, C51.--, C52.--, C77.--, C89.2
Routing:
- net +3V3D: track 65.7 -> 71.0 mm, vias 16 -> 17
- net GND: vias 547 -> 546

Commit message: TAS2770
Parts:
- removed C38, C42, C60, C61, C67, C71: 10u, my_rcl:2012
- removed C40, C54, C55, C58, C59, C64, C68: 0.1u, my_rcl:1608C
- removed C41, C53, C69: 10p, my_rcl:1608C
- removed C47, C62: 470p, my_rcl:1608C
- removed C49: 10u, my_rcl:3216
- removed C50, C65: 3.3n, my_rcl:1608C
- removed C52: 470u, my_rcl:E5-10-DUAL
- removed C56: 1u, my_rcl:1608C
- removed C63: 10n, my_rcl:1608C
- removed IC4, IC8: +5V, my_ic:TO220-SOP-DUAL
- removed R23, R30, R38: 330, my_rcl:1608
- removed R25, R26, R27, R33, R34, R40, R41, R42: 1k, my_rcl:1608
- removed R28, R35, R43: DNP, my_rcl:1608
- removed R36: DATA, my_rcl:1608-J
- removed R37: LRCLK, my_rcl:1608-J
- removed R39: SCK, my_rcl:1608-J
- added R14: DATA, my_rcl:1608-J
- C16, C43, C80, C84: device my_rcl:C050 -> my_rcl:C050W
- C18: value 470p -> 0.1u
- C20: value 10u -> 0.1u; device my_rcl:3216 -> my_rcl:1608C
- C21: value 3.3n -> 1u
- C23: value 470u -> 0.1u; device my_rcl:E5-10-DUAL -> my_rcl:1608C
- C24: value 10p -> 0.1u
- C29: value 0.1u -> 1u
- C30: value 0.1u -> 10u; device my_rcl:1608C -> my_rcl:2012
- C31: value 10u -> 0.1u; device my_rcl:2012 -> my_rcl:1608C
- C33: value 470p -> 1u
- C34: value 10n -> 0.1u
- C37: value 3.3n -> 0.1u
- IC5, IC9: value TAS2780 -> TAS2770; device my_ic:VQFN30 -> my_ic:VQFN26
- R15: value 330 -> LRCLK; device my_rcl:1608 -> my_rcl:1608-J
- R18: value 1k -> SCK; device my_rcl:1608 -> my_rcl:1608-J
- R19: value 1k -> ADDR
- R20: value DNP -> ADDR
- moved C23 136.6 mm to (-9.50, -62.5), turned to 0 degrees
- moved C37 133.8 mm to (-9.00, -74.0), flipped to the top, turned to 0 degrees
- moved C35 123.6 mm to (-9.00, -68.0)
- moved C20 123.2 mm to (-9.50, -59.0), turned to 0 degrees
- moved C33 107.1 mm to (-9.50, -46.5), flipped to the top, turned to 0 degrees
- moved R20 99.1 mm to (-9.50, -54.5), flipped to the top, turned to 0 degrees
- moved R19 96.0 mm to (-9.50, -51.0), flipped to the top, turned to 0 degrees
- moved C24 90.7 mm to (-1.50, -42.0), flipped to the top, turned to 0 degrees
- moved C34 87.3 mm to (-9.50, -25.5), turned to 0 degrees
- moved R18 87.1 mm to (-1.50, -46.5), flipped to the top, turned to 0 degrees
- moved C21 86.6 mm to (-5.50, -42.0), flipped to the top, turned to 0 degrees
- moved C32 86.4 mm to (-9.50, -21.0), turned to 0 degrees
- moved C18 85.4 mm to (-9.50, -42.0), flipped to the top, turned to 0 degrees
- moved C31 80.7 mm to (-9.50, -16.0), turned to 0 degrees
- moved R15 77.4 mm to (-2.00, -34.5), flipped to the top, turned to 0 degrees
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Connections:
- removed net AMP_VDD_1S_L: C20.1, C23.+, C30.1, C32.1, IC4.3, IC4.6, IC5.27
- removed net AMP_VDD_1S_R: C49.1, C52.+, C59.1, C61.1, IC8.3, IC8.6, IC9.27
- removed net N$14 (its old number): C34.1, IC5.26, R27.1
- removed net N$16 (its old number): IC5.13, R21.2
- removed net N$28: IC9.14, R37.2
- removed net N$29: IC9.15, R39.2
- removed net N$32: C47.2, C50.1, R34.1
- removed net N$33: C47.1, R30.2
- removed net N$34: C62.2, C65.1, R41.1
- removed net N$35: C62.1, R38.2
- removed net NC1: IC5.9-1, IC5.9-2
- removed net NC2: IC5.16-1, IC5.16-2
- removed net NC3: IC9.9-1, IC9.9-2
- removed net NC4: IC9.16-1, IC9.16-2
- new net AMP_PVDD_L: IC5.25
- new net AMP_PVDD_R: IC9.25
- new net N$12: IC5.13, R24.2
- new net N$17: C26.2, IC5.1
- net AMP_AVDD_L: now also C20.1, IC5.9; no longer C35.1, C38.1, IC5.24-1, IC5.24-2
- net AMP_AVDD_R: now also C37.1, IC9.9; no longer C64.1, C67.1, IC9.23, IC9.24-1, IC9.24-2
- net AMP_IOVDD_L: now also C30.1, C31.1, IC5.8; no longer C40.1, C42.1, IC5.20
- net AMP_IOVDD_R: now also C32.1, C34.1, IC9.8; no longer C68.1, C71.1, IC9.20
- net AMP_OUTN_L: now also IC5.26; no longer IC5.29, R26.2, R28.1
- net AMP_OUTN_R: now also C24.1, IC9.26; no longer C55.1, IC9.29, R41.2, R43.1
- net AMP_OUTP_L: no longer R19.2, R20.1
- net AMP_OUTP_R: now also C18.2; no longer C54.2, R34.2, R35.1
- net AMP_SDZ: now also IC5.21, IC9.21; no longer IC5.22, IC9.22
- net AMP_SNS_N_L: now also IC5.6; no longer C37.2, C41.1, IC5.1-1, IC5.1-2, R25.2, R28.2
- net AMP_SNS_N_R: now also IC9.6; no longer C65.2, C69.1, IC9.1-1, IC9.1-2, R40.2, R43.2
- net AMP_SNS_P_L: no longer C21.2, C24.1, R18.2, R20.2
- net AMP_SNS_P_R: no longer C50.2, C53.1, R33.2, R35.2
- net AMP_VDD_L: now also C23.1; no longer C29.1, C31.1, IC5.28, R27.2
- net AMP_VDD_R: now also C35.1; no longer C58.1, C60.1, IC9.28, R42.2
- net GND: now also C21.2, C23.2, C29.1, C33.1, C37.2, IC5.10, IC5.15, IC5.16, IC9.10, IC9.15, IC9.16, R19.2, R20.2; no longer C23.-, C23.--, C24.2, C29.2, C38.2, C40.2, C41.2, C42.2, C49.2, C52.-, C52.--, C53.2, C56.2, C58.2, C59.2, C60.2, C61.2, C63.2, C64.2, C67.2, C68.2, C69.2, C71.2, IC4.2, IC4.5, IC5.23, IC5.25, IC5.7, IC8.2, IC8.5, IC9.25, IC9.7
- net I2C_SCL: now also IC5.23, IC9.23; no longer IC5.18, IC9.18
- net I2C_SDA: now also IC5.22, IC9.22; no longer IC5.19, IC9.19
- net I2S_DATA: now also R14.1; no longer R36.1
- net I2S_LRCLK: now also R15.1; no longer R37.1
- net I2S_SCK: now also R18.1; no longer R39.1
- net N$10: now also IC9.11, R14.2; no longer C33.2, C37.1, R26.1
- net N$11: now also IC5.11, R21.2; no longer C26.2, IC5.30
- net N$13: now also IC9.13, R18.2; no longer C18.2, C21.1, R19.1
- net N$15: now also IC5.7; no longer IC5.10
- net N$18: now also C29.2, IC5.24; no longer IC5.15, R24.2
- net N$19: now also IC9.14, R15.2; no longer C33.1, R23.2
- net N$20: now also C21.1, IC9.7; no longer C18.1, R15.2
- net N$23: now also C18.1, IC9.4; no longer C55.2, IC9.30
- net N$24: now also C24.2, IC9.1; no longer C54.1, IC9.4
- net N$25: now also C33.2, IC9.24; no longer C63.1, IC9.26, R42.1
- net N$26: now also IC9.19, R19.1; no longer C56.1, IC9.10
- net N$27: now also IC5.19, R20.1; no longer IC9.13, R36.2
- net SP_OUTN_L: no longer R23.1, R25.1
- net SP_OUTN_R: no longer R38.1, R40.1
- net SP_OUTP_L: no longer R15.1, R18.1
- net SP_OUTP_R: no longer R30.1, R33.1
- net V+: no longer IC4.1, IC4.4, IC8.1, IC8.4
Routing:
- net V+: track 105.4 -> 0.00 mm
- net +5V: track 104.4 -> 0.00 mm, vias 2 -> 0
- net I2S_DATA: track 93.9 -> 0.00 mm, vias 4 -> 0
- net I2S_LRCLK: track 89.8 -> 0.00 mm, vias 2 -> 0
- net I2C_SDA: track 88.1 -> 0.00 mm, vias 3 -> 0
- net I2C_SCL: track 87.7 -> 0.00 mm, vias 2 -> 0
- net I2S_SCK: track 84.7 -> 0.00 mm
- net AMP_SDZ: track 83.5 -> 0.00 mm, vias 5 -> 0
- net +3V3D: track 71.0 -> 3.41 mm, vias 17 -> 2
- net +3V3: track 54.6 -> 0.00 mm, vias 2 -> 0
- net AMP_VDD_L: track 37.0 -> 0.00 mm, vias 2 -> 0
- net AMP_VDD_R: track 36.9 -> 0.00 mm, vias 2 -> 0
- net MCLR: track 33.7 -> 0.00 mm, vias 1 -> 0
- net PIC_COM2: track 29.3 -> 0.00 mm, vias 2 -> 0
- net PIC_COM3: track 29.1 -> 0.00 mm, vias 2 -> 0
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- removed copper zone on layer 1, net +3V3D
- removed copper zone on layer 1, net AMP_OUTN_L
- removed copper zone on layer 1, net AMP_OUTN_R
- removed copper zone on layer 1, net AMP_OUTP_L
- removed copper zone on layer 1, net AMP_OUTP_R
- removed copper zone on layer 1, net V+

Commit message: ver2
Parts:
- removed C66: 1u, my_rcl:1608C
- removed C70: 10u, my_rcl:3216
- removed C72, C73, C78, C89: 0.1u, my_rcl:1608C
- removed C74: DNP, my_rcl:1608C
- removed C75, C76: 1000u, my_rcl:E5-10
- removed C77: 470u, my_rcl:E5-10-DUAL
- removed C79: 22u, my_rcl:2012
- removed C80, C84: 0.47uF, my_rcl:C050W
- removed C81, C85: 0.47uF, my_rcl:3225-3
- removed C82, C83, C86, C87: 1n, my_rcl:1608-2
- removed C88: 22u, my_rcl:3225
- removed IC10: 1.8V, my_ic:SOT23-5
- removed IC11: STM32G031F, my_ic:TSSOP20
- removed IC12: +5V, my_ic:TO220-SOP-DUAL
- removed IC13: 3.3V, my_ic:SOT23-5
- removed R31, R32: 10, my_rcl:2012
- removed R44: 100k, my_rcl:1608
- removed R45, R46, R47, R48: 10k, my_rcl:1608
- removed R49: 1k, my_rcl:1608
- removed TP5: VIN+, my_connector:TESTPIN-BIG
- removed TP6: VIN-, my_connector:TESTPIN-BIG
- added C38: 47u, my_rcl:E2.5-5
- added C40: 10u, my_rcl:2012
- added C41, C42, C54, C55: DNP, my_rcl:1608-2
- added C47: 100p, my_rcl:1608-2
- added C49: 0.1u, my_rcl:C050W
- added C50: 0.47uF, my_rcl:C050W
- added C52, C53: 470u, my_rcl:E5-10
- added C56: 1000u, my_rcl:E5-13
- added C58, C63: 0.1u, my_rcl:1608C
- added C59: DNP, my_rcl:1608C
- added C60, C61: 1000u, my_rcl:E5-10
- added C62: 220u, my_rcl:E2,5-8
- added C64: 22u, my_rcl:2012
- added CON5: SWD, my_connector:SWD_CON
- added D5: PWR, my_rcl:D1608
- added FB6, FB7, FB8: FB, my_rcl:2012-FB
- added FB9: FB, my_rcl:3216-FB
- added IC4, IC8: +5V, my_ic:TO220-SOP-DUAL
- added Q1: NPN, my_ic:SC59
- added Q2: NPN, my_ic:SOT223
- added R23, R25, R26: 10k, my_rcl:1608
- C12, C13: value 22p -> 0.1u
- C14: value 0.47uF -> 22p; device my_rcl:3225-3 -> my_rcl:1608C
- C15: value 10n -> 22p; device my_rcl:3216-3 -> my_rcl:1608C
- C16: value 0.47uF -> 0.22u; device my_rcl:C050W -> my_rcl:1608C
- C17: value 10n -> 0.22u; device my_rcl:3216-3 -> my_rcl:1608C
- C18: value 0.1u -> 0.22u
- C19: value 10u -> 0.22u; device my_rcl:3216 -> my_rcl:1608C
- C20: value 0.1u -> 10n; device my_rcl:1608C -> my_rcl:1005
- C21: value 1u -> 10n; device my_rcl:1608C -> my_rcl:1005
- C22: value 470u -> 0.1u; device my_rcl:E5-10-DUAL -> my_rcl:1608C
- C24, C25: device my_rcl:1608C -> my_rcl:1005
- C26: value 0.1u -> 10u; device my_rcl:1608C -> my_rcl:2012
- C27: value 1u -> 10u; device my_rcl:1608C -> my_rcl:2012
- C28, C29, C33: value 1u -> 100p; device my_rcl:1608C -> my_rcl:1608-2
- C30: value 10u -> 0.1u; device my_rcl:2012 -> my_rcl:1608C
- C32: value 10u -> 100p; device my_rcl:2012 -> my_rcl:1608-2
- C34, C35: device my_rcl:1608C -> my_rcl:C050W
- C36: value 1u -> 0.47uF; device my_rcl:1608C -> my_rcl:C050W
- C37: value 0.1u -> 0.47uF; device my_rcl:1608C -> my_rcl:C050W
- C39: value 10u -> 0.1u; device my_rcl:3216 -> my_rcl:1608C
- C43: value 0.47uF -> 10u; device my_rcl:C050W -> my_rcl:2012
- C44, C46: value 10n -> 100p; device my_rcl:3216-3 -> my_rcl:1608-2
- C45: value 0.47uF -> 100p; device my_rcl:3225-3 -> my_rcl:1608-2
- C48: value 10u -> 0.1u; device my_rcl:3216 -> my_rcl:C050W
- C51: value 470u -> 0.47uF; device my_rcl:E5-10-DUAL -> my_rcl:C050W
- C57: value 1u -> 0.1u
- C7: value 0.1u -> 22u; device my_rcl:1608C -> my_rcl:3225
- CON2: value PIC32_CON -> PROG
- CON3: value VOLUEME -> DC IN; device my_connector:VOL_CON -> my_connector:2.1MM_CON
- CON4: value SWD -> VOLUEME; device my_connector:SWD_CON -> my_connector:VOL_CON
- D1: value SBD-E -> SBD
- D4: value PWR -> 5.6mA; device my_rcl:D1608 -> my_rcl:SOD123
- IC3: value +12V -> SSM3582; device my_ic:TO220-SOP-DUAL -> my_ic:QFN40HT
- IC5: value TAS2770 -> 1.8V; device my_ic:VQFN26 -> my_ic:SOT23-5
- IC6: value 1.8V -> TL431; device my_ic:SOT23-5 -> my_ic:SOT89
- IC7: value +12V -> STM32G031F; device my_ic:TO220-SOP-DUAL -> my_ic:TSSOP20
- IC9: value TAS2770 -> 3.3V; device my_ic:VQFN26 -> my_ic:SOT23-5
- R13: value 1k -> LRCLK; device my_rcl:1608 -> my_rcl:1608-J
- R15: value LRCLK -> SCK
- R18: value SCK -> 1k; device my_rcl:1608-J -> my_rcl:1608
- R19, R20: value ADDR -> 10; device my_rcl:1608 -> my_rcl:2012
- R21: value DATA -> 3.6k; device my_rcl:1608-J -> my_rcl:1608
- R22: value LRCLK -> 1k; device my_rcl:1608-J -> my_rcl:1608
- R24: value SCK -> 100k; device my_rcl:1608-J -> my_rcl:1608
- moved R20 119.7 mm to (25.2, 60.0), flipped to the bottom, turned to 270 degrees
- moved R19 114.1 mm to (16.8, 60.0), flipped to the bottom, turned to 90 degrees
- moved R18 106.3 mm to (36.0, 53.0), turned to 270 degrees
- moved IC9 105.0 mm to (60.5, 44.5), turned to 180 degrees
- moved C23 102.4 mm to (14.5, 37.0), turned to 180 degrees
- moved C20 94.1 mm to (22.5, 29.5)
- moved C37 93.8 mm to (26.0, 13.0), turned to 180 degrees
- moved R14 89.6 mm to (29.5, 36.0), turned to 180 degrees
- moved C21 89.0 mm to (22.5, 42.5)
- moved C35 84.1 mm to (29.0, 7.00)
- moved R15 79.0 mm to (29.5, 38.0), turned to 180 degrees
- moved C18 77.7 mm to (17.0, 31.0), turned to 90 degrees
- moved C15 76.2 mm to (68.8, 11.8), flipped to the top, turned to 270 degrees
- moved FB4 75.7 mm to (2.50, 44.8), flipped to the bottom, turned to 270 degrees
- moved C24 74.5 mm to (19.5, 29.5), turned to 180 degrees
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Connections:
- removed net AMP_AVDD_L: C20.1, C39.1, IC5.9, IC6.5
- removed net AMP_AVDD_R: C37.1, C70.1, IC10.5, IC9.9
- removed net AMP_IOVDD_L: C30.1, C31.1, FB3.1, IC5.8
- removed net AMP_IOVDD_R: C32.1, C34.1, FB4.1, IC9.8
- removed net AMP_PVDD_L: IC5.25
- removed net AMP_PVDD_R: IC9.25
- removed net AMP_SDZ: IC5.21, IC9.21, R49.1
- removed net AMP_SNS_N_L: IC5.6
- removed net AMP_SNS_N_R: IC9.6
- removed net AMP_SNS_P_L: IC5.5
- removed net AMP_SNS_P_R: IC9.5
- removed net AMP_VDD_L: C19.1, C22.+, C23.1, IC3.3, IC3.6
- removed net AMP_VDD_R: C35.1, C48.1, C51.+, IC7.3, IC7.6
- removed net N$25: C33.2, IC9.24
- removed net N$26: IC9.19, R19.1
- removed net N$27: IC5.19, R20.1
- removed net N$37: IC11.3, R45.2, R49.2
- removed net N$42: C36.1, IC6.4
- removed net N$44: C66.1, IC10.4
- removed net N$6: IC2.32, R13.2
- new net +12V: C20.1, C21.1, C24.1, C25.1, C26.1, C27.1, C52.+, C53.+, C56.+, IC3.14, IC3.15, IC3.16, IC3.17, IC3.34, IC3.35, IC3.36, IC3.37, Q2.3, R18.2, R21.2
- new net AMP_AVDD: C23.1, C38.+, C40.1, IC3.24, IC4.3, IC4.6
- new net AMP_DVDD: C22.1, C43.1, IC3.28, IC5.5
- net +3V3: now also C57.1, C64.1, CON4.1, D5.A, IC7.4, IC9.5, R25.2, R26.2; no longer C72.1, C79.1, CON3.1, D4.A, IC11.4, IC13.5, R46.2, R47.2
- net +3V3D: now also C12.1, C13.1; no longer C88.1, C89.1, FB3.2, FB4.2
- net +5V: now also C62.+, C63.1, FB3.1, IC8.3, IC8.6, IC9.1, IC9.3; no longer C28.1, C57.1, C77.+, C78.1, IC10.1, IC10.3, IC12.3, IC12.6, IC13.1, IC13.3, IC6.1, IC6.3
- net AMP_OUTN_L: now also C18.1, C41.2, FB5.2, IC3.32, IC3.33; no longer C26.1, IC5.26
- net AMP_OUTN_R: now also C19.2, C54.2, FB7.2, IC3.18, IC3.19, L3.2; no longer C24.1, IC9.26, L3.1
- net AMP_OUTP_L: now also C16.1, C42.1, FB6.1, IC3.38, IC3.39, L2.2; no longer C25.2, IC5.3, L2.1
- net AMP_OUTP_R: now also C17.2, C55.1, FB8.1, IC3.12, IC3.13; no longer C18.2, IC9.3
- net EN_DDC: now also IC7.8; no longer IC11.8
- net GND: now also C15.2, C22.2, C24.2, C25.2, C26.2, C28.1, C29.2, C32.1, C33.2, C34.1, C34.3, C35.4, C36.1, C36.3, C37.1, C37.3, C38.-, C40.2, C41.1, C42.2, C43.2, C46.1, C47.2, C48.1, C48.3, C49.2, C49.4, C50.1, C50.3, C51.1, C51.3, C52.-, C53.-, C54.1, C55.2, C56.-, C58.2, C59.2, C60.-, C61.-, C62.-, C63.2, C64.2, CON3.2, CON3.4, CON3.5, CON3.6, CON5.3, IC3.1, IC3.10, IC3.21, IC3.22, IC3.23, IC3.25, IC3.26, IC3.27, IC3.29, IC3.3, IC3.30, IC3.9, IC3.HT, IC3.HT1, IC3.HT2, IC3.HT3, IC3.HT4, IC4.2, IC4.5, IC8.2, IC8.5, R22.1, R23.1, R24.1; no longer C15.1, C16.1, C17.2, C19.2, C22.-, C22.--, C28.2, C29.1, C32.2, C33.1, C34.2, C36.2, C37.2, C43.1, C46.2, C48.2, C51.-, C51.--, C66.2, C70.2, C72.2, C73.2, C74.2, C75.-, C76.-, C77.-, C77.--, C78.2, C79.2, C80.1, C81.2, C82.2, C83.1, C84.1, C85.2, C86.2, C87.1, C88.2, C89.2, IC10.2, IC11.5, IC12.2, IC12.5, IC13.2, IC3.5, IC5.10, IC5.15, IC5.16, IC7.2, IC9.10, IC9.15, IC9.16, R19.2, R20.2, R44.1, R45.1, R48.1, TP6.1
- net I2C_SCL: now also IC3.4, IC7.1, R25.1; no longer IC11.1, IC5.23, IC9.23, R46.1
- net I2C_SDA: now also IC3.5, IC7.2, R26.1; no longer IC11.2, IC5.22, IC9.22, R47.1
- net I2S_DATA: no longer R21.1
- net I2S_LRCLK: now also R13.1; no longer R15.1, R22.1
- net I2S_SCK: now also R15.1; no longer R18.1, R24.1
- net N$10: now also IC3.6, R13.2; no longer IC9.11, R14.2
- net N$11: now also IC3.7, R14.2; no longer IC5.11, R21.2
- net N$12: now also C18.2, IC3.31; no longer IC5.13, R24.2
- net N$13: now also C16.2, IC3.40; no longer IC9.13, R18.2
- net N$14: now also IC3.8, R15.2; no longer IC5.14, R22.2
- net N$15: now also C39.1, IC5.4; no longer C27.1, IC5.7
- net N$16: now also Q1.2, Q2.1, R18.1; no longer C25.1, IC5.4
- net N$17: now also C17.1, IC3.11; no longer C26.2, IC5.1
- net N$18: now also C19.1, IC3.20; no longer C29.2, IC5.24
- net N$19: now also C30.1, FB3.2, IC5.1, IC5.3; no longer IC9.14, R15.2
- net N$20: now also IC6.1, R21.1, R22.2; no longer C21.1, IC9.7
- net N$21: now also C34.2, C34.4; no longer C15.2
- net N$22: now also C35.1, C35.3; no longer C17.1
- net N$23: now also D4.2, IC6.3, Q1.1; no longer C18.1, IC9.4
- net N$24: now also C31.1, FB4.2, IC4.1, IC4.4; no longer C24.2, IC9.1
- net N$30: now also C48.2, C48.4, R19.2; no longer C44.2, R31.2
- net N$31: now also C49.1, C49.3, R20.1; no longer C46.1, R32.1
- net N$36: now also D5.K, R23.2; no longer D4.K, R48.2
- net N$5: now also C14.1; no longer C12.1
- net N$7: now also C15.1, IC2.32; no longer C13.1, R13.1
- net N$72: now also C59.1, CON4.2, IC7.11, R24.2; no longer C74.1, CON3.2, IC11.11, R44.2
- net PIC_COM1: now also IC7.12; no longer IC11.12
- net PIC_COM2: now also IC7.13; no longer IC11.13
- net PIC_COM3: now also IC7.14; no longer IC11.14
- net SP_OUTN_L: now also C28.2, C32.2, C36.2, C36.4, FB5.1; no longer C80.2, C81.1, C83.2
- net SP_OUTN_R: now also C44.2, C46.2, C50.2, C50.4, FB7.1, L3.1, R19.1; no longer C43.2, C45.1, C87.2, L3.2, R31.1
- net SP_OUTP_L: now also C29.1, C33.1, C37.2, C37.4, FB6.2, L2.1; no longer C14.1, C16.2, C82.1, L2.2
- net SP_OUTP_R: now also C45.1, C47.1, C51.2, C51.4, FB8.2, R20.2; no longer C84.2, C85.1, C86.1, R32.2
- net STM_IO16: now also IC7.16; no longer IC11.16
- net STM_IO17: now also IC7.17; no longer IC11.17
- net STM_IO20: now also IC7.20; no longer IC11.20
- net STM_TX: now also CON5.5, IC7.9; no longer CON4.5, IC11.9
- net SWCLK: now also CON5.1, IC7.19; no longer CON4.1, IC11.19
- net SWDIO: now also CON5.4, IC7.18; no longer CON4.4, IC11.18
- net V+: now also C58.1, C60.+, C61.+, D4.1, FB4.1, FB9.2, IC8.1, IC8.4, Q1.3, Q2.2, Q2.4; no longer C73.1, C75.+, C76.+, FB5.2, IC12.1, IC12.4, IC3.1, IC3.4, IC7.1, IC7.4
- net VIN+: now also CON3.1, FB9.1; no longer FB5.1, TP5.1
Routing:
- net +5V: track 0.00 -> 97.1 mm
- net V+: track 0.00 -> 68.4 mm
- net I2C_SDA: track 0.00 -> 51.9 mm, vias 0 -> 2
- net +12V: track 0.00 -> 51.8 mm, vias 0 -> 12
- net I2C_SCL: track 0.00 -> 51.4 mm, vias 0 -> 2
- net +3V3: track 0.00 -> 42.4 mm, vias 0 -> 2
- net I2S_SCK: track 0.00 -> 39.8 mm
- net GND: track 0.00 -> 39.1 mm, vias 0 -> 337
- net I2S_LRCLK: track 0.00 -> 36.7 mm
- net I2S_DATA: track 0.00 -> 35.7 mm
- net PIC_COM3: track 0.00 -> 35.6 mm, vias 0 -> 2
- net PIC_COM2: track 0.00 -> 34.6 mm, vias 0 -> 2
- net MCLR: track 0.00 -> 33.2 mm, vias 0 -> 1
- net PIC_COM1: track 0.00 -> 32.8 mm, vias 0 -> 2
- net USB_VBUS: track 0.00 -> 30.4 mm, vias 0 -> 2
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- added copper zone on layer 1, net +12V
- added copper zone on layer 16, net +12V
- added copper zone on layer 1, net AMP_OUTN_L
- added copper zone on layer 1, net AMP_OUTN_R
- added copper zone on layer 1, net AMP_OUTP_L
- added copper zone on layer 1, net AMP_OUTP_R
- added copper zone on layer 1, net V+
- added copper zone on layer 16, net V+
Other:
- board text added: "ver2"

Commit message: インダクタ変更
Parts:
- removed D5: PWR, my_rcl:D1608
- removed L3, L4: 15uH, my_rcl:L5-7,5
- added C65: 0.1u, my_rcl:1608C
- added C66: 22u, my_rcl:2012
- added Q3: NPN, my_ic:SOT223
- added R27, R28: 1k, my_rcl:3216-3
- C26, C27: device my_rcl:2012 -> my_rcl:3225-2
- C46: value 100p -> DNP; device my_rcl:1608-2 -> my_rcl:1608C
- C48: value 0.1u -> 100p; device my_rcl:C050W -> my_rcl:1608-2
- C50: value 0.47uF -> 0.1u
- C52: value 470u -> 0.47uF; device my_rcl:E5-10 -> my_rcl:C050W
- C53: value 470u -> DNP; device my_rcl:E5-10 -> my_rcl:1608C
- C54: value DNP -> 470u; device my_rcl:1608-2 -> my_rcl:E5-10
- C56: value 1000u -> DNP; device my_rcl:E5-13 -> my_rcl:1608-2
- C57: value 0.1u -> 470u; device my_rcl:1608C -> my_rcl:E5-10
- C58: value 0.1u -> 1000u; device my_rcl:1608C -> my_rcl:E5-13
- C59: value DNP -> 0.1u
- C60: value 1000u -> 0.1u; device my_rcl:E5-10 -> my_rcl:1608C
- C61: value 1000u -> DNP; device my_rcl:E5-10 -> my_rcl:1608C
- C62: value 220u -> 1000u; device my_rcl:E2,5-8 -> my_rcl:E5-10
- C63: value 0.1u -> 1000u; device my_rcl:1608C -> my_rcl:E5-10
- C64: value 22u -> 220u; device my_rcl:2012 -> my_rcl:E2,5-8
- D4: value 5.6mA -> PWR; device my_rcl:SOD123 -> my_rcl:D1608
- L1, L2: value 15uH -> 10uH; device my_rcl:L5-7,5 -> my_rcl:CSD1013
- Q1: value NPN -> JFET
- Q2: device my_ic:SOT223 -> my_ic:SC59
- R16, R17, R19, R20: device my_rcl:2012 -> my_rcl:3216-3
- moved C58 42.4 mm to (39.5, 16.0), flipped to the top, turned to 0 degrees
- moved C57 37.4 mm to (34.0, 43.5), turned to 270 degrees
- moved C52 34.4 mm to (26.0, 62.0), turned to 180 degrees
- moved L2 32.4 mm to (21.0, 53.0), turned to 0 degrees
- moved C56 31.6 mm to (24.8, 44.0), turned to 180 degrees
- moved D4 30.3 mm to (73.0, 55.0)
- moved C54 22.8 mm to (34.0, 28.5), turned to 90 degrees
- moved C61 21.9 mm to (73.0, 51.0), turned to 180 degrees
- moved C46 18.1 mm to (35.0, 58.0)
- moved C49 16.8 mm to (12.5, 68.0)
- moved C50 16.2 mm to (29.5, 68.0)
- moved C59 13.2 mm to (71.0, 38.0), turned to 0 degrees
- moved C63 10.9 mm to (53.0, 42.0), turned to 0 degrees
- moved C51 10.4 mm to (16.0, 62.0), turned to 0 degrees
- moved C62 10.0 mm to (53.0, 53.0), turned to 0 degrees
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Connections:
- net +12V: now also C53.1, C54.+, C57.+, C58.+, Q3.3, R27.2, R28.2; no longer C52.+, C53.+, C56.+, Q2.3
- net +3V3: now also C59.1, C66.1, D4.A; no longer C57.1, C64.1, D5.A
- net +5V: now also C64.+, C65.1; no longer C62.+, C63.1
- net AMP_OUTN_R: now also C55.2, L2.2; no longer C54.2, L3.2
- net AMP_OUTP_L: now also L1.4; no longer L2.2
- net AMP_OUTP_R: now also C56.1, L2.3; no longer C55.1, L4.1
- net GND: now also C47.1, C48.2, C49.1, C49.3, C50.2, C50.4, C52.1, C52.3, C54.-, C55.1, C56.2, C57.-, C58.-, C60.2, C61.2, C63.-, C64.-, C65.2, C66.2, R27.1, R28.1; no longer C46.1, C47.2, C48.1, C48.3, C49.2, C49.4, C50.1, C50.3, C52.-, C53.-, C54.1, C55.2, C56.-, C57.2, C58.2, C60.-, C61.-, C63.2, C64.2
- net N$16: now also Q2.2, Q3.1; no longer Q1.2, Q2.1
- net N$20: now also C46.2, C53.2
- net N$23: now also C46.1, Q1.3, Q2.1; no longer D4.2
- net N$30: now also C49.2, C49.4; no longer C48.2, C48.4
- net N$31: now also C50.1, C50.3; no longer C49.1, C49.3
- net N$36: now also D4.K; no longer D5.K
- net N$72: now also C61.1; no longer C59.1
- net SP_OUTN_R: now also C47.2, C51.2, C51.4, L2.1; no longer C46.2, C50.2, C50.4, L3.1
- net SP_OUTP_L: now also L1.3; no longer L2.1
- net SP_OUTP_R: now also C48.1, C52.2, C52.4, L2.4; no longer C47.1, C51.2, C51.4, L4.2
- net V+: now also C60.1, C62.+, C63.+, Q1.2, Q2.3, Q3.2, Q3.4; no longer C58.1, C60.+, C61.+, D4.1, Q1.3, Q2.2, Q2.4
Routing:
- net SP_OUTP_R: track 22.6 -> 4.44 mm
- net SP_OUTN_R: track 22.5 -> 4.44 mm
- net SP_OUTN_L: track 22.2 -> 4.44 mm
- net SP_OUTP_L: track 22.3 -> 5.15 mm
- net N$23: track 10.7 -> 17.9 mm
- net N$20: track 10.5 -> 12.8 mm
- net AMP_OUTP_L: track 7.15 -> 5.51 mm
- net +5V: track 97.1 -> 98.5 mm
- net AMP_OUTN_L: track 6.90 -> 5.51 mm
- net AMP_OUTN_R: track 7.40 -> 6.01 mm
- net N$31: track 5.98 -> 4.84 mm
- net N$30: track 5.98 -> 4.84 mm
- net N$22: track 5.98 -> 4.84 mm
- net N$21: track 5.98 -> 4.84 mm
- net N$16: track 10.4 -> 9.72 mm
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- added copper zone on layer 1, net SP_OUTN_L
- added copper zone on layer 1, net SP_OUTN_R
- added copper zone on layer 1, net SP_OUTP_L
- added copper zone on layer 1, net SP_OUTP_R
