File: USB_Amp.brd (EAGLE design)
At the start: 80 x 72 mm, 142 parts, among them CON1 USB-C, CON2 PROG, CON3 DC IN, CON4 VOLUEME, CON5 SWD, IC1 3.3V, IC2 PIC32MZEF, IC3 SSM3582, IC4 +5V, IC5 1.8V, IC6 TL431, IC7 STM32G031F, IC8 +5V, IC9 3.3V, Q1 JFET, Q2 NPN, Q3 NPN, X1 24.576MHz, X2 22.5792MHz, X3 12MHz

Commit message: 発注
Parts:
- added C67: DNP, my_rcl:1608C
- added C68: 1000u, my_rcl:E5-10
- added C69: 220u, my_rcl:E2,5-8
- added C70: 0.1u, my_rcl:1608C
- added C71: 22u, my_rcl:2012
- added IC10: STM32G031F, my_ic:TSSOP20
- added IC11: +5V, my_ic:TO220-SOP-DUAL
- added IC12: 3.3V, my_ic:SOT23-5
- added R29, R30, R31, R32, R33: 10k, my_rcl:1608
- added R34, R35: 1k, my_rcl:3216
- C14, C15: value 22p -> 0.1u
- C16, C19: value 0.22u -> 0.1u
- C17, C18: value 0.22u -> 22p
- C20, C21: value 10n -> 0.1u; device my_rcl:1005 -> my_rcl:1608C
- C23: value 0.1u -> 1u
- C24, C25: value 0.1u -> 1u; device my_rcl:1005 -> my_rcl:1608C
- C26: value 10u -> 1u; device my_rcl:3225-2 -> my_rcl:1608C
- C27: value 10u -> 0.1u; device my_rcl:3225-2 -> my_rcl:1005
- C28: value 100p -> 0.1u; device my_rcl:1608-2 -> my_rcl:1005
- C29: value 100p -> 1u
- C3: value 10u -> 0.1u; device my_rcl:2012 -> my_rcl:1608C
- C30: value 0.1u -> 1u; device my_rcl:1608C -> my_rcl:1608-2
- C31: value 0.1u -> 10u; device my_rcl:1608C -> my_rcl:3225-3
- C32: value 100p -> 10u; device my_rcl:1608-2 -> my_rcl:3225-3
- C33: value 100p -> 0.1u; device my_rcl:1608-2 -> my_rcl:1608C
- C34, C49, C50: device my_rcl:C050W -> my_rcl:1608C
- C35: value 0.1u -> 100p; device my_rcl:C050W -> my_rcl:1608-2
- C36, C37, C51, C52: value 0.47uF -> 100p; device my_rcl:C050W -> my_rcl:1608-2
- C38: value 47u -> 100p; device my_rcl:E2.5-5 -> my_rcl:1608-2
- C39: device my_rcl:1608C -> my_rcl:C050W2
- C40: value 10u -> 0.1u; device my_rcl:2012 -> my_rcl:C050W2
- C41, C42: value DNP -> 0.1u; device my_rcl:1608-2 -> my_rcl:1608C
- C43: value 10u -> 0.47uF; device my_rcl:2012 -> my_rcl:C050W
- C44: value 100p -> 0.47uF; device my_rcl:1608-2 -> my_rcl:C050W
- C45: value 100p -> 22u; device my_rcl:1608-2 -> my_rcl:3225
- C46: value DNP -> 22u; device my_rcl:1608C -> my_rcl:3225
- C47, C48: value 100p -> 10u; device my_rcl:1608-2 -> my_rcl:2012
- C5, C9: value 0.1u -> 10u; device my_rcl:1608C -> my_rcl:2012
- C53: value DNP -> 100p; device my_rcl:1608C -> my_rcl:1608-2
- C54: value 470u -> 100p; device my_rcl:E5-10 -> my_rcl:1608-2
- C55: device my_rcl:1608-2 -> my_rcl:1608C
- C56: value DNP -> 0.1u; device my_rcl:1608-2 -> my_rcl:C050W2
- C57: value 470u -> 0.1u; device my_rcl:E5-10 -> my_rcl:C050W2
- C58: value 1000u -> 0.47uF; device my_rcl:E5-13 -> my_rcl:C050W
- C59: value 0.1u -> 0.47uF; device my_rcl:1608C -> my_rcl:C050W
- C60: value 0.1u -> DNP
- C61: value DNP -> 470u; device my_rcl:1608C -> my_rcl:E5-10
- C62: value 1000u -> 470u
- C63: device my_rcl:E5-10 -> my_rcl:E5-13
- C64: value 220u -> 0.1u; device my_rcl:E2,5-8 -> my_rcl:1608C
- C66: value 22u -> 1000u; device my_rcl:2012 -> my_rcl:E5-10
- C7: value 22u -> 0.1u; device my_rcl:3225 -> my_rcl:1608C
- C8: value 0.1u -> 22u; device my_rcl:1608C -> my_rcl:3225
- IC2: value PIC32MZEF -> 1.8V; device my_ic:QFN64HT -> my_ic:SOT23-5
- IC3: value SSM3582 -> 7WZ07; device my_ic:QFN40HT -> my_ic:SOT765
- IC4: value +5V -> PIC32MZEF; device my_ic:TO220-SOP-DUAL -> my_ic:QFN64HT
- IC5: value 1.8V -> TAS2770; device my_ic:SOT23-5 -> my_ic:VQFN26
- IC6: value TL431 -> TAS2770; device my_ic:SOT89 -> my_ic:VQFN26
- IC7: value STM32G031F -> 1.8V; device my_ic:TSSOP20 -> my_ic:SOT23-5
- IC8: value +5V -> 1.8V; device my_ic:TO220-SOP-DUAL -> my_ic:SOT23-5
- IC9: value 3.3V -> TL431; device my_ic:SOT23-5 -> my_ic:SOT89
- R11: value DATA -> 10k; device my_rcl:1608-J -> my_rcl:1608
- R12: value SCK -> 10k; device my_rcl:1608-J -> my_rcl:1608
- R13: value LRCLK -> 1k; device my_rcl:1608-J -> my_rcl:1608
- R14: value DATA -> 1k; device my_rcl:1608-J -> my_rcl:1608
- R15: value SCK -> 1k; device my_rcl:1608-J -> my_rcl:1608
- R16: value 10 -> 1k; device my_rcl:3216-3 -> my_rcl:1608
- R17: value 10 -> ADDR; device my_rcl:3216-3 -> my_rcl:1608
- R18: value 1k -> ADDR
- R21: value 3.6k -> 10; device my_rcl:1608 -> my_rcl:3216-3
- R22: value 1k -> 10; device my_rcl:1608 -> my_rcl:3216-3
- R23, R25: value 10k -> 1k
- R24: value 100k -> 3.6k
- R27: value 1k -> 100k; device my_rcl:3216-3 -> my_rcl:1608
- R28: value 1k -> 10k; device my_rcl:3216-3 -> my_rcl:1608
- R8: value 10k -> DATA; device my_rcl:1608 -> my_rcl:1608-J
- R9: value 10k -> SCK; device my_rcl:1608 -> my_rcl:1608-J
- TP3: value R_P -> R_N
- TP4: value R_N -> R_P
- moved IC4 70.4 mm to (72.5, 20.0), turned to 270 degrees
- moved C18 64.7 mm to (78.8, 11.8), turned to 270 degrees
- moved C59 62.0 mm to (10.0, 27.0), turned to 270 degrees
- moved C17 60.0 mm to (75.8, 9.00), turned to 0 degrees
- moved IC8 59.5 mm to (29.5, 12.5), turned to 270 degrees
- moved IC3 53.8 mm to (74.5, 30.0)
- moved R27 53.4 mm to (83.0, 49.0), flipped to the top
- moved TP2 52.8 mm to (2.00, 52.0), turned to 0 degrees
- moved TP4 52.8 mm to (2.00, 20.0), turned to 0 degrees
- moved C48 52.0 mm to (34.2, 15.8), turned to 270 degrees
- moved C50 51.8 mm to (32.0, 16.2), turned to 270 degrees
- moved TP1 50.6 mm to (2.00, 48.0), turned to 0 degrees
- moved TP3 50.6 mm to (2.00, 24.0), turned to 0 degrees
- moved C35 49.9 mm to (15.0, 51.8), turned to 90 degrees
- moved C16 49.0 mm to (74.0, 29.0), flipped to the bottom, turned to 180 degrees
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Connections:
- removed net AMP_AVDD: C23.1, C38.+, C40.1, IC3.24, IC4.3, IC4.6
- removed net AMP_DVDD: C22.1, C43.1, IC3.28, IC5.5
- removed net N$40: IC2.48, IC2.49, R12.1
- removed net N$41: IC2.50, R11.1
- removed net N$43: IC2.52, R10.1
- new net +1V8: C16.1, C9.1, IC2.5, IC3.8
- new net AMP_AVDD_L: C45.1, C47.1, C49.1, IC5.8, IC5.9, IC7.5
- new net AMP_AVDD_R: C46.1, C48.1, C50.1, IC6.8, IC6.9, IC8.5
- new net AMP_SDZ: IC5.21, IC6.21, R32.2, R33.1
- new net I2S_DATA_PIC: IC3.1, IC4.50
- new net I2S_LRCLK_PIC: IC3.6, IC4.52
- new net I2S_SCK_PIC: IC3.3, IC4.48, IC4.49
- new net N$25: C26.2, IC6.24
- new net N$26: IC6.19, R18.2
- new net N$27: C24.1, IC6.7
- new net N$28: IC6.6, R16.1
- new net N$29: IC6.5, R14.2
- new net N$32: IC10.3, R32.1
- new net N$33: IC3.7, R8.2
- new net N$34: IC3.5, R9.2
- new net N$35: IC3.2, R10.2
- new net N$37: C42.1, IC8.4
- new net N$38: C34.1, FB4.2, IC8.1, IC8.3
- new net N$6: C19.1, IC5.4
- net +12V: now also C28.1, C29.1, C30.1, C31.1, C32.1, C60.1, C61.+, C62.+, C63.+, IC5.25, IC6.25, R23.2, R24.2, R34.2, R35.2; no longer C20.1, C21.1, C24.1, C25.1, C26.1, C53.1, C54.+, C57.+, C58.+, IC3.14, IC3.15, IC3.16, IC3.17, IC3.34, IC3.35, IC3.36, IC3.37, R18.2, R21.2, R27.2, R28.2
- net +3V3: now also C64.1, C71.1, IC10.4, IC12.5, R28.2, R30.2; no longer C59.1, C66.1, IC7.4, IC9.5, R25.2, R26.2
- net +3V3D: now also C14.1, C15.1, C5.1, IC4.19, IC4.26, IC4.34, IC4.39, IC4.54, IC4.60, IC4.8; no longer C4.1, C7.1, C9.1, IC2.19, IC2.26, IC2.34, IC2.39, IC2.54, IC2.60, IC2.8
- net +5V: now also C3.1, C69.+, C70.1, FB4.1, IC11.3, IC11.6, IC12.1, IC12.3, IC2.1, IC2.3; no longer C64.+, C65.1, IC8.3, IC8.6, IC9.1, IC9.3
- net AMP_OUTN_L: now also C20.1, IC5.26, R15.2; no longer C18.1, C41.2, IC3.32, IC3.33
- net AMP_OUTN_R: now also C22.1, FB8.1, IC6.26, L2.3, R16.2; no longer C19.2, C55.2, FB7.2, IC3.18, IC3.19, L2.2
- net AMP_OUTP_L: now also C19.2, IC5.3, R13.1; no longer C16.1, C42.1, IC3.38, IC3.39
- net AMP_OUTP_R: now also C21.2, FB7.2, IC6.3, L2.2, R14.1; no longer C17.2, C56.1, FB8.1, IC3.12, IC3.13, L2.3
- net EN_44.1K: now also IC4.29, R12.2; no longer IC2.29, R9.2
- net EN_48K: now also IC4.28, R11.2; no longer IC2.28, R8.2
- net EN_DDC: now also IC10.8; no longer IC7.8
- net GND: now also C16.2, C17.2, C18.2, C25.1, C26.1, C28.2, C32.2, C34.2, C35.1, C36.2, C38.2, C39.1, C39.3, C40.4, C41.2, C43.1, C43.3, C44.3, C46.2, C47.2, C49.2, C52.2, C53.1, C54.2, C56.1, C56.3, C57.2, C57.4, C58.1, C58.3, C59.1, C59.3, C61.-, C64.2, C66.-, C67.2, C68.-, C69.-, C70.2, C71.2, IC10.5, IC11.2, IC11.5, IC12.2, IC2.2, IC3.4, IC4.20, IC4.25, IC4.35, IC4.40, IC4.55, IC4.59, IC4.7, IC4.HT, IC5.10, IC5.15, IC5.16, IC6.10, IC6.15, IC6.16, IC7.2, R11.1, R12.1, R17.1, R18.1, R25.1, R26.1, R29.1, R31.1, R33.2, R34.1, R35.1; no longer C20.2, C21.2, C22.2, C25.2, C26.2, C28.1, C32.1, C34.1, C34.3, C35.2, C35.4, C36.1, C36.3, C37.3, C38.-, C39.2, C41.1, C43.2, C47.1, C49.1, C49.3, C50.4, C51.3, C52.1, C52.3, C54.-, C55.1, C56.2, C57.-, C58.-, C59.2, C60.2, C61.2, C64.-, C66.2, IC2.20, IC2.25, IC2.35, IC2.40, IC2.55, IC2.59, IC2.7, IC2.HT, IC3.1, IC3.10, IC3.2, IC3.21, IC3.22, IC3.23, IC3.25, IC3.26, IC3.27, IC3.29, IC3.3, IC3.30, IC3.9, IC3.HT, IC3.HT1, IC3.HT2, IC3.HT3, IC3.HT4, IC4.2, IC4.5, IC7.5, IC8.5, R22.1, R23.1, R24.1, R28.1, R8.1, R9.1
- net I2C_SCL: now also IC10.1, IC5.23, IC6.23, R28.1, R29.2; no longer IC3.4, IC7.1, R25.1
- net I2C_SDA: now also IC10.2, IC5.22, IC6.22, R30.1, R31.2; no longer IC3.5, IC7.2, R26.1
- net I2S_DATA: now also IC5.11, IC6.11, R8.1; no longer R11.2, R14.1
- net I2S_LRCLK: now also IC5.14, IC6.14, R10.1; no longer R10.2, R13.1
- net I2S_SCK: now also IC5.13, IC6.13, R9.1; no longer R12.2, R15.1
- net LED0: now also IC4.2; no longer IC2.2
- net LED1: now also IC4.3; no longer IC2.3
- net MCLK: now also IC4.22; no longer IC2.22
- net MCLR: now also IC4.9; no longer IC2.9
- net N$10: now also C25.2, IC5.24; no longer IC3.6, R13.2
- net N$11: now also C20.2, IC5.1; no longer IC3.7, R14.2
- net N$12: now also IC5.19, R17.2; no longer C18.2, IC3.31
- net N$13: now also C23.1, IC5.7; no longer C16.2, IC3.40
- net N$14: now also IC5.6, R15.1; no longer IC3.8, R15.2
- net N$15: now also C41.1, IC7.4; no longer C39.1, IC5.4
- net N$16: now also R23.1; no longer R18.1
- net N$17: now also IC5.5, R13.2; no longer C17.1, IC3.11
- net N$18: now also C21.1, IC6.4; no longer C19.1, IC3.20
- net N$19: now also C33.1, IC7.1, IC7.3; no longer C30.1, IC5.1, IC5.3
- net N$20: now also C55.2, C60.2, IC9.1, R24.1, R25.2; no longer C46.2, C53.2, IC6.1, R21.1, R22.2
- net N$21: now also C39.2, C39.4, R19.2; no longer C34.2, C34.4, R16.2
- net N$22: now also C40.1, C40.3, R20.1; no longer C35.1, C35.3, R17.1
- net N$23: now also C55.1, IC9.3; no longer C46.1, IC6.3
- net N$24: now also C22.2, IC6.1; no longer C31.1, FB4.2, IC4.1, IC4.4
- net N$30: now also C56.2, C56.4, R21.2; no longer C49.2, C49.4, R19.2
- net N$31: now also C57.1, C57.3, R22.1; no longer C50.1, C50.3, R20.1
- net N$36: now also R26.2; no longer R23.2
- net N$5: now also C17.1, IC4.31; no longer C14.1, IC2.31
- net N$7: now also C18.1, IC4.32; no longer C15.1, IC2.32
- net N$72: now also C67.1, IC10.11, R27.2; no longer C61.1, IC7.11, R24.2
- net PGEC: now also IC4.15; no longer IC2.15
- net PGED: now also IC4.16; no longer IC2.16
- net PIC_COM1: now also IC10.12, IC4.62; no longer IC2.62, IC7.12
- net PIC_COM2: now also IC10.13, IC4.64; no longer IC2.64, IC7.13
- net PIC_COM3: now also IC10.14, IC4.63; no longer IC2.63, IC7.14
- net SP_OUTN_L: now also C35.2, C37.2, C43.2, C43.4, R19.1; no longer C28.2, C32.2, C36.2, C36.4, R16.1
- net SP_OUTN_R: now also C52.1, C54.1, C59.2, C59.4, FB8.2, L2.4, R22.2, TP3.1; no longer C44.2, C47.2, C51.2, C51.4, FB7.1, L2.1, R19.1, TP4.1
- net SP_OUTP_L: now also C36.1, C38.1, C44.2, C44.4, R20.2; no longer C29.1, C33.1, C37.2, C37.4, R17.2
- net SP_OUTP_R: now also C51.2, C53.2, C58.2, C58.4, FB7.1, L2.1, R21.1, TP4.1; no longer C45.1, C48.1, C52.2, C52.4, FB8.2, L2.4, R20.2, TP3.1
- net STM_IO16: now also IC10.16; no longer IC7.16
- net STM_IO17: now also IC10.17; no longer IC7.17
- net STM_IO20: now also IC10.20; no longer IC7.20
- net STM_TX: now also IC10.9; no longer IC7.9
- net SWCLK: now also IC10.19; no longer IC7.19
- net SWDIO: now also IC10.18; no longer IC7.18
- net UART_TX: now also IC4.1; no longer IC2.1
- net USB_D+: now also IC4.37; no longer IC2.37
- net USB_D-: now also IC4.36; no longer IC2.36
- net USB_VBUS: now also IC4.33; no longer IC2.33
- net V+: now also C65.1, C66.+, C68.+, IC11.1, IC11.4; no longer C60.1, C62.+, C63.+, FB4.1, IC8.1, IC8.4
- net XVCC: now also C4.1, C7.1; no longer C3.1, C5.1
Routing:
- net AMP_SDZ: track 0.00 -> 87.1 mm, vias 0 -> 4
- net V+: track 68.9 -> 11.0 mm
- net +5V: track 98.5 -> 146.7 mm, vias 0 -> 5
- net I2C_SCL: track 51.4 -> 95.9 mm, vias 2 -> 4
- net I2C_SDA: track 51.9 -> 91.3 mm, vias 2 -> 3
- net I2S_DATA: track 35.7 -> 73.4 mm, vias 0 -> 2
- net I2S_LRCLK: track 36.7 -> 73.1 mm, vias 0 -> 2
- net I2S_SCK: track 39.8 -> 70.0 mm
- net AMP_AVDD_R: track 0.00 -> 16.5 mm
- net AMP_AVDD_L: track 0.00 -> 16.4 mm
- net AMP_AVDD: track 15.1 -> 0.00 mm
- net AMP_DVDD: track 12.9 -> 0.00 mm
- net +1V8: track 0.00 -> 12.3 mm, vias 0 -> 2
- net I2S_SCK_PIC: track 0.00 -> 9.87 mm
- net GND: track 39.1 -> 29.3 mm, vias 366 -> 420
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Other:
- board size 80 x 72 mm -> 90 x 72 mm
- board text added: "USB Audio Amp ver3"
- board text removed: "USB Audio Amp"
- board text removed: "ver2"

Commit message: 修正
Parts:
- IC12: value 3.3V -> 2.5V
- R28, R30, R32: value 10k -> 5.1k
Connections:
- net +3V3 renamed +2V5
Changed lines of the file:
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@@
 <attribute name="VALUE" x="88.71" y="42.56" size="0.8128" layer="27" font="vector" ratio="15" rot="R270"/>
 </element>
-<element name="R28" library="my_rcl" package="1608" value="10k" x="76" y="40" smashed="yes" rot="R90">
+<element name="R28" library="my_rcl" package="1608" value="5.1k" x="76" y="40" smashed="yes" rot="R90">
 <attribute name="NAME" x="75" y="38.4" size="0.8128" layer="25" rot="R90"/>
 <attribute name="VALUE" x="70.2" y="37.85" size="0.8128" layer="27" font="vector" ratio="15" rot="R270"/>
 </element>
-<element name="R30" library="my_rcl" package="1608" value="10k" x="74" y="40" smashed="yes" rot="R90">
+<element name="R30" library="my_rcl" package="1608" value="5.1k" x="74" y="40" smashed="yes" rot="R90">
 <attribute name="NAME" x="73" y="38.4" size="0.8128" layer="25" rot="R90"/>
 <attribute name="VALUE" x="69.2" y="37.85" size="0.8128" layer="27" font="vector" ratio="15" rot="R270"/>
@@
 <attribute name="VALUE" x="74.6145" y="57.187" size="0.8128" layer="27" font="vector" ratio="15" rot="R180"/>
 </element>
-<element name="IC12" library="my_ic" package="SOT23-5" value="3.3V" x="70.5" y="44.5" smashed="yes" rot="R180">
+<element name="IC12" library="my_ic" package="SOT23-5" value="2.5V" x="70.5" y="44.5" smashed="yes" rot="R180">
 <attribute name="NAME" x="72.405" y="41.96" size="0.8128" layer="25" rot="R180"/>
 <attribute name="VALUE" x="71.655" y="47.6115" size="0.8128" layer="27" font="vector" ratio="15" rot="R180"/>
@@
 <attribute name="VALUE" x="66.7" y="37.85" size="0.8128" layer="27" font="vector" ratio="15" rot="R270"/>
 </element>
-<element name="R32" library="my_rcl" package="1608" value="10k" x="77" y="37" smashed="yes" rot="R180">
+<element name="R32" library="my_rcl" package="1608" value="5.1k" x="77" y="37" smashed="yes" rot="R180">
 <attribute name="NAME" x="78.6" y="36" size="0.8128" layer="25" rot="R180"/>
 <attribute name="VALUE" x="77.85" y="36.05" size="0.8128" layer="27" font="vector" ratio="15" rot="R180"/>
@@
 <wire x1="10" y1="26.3" x2="9.8" y2="26.5" width="1.016" layer="16"/>
 </signal>
-<signal name="+3V3">
+<signal name="+2V5">
 <contactref element="IC10" pad="4"/>
 <contactref element="CON4" pad="1"/>
