File: USB_Amp.sch (EAGLE design)
At the start: 149 parts, among them CON1 USB-C, CON2 PIC32_CON, CON4 VOLUEME, CON5 SWD, IC1 3.3V, IC10 +12V, IC16 STM32G031F, IC2 PIC32MZEF, IC3 TAS2780, IC4 TAS2780, IC5 1.8V, IC6 1.8V, IC7 +5V, IC8 +5V, IC9 +12V, X1 24.576MHz, X2 22.5792MHz, X3 12MHz

Commit message: 発注
Parts:
- removed CON5: SWD, my_connector:SWD_CON
- removed FB6: FB2012-FB, my_rcl:FB2012-FB
- removed IC16: STM32G031F, my_ic:STM32G031F
- removed R14, R29: 1k, my_rcl:R-1608
- removed TP12: IO13, my_connector:TESTPIN
- removed TP13, TP14: GND, my_connector:TESTPIN
- removed TP17: +3V3, my_connector:TESTPIN
- added C69: 10p, my_rcl:C-1608
- added C70: 10u, my_rcl:C-3216
- added C71: 10u, my_rcl:C-2012
- added C72, C73, C78: 0.1u, my_rcl:C-1608
- added C74: DNP, my_rcl:C-1608
- added C75, C76: 1000u, my_rcl:CPOLE5-10
- added C77: 470u, my_rcl:CPOLE5-10
- added C79: 22u, my_rcl:C-2012
- added C80, C84: 0.47uF, my_rcl:C-5
- added C81, C85: 0.47uF, my_rcl:C-3225-3
- added C82, C83, C86, C87: 1n, my_rcl:C-1608-2
- added C88: 22u, my_rcl:C-3225
- added CON3: VOLUEME, my_connector:VOL_CON
- added D3: LED1, my_rcl:LED-SMD1608
- added DR1, DR2, DR3, DR4: HOLE-3.2, my_connector:HOLE-3.2
- added IC11: STM32G031F, my_ic:STM32G031F
- added IC12: +5V, my_ic:78X-3
- added IC13: 3.3V, my_ic:TLV740
- added JP1: IO, my_connector:PINHD-1X5
- added R39: SCK, my_rcl:R-1608J
- added R40, R41, R42, R49: 1k, my_rcl:R-1608
- added R43: DNP, my_rcl:R-1608
- added R44: 100k, my_rcl:R-1608
- added R45, R46, R47, R48: 10k, my_rcl:R-1608
- added TP7, TP8: G, my_connector:TESTPIN
- C1, C42: value 0.1u -> 10u; device my_rcl:C-1608 -> my_rcl:C-2012
- C12: value 0.1u -> 22p
- C14: value 22p -> 0.47uF; device my_rcl:C-1608 -> my_rcl:C-3225-3
- C15, C17: value 0.1u -> 10n; device my_rcl:C-1608 -> my_rcl:C-3216-3
- C16, C43: value 0.1u -> 0.47uF; device my_rcl:C-1608 -> my_rcl:C-5
- C18: value 1u -> 470p
- C19, C39: value (none) -> 10u; device my_rcl:C-5 -> my_rcl:C-3216
- C2, C36: value 0.1u -> 1u
- C20: value 10n -> 10u; device my_rcl:C-2012 -> my_rcl:C-3216
- C21: value 10n -> 3.3n; device my_rcl:C-2012 -> my_rcl:C-1608
- C22, C23: value 0.1u -> 470u; device my_rcl:C-1608 -> my_rcl:CPOLE5-10
- C24: value 3.3n -> 10p
- C25: value 470p -> 0.1u
- C26, C29: value 10p -> 0.1u
- C27: value 3.3n -> 1u
- C28: value 470p -> 1u
- C3, C38: value 1u -> 10u; device my_rcl:C-1608 -> my_rcl:C-2012
- C30: value 10u -> 0.1u; device my_rcl:C-2012 -> my_rcl:C-1608
- C33: value 0.1u -> 470p
- C34: value 0.1u -> 10n
- C37: value 0.1u -> 3.3n
- C40: value 10n -> 0.1u; device my_rcl:C-2012 -> my_rcl:C-1608
- C41: value 10n -> 10p; device my_rcl:C-2012 -> my_rcl:C-1608
- C44: value 3.3n -> 10n; device my_rcl:C-1608 -> my_rcl:C-3216-3
- C45: value 470p -> 0.47uF; device my_rcl:C-1608 -> my_rcl:C-3225-3
- C46: value 10p -> 10n; device my_rcl:C-1608 -> my_rcl:C-3216-3
- C47: value 3.3n -> 470p
- C48: value 470p -> 10u; device my_rcl:C-1608 -> my_rcl:C-3216
- C49: value 10p -> 10u; device my_rcl:C-1608 -> my_rcl:C-3216
- C5: value 22u -> 0.1u; device my_rcl:C-2012 -> my_rcl:C-1608
- C50: value 10u -> 3.3n; device my_rcl:C-2012 -> my_rcl:C-1608
- C51, C52: value 10u -> 470u; device my_rcl:C-2012 -> my_rcl:CPOLE5-10
- C53: value DNP -> 10p
- C54: value 1u -> 0.1u
- C55, C58, C59: value 10u -> 0.1u; device my_rcl:C-3216 -> my_rcl:C-1608
- C57: value 10u -> 1u; device my_rcl:C-3216 -> my_rcl:C-1608
- C60, C61: device my_rcl:C-3216 -> my_rcl:C-2012
- C62: value 470u -> 470p; device my_rcl:CPOLE5-10 -> my_rcl:C-1608
- C63: value 470u -> 10n; device my_rcl:CPOLE5-10 -> my_rcl:C-1608
- C64, C68: value 100u -> 0.1u; device my_rcl:CPOLE5-10 -> my_rcl:C-1608
- C65: value 100u -> 3.3n; device my_rcl:CPOLE5-10 -> my_rcl:C-1608
- C66: value 10u -> 1u; device my_rcl:C-2012 -> my_rcl:C-1608
- CON4: value VOLUEME -> SWD; device my_connector:VOL_CON -> my_connector:SWD_CON
- D1: value LED0 -> SBD-E; device my_rcl:LED-SMD1608 -> my_rcl:SBD-E
- D2: value LED1 -> LED0
- D4: value SBD-E -> PWR; device my_rcl:SBD-E -> my_rcl:LED-SMD1608
- FB5: device my_rcl:FB -> my_rcl:FB2012-FB
- IC10: value +12V -> 1.8V; device my_ic:78X-3 -> my_ic:TAR5SB33
- IC3: value TAS2780 -> +12V; device my_ic:TAS2780 -> my_ic:78X-3
- IC4: value TAS2780 -> +5V; device my_ic:TAS2780 -> my_ic:78X-3
- IC5: value 1.8V -> TAS2780; device my_ic:TAR5SB33 -> my_ic:TAS2780
- IC7: value +5V -> +12V
- IC9: value +12V -> TAS2780; device my_ic:78X-3 -> my_ic:TAS2780
- L1, L2, L3, L4: value (none) -> 15uH
- R1: value 1k -> 10k
- R10, R22, R37: value 39 -> LRCLK
- R11: value 10 -> DATA; device my_rcl:R-2012 -> my_rcl:R-1608J
- R12, R24: value 10 -> SCK; device my_rcl:R-2012 -> my_rcl:R-1608J
- R13, R26: value DNP -> 1k
- R16, R31: value 1k -> 10; device my_rcl:R-1608 -> my_rcl:R-2012
- R17: value DNP -> 10; device my_rcl:R-1608 -> my_rcl:R-2012
- R19: value 330 -> 1k
- R2, R4: value 1k -> 5.1k
- R20: value 1k -> DNP
- R21, R36: value 39 -> DATA
- R23, R38: value 39 -> 330; device my_rcl:R-1608J -> my_rcl:R-1608
- R25: value 10 -> 1k; device my_rcl:R-2012 -> my_rcl:R-1608
- R28: value 330 -> DNP
- R3, R9: value 39 -> 10k; device my_rcl:R-1608J -> my_rcl:R-1608
- R30: value DNP -> 330
- R32: value 330 -> 10; device my_rcl:R-1608 -> my_rcl:R-2012
- R34, R7: value 10k -> 1k
- R35: value 10k -> DNP
- R5: value 5.1k -> 10k
- R6: value 5.1k -> 1k
- TP1: value (none) -> L_P
- TP10: value IO14 -> G
- TP2: value (none) -> L_N
- TP3: value (none) -> R_P
- TP4: value (none) -> R_N
- TP5: value (none) -> VIN+
- TP6: value (none) -> VIN-
- TP9: value IO15 -> G
Connections:
- removed net N$38: IC16.IO14, TP10.1
- removed net N$39: IC16.IO16
- removed net N$52: IC16.IO15, TP9.1
- new net PIC_COM1: IC11.IO12, IC2.RE2
- new net PIC_COM2: IC11.IO13, IC2.RE4
- new net PIC_COM3: IC11.IO14, IC2.RE3
- new net STM_IO16: IC11.IO16, JP1.2
- new net STM_IO17: IC11.IO17, JP1.3
- new net STM_IO20: IC11.IO20, JP1.4
- net +3V3: now also C72.1, C79.1, CON3.VCC, D4.A, IC11.VDD, IC13.OUT, JP1.1, R46.2, R47.2; no longer CON4.VCC, IC16.VDD, R34.2, R35.2, TP17.1
- net +3V3D: now also C4.1, C7.1, C88.1, FB2.1, FB3.2, R5.2; no longer C12.1, C5.1, FB5.2, R8.2
- net +5V: now also C28.1, C57.1, C77.1, C78.1, IC10.CONTROL, IC10.VIN, IC12.OUT, IC13.EN, IC13.IN; no longer IC5.CONTROL, IC5.VIN
- net AMP_AVDD_L: now also C35.1, C38.1, C39.1, IC5.AVDD, IC6.VOUT; no longer C22.1, C32.1, C55.1, IC3.AVDD, IC5.VOUT
- net AMP_AVDD_R: now also C64.1, C67.1, C70.1, IC10.VOUT, IC9.ADDR, IC9.AVDD; no longer C42.1, C52.1, C57.1, IC4.ADDR, IC4.AVDD, IC6.VOUT
- net AMP_IOVDD_L: now also C40.1, C42.1, FB3.1, IC5.IOVDD; no longer C23.1, C66.1, FB4.1, IC3.IOVDD
- net AMP_IOVDD_R: now also C68.1, C71.1, FB4.1, IC9.IOVDD; no longer C43.1, C67.1, FB5.1, IC4.IOVDD
- net AMP_OUTN_L: now also C26.1, IC5.OUT_N, R26.2, R28.1; no longer C6.1, IC3.OUT_N, R17.1, R18.2
- net AMP_OUTN_R: now also C55.1, IC9.OUT_N, R41.2, R43.1; no longer C33.1, IC4.OUT_N, R30.1, R31.2
- net AMP_OUTP_L: now also C25.2, IC5.OUT_P, R19.2, R20.1; no longer C7.2, IC3.OUT_P, R13.1, R14.2
- net AMP_OUTP_R: now also C54.2, IC9.OUT_P, R34.2, R35.1; no longer C34.2, IC4.OUT_P, R26.1, R27.2
- net AMP_SDZ: now also IC5.SDZ, IC9.SDZ, R49.1; no longer IC16.IO3, IC3.SDZ, IC4.SDZ
- net AMP_SNS_N_L: now also C37.2, C41.1, IC5.VSNS_N, R25.2, R28.2; no longer C27.2, C29.1, IC3.VSNS_N, R17.2, R20.2
- net AMP_SNS_N_R: now also C65.2, C69.1, IC9.VSNS_N, R40.2, R43.2; no longer C47.2, C49.1, IC4.VSNS_N, R30.2, R33.2
- net AMP_SNS_P_L: now also C21.2, C24.1, IC5.VSNS_P, R18.2, R20.2; no longer C24.2, C26.1, IC3.VSNS_P, R13.2, R16.2
- net AMP_SNS_P_R: now also C50.2, C53.1, IC9.VSNS_P, R33.2, R35.2; no longer C44.2, C46.1, IC4.VSNS_P, R26.2, R29.2
- net AMP_VDD_1S_L: now also C20.1, C23.1, C30.1, C32.1, IC4.OUT, IC5.VBAT1S; no longer C16.1, C31.1, C58.1, C65.1, IC3.VBAT1S, IC7.OUT
- net AMP_VDD_1S_R: now also C49.1, C52.1, C61.1, IC9.VBAT1S; no longer C36.1, C51.1, C63.1, IC4.VBAT1S
- net AMP_VDD_L: now also C19.1, C22.1, C29.1, C31.1, IC3.OUT, IC5.PVDD, R27.2; no longer C17.1, C30.1, C60.1, C64.1, FB2.2, IC3.PVDD, IC9.OUT
- net AMP_VDD_R: now also C48.1, C51.1, C58.1, C60.1, IC7.OUT, IC9.PVDD, R42.2; no longer C37.1, C50.1, C61.1, C62.1, FB3.2, IC10.OUT, IC4.PVDD
- net EN_44.1K: now also R9.2
- net EN_48K: now also R8.2
- net EN_DDC: now also IC11.IO8, R1.1, R3.2; no longer IC16.IO20, R7.1
- net GND: now also C15.1, C16.1, C19.2, C20.2, C24.2, C27.2, C28.2, C34.2, C39.2, C40.2, C43.1, C44.1, C45.2, C48.2, C6.2, C69.2, C7.2, C70.2, C71.2, C72.2, C73.2, C74.2, C75.2, C76.2, C77.2, C78.2, C79.2, C80.1, C81.2, C82.2, C83.1, C84.1, C85.2, C86.2, C87.1, C88.2, CON3.GND, D3.K, IC11.VSS, IC12.GND, IC13.GND, IC3.GND, IC4.GND, IC5.ADDR, IC5.DGND, IC5.GND@1, IC5.PGND@1, IC9.DGND, IC9.GND@1, IC9.PGND@1, JP1.5, R2.1, R3.1, R4.1, R44.1, R45.1, R48.1, R8.1, R9.1, TP10.1, TP7.1, TP8.1, TP9.1; no longer C15.2, C16.2, C18.2, C20.1, C21.2, C26.2, C37.2, C40.1, C43.2, C50.2, C54.2, C55.2, C62.2, C65.2, CON5.GND, D1.K, IC16.VSS, IC3.ADDR, IC3.DGND, IC3.GND@1, IC3.PGND@1, IC4.DGND, IC4.GND@1, IC4.PGND@1, IC5.GND, IC9.GND, R5.1, R6.1, TP13.1, TP14.1
- net I2C_SCL: now also IC11.IO1, IC5.SCL, IC9.SCL, R46.1; no longer IC16.IO1, IC3.SCL, IC4.SCL, R34.1
- net I2C_SDA: now also IC11.IO2, IC5.SDA, IC9.SDA, R47.1; no longer IC16.IO2, IC3.SDA, IC4.SDA, R35.1
- net I2S_DATA: now also R11.2, R36.1; no longer R3.1, R37.2
- net I2S_LRCLK: now also R10.2, R37.1; no longer R36.2, R9.1
- net I2S_SCK: now also R12.2, R24.1, R39.1; no longer R10.1, R23.1, R38.2
- net LED0: now also IC2.RE6, R6.2; no longer IC2.RE7, R1.2
- net LED1: now also IC2.RE7, R7.2; no longer IC2.RG6, R2.2
- net MCLR: now also R5.1; no longer R8.1
- net N$1: now also R2.2; no longer R5.2
- net N$10: now also C33.2, C37.1, R26.1; no longer C27.1, C28.2, R18.1
- net N$11: now also C26.2, IC5.BST_N; no longer C6.2, IC3.BST_N
- net N$12: now also C25.1, IC5.BST_P; no longer C7.1, IC3.BST_P
- net N$13: now also C18.2, C21.1, R19.1; no longer C24.1, C25.2, R14.1
- net N$14: now also C34.1, IC5.PVDD_SNS, R27.1; no longer C15.1, FB2.1, IC3.PVDD_SNS
- net N$15: now also C27.1, IC5.DREG; no longer C18.1, IC3.DREG
- net N$16: now also IC5.SDIN, R21.2; no longer IC3.SDIN, R3.2
- net N$17: now also IC5.FSYNC, R22.2; no longer IC3.FSYNC, R9.2
- net N$18: now also IC5.SBLK, R24.2; no longer IC3.SBLK, R10.2
- net N$19: now also C33.1, R23.2; no longer C28.1, R19.2
- net N$2: now also R4.2; no longer R6.2
- net N$20: now also C18.1; no longer C25.1
- net N$21: now also C15.2, R16.2; no longer C20.2, R12.2
- net N$22: now also C17.1, R17.1; no longer C21.1, R11.1
- net N$23: now also C55.2, IC9.BST_N; no longer C33.2, IC4.BST_N
- net N$24: now also C54.1, IC9.BST_P; no longer C34.1, IC4.BST_P
- net N$25: now also C63.1, IC9.PVDD_SNS, R42.1; no longer C35.1, FB3.1, IC4.PVDD_SNS
- net N$26: now also C56.1, IC9.DREG; no longer C38.1, IC4.DREG
- net N$27: now also IC9.SDIN, R36.2; no longer IC4.SDIN, R21.2
- net N$28: now also IC9.FSYNC, R37.2; no longer IC4.FSYNC, R22.2
- net N$29: now also IC9.SBLK, R39.2; no longer IC4.SBLK, R23.2
- net N$30: now also C44.2, R31.2; no longer C40.2, R25.2
- net N$31: now also C46.1, R32.1; no longer C41.1, R24.1
- net N$32: now also C47.2, C50.1, R34.1; no longer C44.1, C45.2, R27.1
- net N$33: now also C47.1, R30.2; no longer C45.1, R28.2
- net N$34: now also C62.2, C65.1, R41.1; no longer C47.1, C48.2, R31.1
- net N$35: now also C62.1, R38.2; no longer C48.1, R32.2
- net N$36: now also D4.K, R48.2; no longer IC16.IO13, TP12.1
- net N$37: now also IC11.IO3, R45.2, R49.2; no longer IC16.IO17
- net N$4: now also D1.A, R1.2; no longer D4.A, R7.2
- net N$40: now also R12.1; no longer R38.1
- net N$41: now also R11.1; no longer R37.1
- net N$42: now also C36.1, IC6.BYPASS; no longer C54.1, IC5.BYPASS
- net N$43: now also R10.1; no longer R36.1
- net N$44: now also C66.1, IC10.BYPASS; no longer C56.1, IC6.BYPASS
- net N$5: now also C12.1; no longer C13.1
- net N$6: now also R13.2; no longer R4.2
- net N$7: now also C13.1, R13.1; no longer C14.1, R4.1
- net N$72: now also C74.1, CON3.VOL, IC11.IO11, R44.2; no longer C53.1, CON4.VOL, IC16.IO7
- net N$8: now also D2.A, R6.1; no longer D1.A, R1.1
- net N$9: now also D3.A, R7.1; no longer D2.A, R2.1
- net NC1: now also IC5.NC@2; no longer IC3.NC@2
- net NC2: now also IC5.NC@3; no longer IC3.NC@3
- net NC3: now also IC9.NC@2; no longer IC4.NC@2
- net NC4: now also IC9.NC@3; no longer IC4.NC@3
- net SP_OUTN_L: now also C80.2, C81.1, C83.2, R16.1, R23.1, R25.1; no longer C19.2, R12.1, R19.1, R20.1
- net SP_OUTN_R: now also C43.2, C45.1, C87.2, R31.1, R38.1, R40.1; no longer C39.2, R25.1, R32.1, R33.1
- net SP_OUTP_L: now also C14.1, C16.2, C82.1, R17.2, R18.1; no longer C19.1, R11.2, R16.1
- net SP_OUTP_R: now also C84.2, C85.1, C86.1, R30.1, R32.2, R33.1; no longer C39.1, R24.2, R28.1, R29.1
- net STM_TX: now also CON4.TX, IC11.IO9; no longer CON5.TX, IC16.IO9
- net SWCLK: now also CON4.SWCLK, IC11.SWCLK; no longer CON5.SWCLK, IC16.SWCLK
- net SWDIO: now also CON4.SWDIO, IC11.SWDIO; no longer CON5.SWDIO, IC16.SWDIO
- net USB_VBUS: now also C1.1, C2.1, D1.K; no longer C3.1, C4.1, D4.K
- net V+: now also C73.1, C75.1, C76.1, FB5.2, IC12.IN, IC3.IN, IC4.IN; no longer C68.1, FB6.2, IC10.IN, IC9.IN
- net VIN+: now also FB5.1; no longer FB6.1
- net XVCC: now also C3.1, C5.1, C6.1, FB2.2; no longer C1.1, C2.1
Other:
- note added: "Controller"
- note added: "Power Input"
- moved on the sheet: C1, C10, C11, C12, C13, C14, C15, C16, C17, C18, C19, C2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

Commit message: 微修正
Parts:
- added C89: 0.1u, my_rcl:C-1608
- C22, C23, C51, C52, C77: device my_rcl:CPOLE5-10 -> my_rcl:CPOLE5-10-DUAL
Connections:
- net +3V3D: now also C89.1, IC2.VBUS3V3
- net GND: now also C89.2
Other:
- moved on the sheet: C10, C11, C7, C8, C9

Commit message: TAS2770
Parts:
- removed C38, C42, C60, C61, C67, C71: 10u, my_rcl:C-2012
- removed C40, C54, C55, C58, C59, C64, C68: 0.1u, my_rcl:C-1608
- removed C41, C53, C69: 10p, my_rcl:C-1608
- removed C47, C62: 470p, my_rcl:C-1608
- removed C49: 10u, my_rcl:C-3216
- removed C50, C65: 3.3n, my_rcl:C-1608
- removed C52: 470u, my_rcl:CPOLE5-10-DUAL
- removed C56: 1u, my_rcl:C-1608
- removed C63: 10n, my_rcl:C-1608
- removed IC4, IC8: +5V, my_ic:78X-3
- removed R23, R30, R38: 330, my_rcl:R-1608
- removed R25, R26, R27, R33, R34, R40, R41, R42: 1k, my_rcl:R-1608
- removed R28, R35, R43: DNP, my_rcl:R-1608
- removed R36: DATA, my_rcl:R-1608J
- removed R37: LRCLK, my_rcl:R-1608J
- removed R39: SCK, my_rcl:R-1608J
- added R14: DATA, my_rcl:R-1608J
- C16, C43, C80, C84: device my_rcl:C-5 -> my_rcl:C-5W
- C18: value 470p -> 0.1u
- C20: value 10u -> 0.1u; device my_rcl:C-3216 -> my_rcl:C-1608
- C21: value 3.3n -> 1u
- C23: value 470u -> 0.1u; device my_rcl:CPOLE5-10-DUAL -> my_rcl:C-1608
- C24: value 10p -> 0.1u
- C29: value 0.1u -> 1u
- C30: value 0.1u -> 10u; device my_rcl:C-1608 -> my_rcl:C-2012
- C31: value 10u -> 0.1u; device my_rcl:C-2012 -> my_rcl:C-1608
- C33: value 470p -> 1u
- C34: value 10n -> 0.1u
- C37: value 3.3n -> 0.1u
- IC5, IC9: value TAS2780 -> TAS2770; device my_ic:TAS2780 -> my_ic:TAS2770
- R15: value 330 -> LRCLK; device my_rcl:R-1608 -> my_rcl:R-1608J
- R18: value 1k -> SCK; device my_rcl:R-1608 -> my_rcl:R-1608J
- R19: value 1k -> ADDR
- R20: value DNP -> ADDR
Connections:
- removed net AMP_VDD_1S_L: C20.1, C23.1, C30.1, C32.1, IC4.OUT, IC5.VBAT1S
- removed net AMP_VDD_1S_R: C49.1, C52.1, C59.1, C61.1, IC8.OUT, IC9.VBAT1S
- removed net N$14 (its old number): C34.1, IC5.PVDD_SNS, R27.1
- removed net N$28: IC9.FSYNC, R37.2
- removed net N$29: IC9.SBLK, R39.2
- removed net N$32: C47.2, C50.1, R34.1
- removed net N$33: C47.1, R30.2
- removed net N$34: C62.2, C65.1, R41.1
- removed net N$35: C62.1, R38.2
- removed net NC1: IC5.NC@2
- removed net NC2: IC5.NC@3
- removed net NC3: IC9.NC@2
- removed net NC4: IC9.NC@3
- new net AMP_PVDD_L: IC5.PVDD
- new net AMP_PVDD_R: IC9.PVDD
- new net N$18: C29.2, IC5.AREG
- net AMP_AVDD_L: now also C20.1; no longer C35.1, C38.1
- net AMP_AVDD_R: now also C37.1; no longer C64.1, C67.1, IC9.ADDR
- net AMP_IOVDD_L: now also C30.1, C31.1; no longer C40.1, C42.1
- net AMP_IOVDD_R: now also C32.1, C34.1; no longer C68.1, C71.1
- net AMP_OUTN_L: no longer R26.2, R28.1
- net AMP_OUTN_R: now also C24.1; no longer C55.1, R41.2, R43.1
- net AMP_OUTP_L: no longer R19.2, R20.1
- net AMP_OUTP_R: now also C18.2; no longer C54.2, R34.2, R35.1
- net AMP_SNS_N_L: no longer C37.2, C41.1, R25.2, R28.2
- net AMP_SNS_N_R: no longer C65.2, C69.1, R40.2, R43.2
- net AMP_SNS_P_L: no longer C21.2, C24.1, R18.2, R20.2
- net AMP_SNS_P_R: no longer C50.2, C53.1, R33.2, R35.2
- net AMP_VDD_L: now also C23.1; no longer C29.1, C31.1, IC5.PVDD, R27.2
- net AMP_VDD_R: now also C35.1; no longer C58.1, C60.1, IC9.PVDD, R42.2
- net GND: now also C21.2, C29.1, C33.1, C37.2, IC5.GND@2, IC5.GND@3, IC5.PGND, IC9.GND@2, IC9.GND@3, IC9.PGND, R19.2, R20.2; no longer C24.2, C29.2, C38.2, C40.2, C41.2, C42.2, C49.2, C52.2, C53.2, C56.2, C58.2, C59.2, C60.2, C61.2, C63.2, C64.2, C67.2, C68.2, C69.2, C71.2, IC4.GND, IC5.ADDR, IC5.DGND, IC5.PGND@1, IC8.GND, IC9.DGND, IC9.PGND@1
- net I2S_DATA: now also R14.1; no longer R36.1
- net I2S_LRCLK: now also R15.1; no longer R37.1
- net I2S_SCK: now also R18.1; no longer R39.1
- net N$10: now also IC9.SDIN, R14.2; no longer C33.2, C37.1, R26.1
- net N$13: now also IC9.SBLK, R18.2; no longer C18.2, C21.1, R19.1
- net N$19: now also IC9.FSYNC, R15.2; no longer C33.1, R23.2
- net N$20: now also C21.1, IC9.DREG; no longer C18.1, R15.2
- net N$23: now also C18.1, IC9.BST_P; no longer C55.2, IC9.BST_N
- net N$24: now also C24.2, IC9.BST_N; no longer C54.1, IC9.BST_P
- net N$25: now also C33.2, IC9.AREG; no longer C63.1, IC9.PVDD_SNS, R42.1
- net N$26: now also IC9.MODE, R19.1; no longer C56.1, IC9.DREG
- net N$27: now also IC5.MODE, R20.1; no longer IC9.SDIN, R36.2
- net SP_OUTN_L: no longer R23.1, R25.1
- net SP_OUTN_R: no longer R38.1, R40.1
- net SP_OUTP_L: no longer R15.1, R18.1
- net SP_OUTP_R: no longer R30.1, R33.1
- net V+: no longer IC4.IN, IC8.IN
Other:
- moved on the sheet: C14, C15, C16, C17, C18, C19, C20, C21, C22, C24, C25, C26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

Commit message: ver2
Parts:
- removed C66: 1u, my_rcl:C-1608
- removed C70: 10u, my_rcl:C-3216
- removed C72, C73, C78, C89: 0.1u, my_rcl:C-1608
- removed C74: DNP, my_rcl:C-1608
- removed C75, C76: 1000u, my_rcl:CPOLE5-10
- removed C77: 470u, my_rcl:CPOLE5-10-DUAL
- removed C79: 22u, my_rcl:C-2012
- removed C80, C84: 0.47uF, my_rcl:C-5W
- removed C81, C85: 0.47uF, my_rcl:C-3225-3
- removed C82, C83, C86, C87: 1n, my_rcl:C-1608-2
- removed C88: 22u, my_rcl:C-3225
- removed IC10: 1.8V, my_ic:TAR5SB33
- removed IC11: STM32G031F, my_ic:STM32G031F
- removed IC12: +5V, my_ic:78X-3
- removed IC13: 3.3V, my_ic:TLV740
- removed R31, R32: 10, my_rcl:R-2012
- removed R44: 100k, my_rcl:R-1608
- removed R45, R46, R47, R48: 10k, my_rcl:R-1608
- removed R49: 1k, my_rcl:R-1608
- removed TP5: VIN+, my_connector:TESTPIN-BIG
- removed TP6: VIN-, my_connector:TESTPIN-BIG
- added C38: 47u, my_rcl:CPOLE2.5-5
- added C40: 10u, my_rcl:C-2012
- added C41, C42, C54, C55: DNP, my_rcl:C-1608-2
- added C47: 100p, my_rcl:C-1608-2
- added C49: 0.1u, my_rcl:C-5W
- added C50: 0.47uF, my_rcl:C-5W
- added C52, C53: 470u, my_rcl:CPOLE5-10
- added C56: 1000u, my_rcl:CPOLE5-13
- added C58, C63: 0.1u, my_rcl:C-1608
- added C59: DNP, my_rcl:C-1608
- added C60, C61: 1000u, my_rcl:CPOLE5-10
- added C62: 220u, my_rcl:CPOLE2.5-8
- added C64: 22u, my_rcl:C-2012
- added CON5: SWD, my_connector:SWD_CON
- added D5: PWR, my_rcl:LED-SMD1608
- added FB6, FB7, FB8: FB, my_rcl:FB2012-FB
- added FB9: FB, my_rcl:FB-3216
- added IC4, IC8: +5V, my_ic:78X-3
- added Q1: NPN, my_ic:NPN2SC3325
- added Q2: NPN, my_ic:NPN-SOT223
- added R23, R25, R26: 10k, my_rcl:R-1608
- C12, C13: value 22p -> 0.1u
- C14: value 0.47uF -> 22p; device my_rcl:C-3225-3 -> my_rcl:C-1608
- C15: value 10n -> 22p; device my_rcl:C-3216-3 -> my_rcl:C-1608
- C16: value 0.47uF -> 0.22u; device my_rcl:C-5W -> my_rcl:C-1608
- C17: value 10n -> 0.22u; device my_rcl:C-3216-3 -> my_rcl:C-1608
- C18: value 0.1u -> 0.22u
- C19: value 10u -> 0.22u; device my_rcl:C-3216 -> my_rcl:C-1608
- C20: value 0.1u -> 10n; device my_rcl:C-1608 -> my_rcl:C-1005
- C21: value 1u -> 10n; device my_rcl:C-1608 -> my_rcl:C-1005
- C22: value 470u -> 0.1u; device my_rcl:CPOLE5-10-DUAL -> my_rcl:C-1608
- C24, C25: device my_rcl:C-1608 -> my_rcl:C-1005
- C26: value 0.1u -> 10u; device my_rcl:C-1608 -> my_rcl:C-2012
- C27: value 1u -> 10u; device my_rcl:C-1608 -> my_rcl:C-2012
- C28, C29, C33: value 1u -> 100p; device my_rcl:C-1608 -> my_rcl:C-1608-2
- C30: value 10u -> 0.1u; device my_rcl:C-2012 -> my_rcl:C-1608
- C32: value 10u -> 100p; device my_rcl:C-2012 -> my_rcl:C-1608-2
- C34, C35: device my_rcl:C-1608 -> my_rcl:C-5W
- C36: value 1u -> 0.47uF; device my_rcl:C-1608 -> my_rcl:C-5W
- C37: value 0.1u -> 0.47uF; device my_rcl:C-1608 -> my_rcl:C-5W
- C39: value 10u -> 0.1u; device my_rcl:C-3216 -> my_rcl:C-1608
- C43: value 0.47uF -> 10u; device my_rcl:C-5W -> my_rcl:C-2012
- C44, C46: value 10n -> 100p; device my_rcl:C-3216-3 -> my_rcl:C-1608-2
- C45: value 0.47uF -> 100p; device my_rcl:C-3225-3 -> my_rcl:C-1608-2
- C48: value 10u -> 0.1u; device my_rcl:C-3216 -> my_rcl:C-5W
- C51: value 470u -> 0.47uF; device my_rcl:CPOLE5-10-DUAL -> my_rcl:C-5W
- C57: value 1u -> 0.1u
- C7: value 0.1u -> 22u; device my_rcl:C-1608 -> my_rcl:C-3225
- CON2: value PIC32_CON -> PROG
- CON3: value VOLUEME -> DC IN; device my_connector:VOL_CON -> my_connector:POWER_CON
- CON4: value SWD -> VOLUEME; device my_connector:SWD_CON -> my_connector:VOL_CON
- D1: value SBD-E -> SBD
- D4: value PWR -> 5.6mA; device my_rcl:LED-SMD1608 -> my_rcl:CRD-SMD
- IC3: value +12V -> SSM3582; device my_ic:78X-3 -> my_ic:SSM3582
- IC5: value TAS2770 -> 1.8V; device my_ic:TAS2770 -> my_ic:NJM12888
- IC6: value 1.8V -> TL431; device my_ic:TAR5SB33 -> my_ic:TL431-SMD
- IC7: value +12V -> STM32G031F; device my_ic:78X-3 -> my_ic:STM32G031F
- IC9: value TAS2770 -> 3.3V; device my_ic:TAS2770 -> my_ic:TLV740
- R13: value 1k -> LRCLK; device my_rcl:R-1608 -> my_rcl:R-1608J
- R15: value LRCLK -> SCK
- R18: value SCK -> 1k; device my_rcl:R-1608J -> my_rcl:R-1608
- R19, R20: value ADDR -> 10; device my_rcl:R-1608 -> my_rcl:R-2012
- R21: value DATA -> 3.6k; device my_rcl:R-1608J -> my_rcl:R-1608
- R22: value LRCLK -> 1k; device my_rcl:R-1608J -> my_rcl:R-1608
- R24: value SCK -> 100k; device my_rcl:R-1608J -> my_rcl:R-1608
Connections:
- removed net AMP_AVDD_L: C20.1, C39.1, IC5.AVDD, IC6.VOUT
- removed net AMP_AVDD_R: C37.1, C70.1, IC10.VOUT, IC9.AVDD
- removed net AMP_IOVDD_L: C30.1, C31.1, FB3.1, IC5.IOVDD
- removed net AMP_IOVDD_R: C32.1, C34.1, FB4.1, IC9.IOVDD
- removed net AMP_PVDD_L: IC5.PVDD
- removed net AMP_PVDD_R: IC9.PVDD
- removed net AMP_SDZ: IC5.SDZ, IC9.SDZ, R49.1
- removed net AMP_SNS_N_L: IC5.VSNS_N
- removed net AMP_SNS_N_R: IC9.VSNS_N
- removed net AMP_SNS_P_L: IC5.VSNS_P
- removed net AMP_SNS_P_R: IC9.VSNS_P
- removed net AMP_VDD_L: C19.1, C22.1, C23.1, IC3.OUT
- removed net AMP_VDD_R: C35.1, C48.1, C51.1, IC7.OUT
- removed net N$25: C33.2, IC9.AREG
- removed net N$26: IC9.MODE, R19.1
- removed net N$27: IC5.MODE, R20.1
- removed net N$37: IC11.IO3, R45.2, R49.2
- removed net N$42: C36.1, IC6.BYPASS
- removed net N$44: C66.1, IC10.BYPASS
- removed net N$6: IC2.OSC2, R13.2
- new net +12V: C20.1, C21.1, C24.1, C25.1, C26.1, C27.1, C52.1, C53.1, C56.1, IC3.PVDD@1, IC3.PVDD@2, IC3.PVDD@3, IC3.PVDD@4, IC3.PVDD@5, IC3.PVDD@6, IC3.PVDD@7, IC3.PVDD@8, Q2.E, R18.2, R21.2
- new net AMP_AVDD: C23.1, C38.1, C40.1, IC3.AVDD, IC4.OUT
- new net AMP_DVDD: C22.1, C43.1, IC3.DVDD, IC5.VOUT
- net +3V3: now also C57.1, C64.1, CON4.VCC, D5.A, IC7.VDD, IC9.OUT, R25.2, R26.2; no longer C72.1, C79.1, CON3.VCC, D4.A, IC11.VDD, IC13.OUT, R46.2, R47.2
- net +3V3D: now also C12.1, C13.1; no longer C88.1, C89.1, FB3.2, FB4.2
- net +5V: now also C62.1, C63.1, FB3.1, IC8.OUT, IC9.EN, IC9.IN; no longer C28.1, C57.1, C77.1, C78.1, IC10.CONTROL, IC10.VIN, IC12.OUT, IC13.EN, IC13.IN, IC6.CONTROL, IC6.VIN
- net AMP_OUTN_L: now also C18.1, C41.2, FB5.2, IC3.OUTL-@1, IC3.OUTL-@2; no longer C26.1, IC5.OUT_N
- net AMP_OUTN_R: now also C19.2, C54.2, FB7.2, IC3.OUTR-@1, IC3.OUTR-@2, L3.1; no longer C24.1, IC9.OUT_N, L3.2
- net AMP_OUTP_L: now also C16.1, C42.1, FB6.1, IC3.OUTL+@1, IC3.OUTL+@2, L2.1; no longer C25.2, IC5.OUT_P, L2.2
- net AMP_OUTP_R: now also C17.2, C55.1, FB8.1, IC3.OUTR+@1, IC3.OUTR+@2; no longer C18.2, IC9.OUT_P
- net EN_DDC: now also IC7.IO8; no longer IC11.IO8
- net GND: now also C15.2, C24.2, C25.2, C26.2, C28.1, C29.2, C32.1, C33.2, C34.1, C36.1, C37.1, C38.2, C40.2, C41.1, C42.2, C43.2, C46.1, C47.2, C48.1, C49.2, C50.1, C51.1, C52.2, C53.2, C54.1, C55.2, C56.2, C58.2, C59.2, C60.2, C61.2, C62.2, C63.2, C64.2, CON3.V-, CON5.GND, IC3.ADDR0, IC3.ADDR1, IC3.AGND, IC3.AVDD_EN, IC3.DVDD_EN, IC3.HT, IC3.PGND@1, IC3.PGND@2, IC3.PGND@3, IC3.PGND@4, IC3.PGND@5, IC3.PGND@6, IC3.PGND@7, IC3.PGND@8, IC4.GND, IC5.GND, IC7.VSS, IC8.GND, IC9.GND, R22.1, R23.1, R24.1; no longer C15.1, C16.1, C17.2, C19.2, C28.2, C29.1, C32.2, C33.1, C34.2, C36.2, C37.2, C43.1, C46.2, C48.2, C51.2, C66.2, C70.2, C72.2, C73.2, C74.2, C75.2, C76.2, C77.2, C78.2, C79.2, C80.1, C81.2, C82.2, C83.1, C84.1, C85.2, C86.2, C87.1, C88.2, C89.2, CON3.GND, IC10.GND, IC11.VSS, IC12.GND, IC13.GND, IC3.GND, IC5.GND@1, IC5.GND@2, IC5.GND@3, IC5.PGND, IC7.GND, IC9.GND@1, IC9.GND@2, IC9.GND@3, IC9.PGND, R19.2, R20.2, R44.1, R45.1, R48.1, TP6.1
- net I2C_SCL: now also IC3.SCL, IC7.IO1, R25.1; no longer IC11.IO1, IC5.SCL, IC9.SCL, R46.1
- net I2C_SDA: now also IC3.SDA, IC7.IO2, R26.1; no longer IC11.IO2, IC5.SDA, IC9.SDA, R47.1
- net I2S_DATA: no longer R21.1
- net I2S_LRCLK: now also R13.1; no longer R15.1, R22.1
- net I2S_SCK: now also R15.1; no longer R18.1, R24.1
- net N$10: now also IC3.FSYNC, R13.2; no longer IC9.SDIN, R14.2
- net N$11: now also IC3.SDATA, R14.2; no longer IC5.SDIN, R21.2
- net N$12: now also C18.2, IC3.BSTL-; no longer IC5.SBLK, R24.2
- net N$13: now also C16.2, IC3.BSTL+; no longer IC9.SBLK, R18.2
- net N$14: now also IC3.BCLK, R15.2; no longer IC5.FSYNC, R22.2
- net N$15: now also C39.1, IC5.BYPASS; no longer C27.1, IC5.DREG
- net N$16: now also Q1.E, Q2.B, R18.1; no longer C25.1, IC5.BST_P
- net N$17: now also C17.1, IC3.BSTR+; no longer C26.2, IC5.BST_N
- net N$18: now also C19.1, IC3.BSTR-; no longer C29.2, IC5.AREG
- net N$19: now also C30.1, FB3.2, IC5.CONTROL, IC5.VIN; no longer IC9.FSYNC, R15.2
- net N$20: now also IC6.REF, R21.1, R22.2; no longer C21.1, IC9.DREG
- net N$21: now also C34.2; no longer C15.2
- net N$22: now also C35.1; no longer C17.1
- net N$23: now also D4.K, IC6.OUT, Q1.B; no longer C18.1, IC9.BST_P
- net N$24: now also C31.1, FB4.2, IC4.IN; no longer C24.2, IC9.BST_N
- net N$30: now also C48.2, R19.2; no longer C44.2, R31.2
- net N$31: now also C49.1, R20.1; no longer C46.1, R32.1
- net N$36: now also D5.K, R23.2; no longer D4.K, R48.2
- net N$5: now also C14.1; no longer C12.1
- net N$7: now also C15.1, IC2.OSC2; no longer C13.1, R13.1
- net N$72: now also C59.1, CON4.VOL, IC7.IO11, R24.2; no longer C74.1, CON3.VOL, IC11.IO11, R44.2
- net PIC_COM1: now also IC7.IO12; no longer IC11.IO12
- net PIC_COM2: now also IC7.IO13; no longer IC11.IO13
- net PIC_COM3: now also IC7.IO14; no longer IC11.IO14
- net SP_OUTN_L: now also C28.2, C32.2, C36.2, FB5.1; no longer C80.2, C81.1, C83.2
- net SP_OUTN_R: now also C44.2, C46.2, C50.2, FB7.1, L3.2, R19.1; no longer C43.2, C45.1, C87.2, L3.1, R31.1
- net SP_OUTP_L: now also C29.1, C33.1, C37.2, FB6.2, L2.2; no longer C14.1, C16.2, C82.1, L2.1
- net SP_OUTP_R: now also C45.1, C47.1, C51.2, FB8.2, R20.2; no longer C84.2, C85.1, C86.1, R32.2
- net STM_IO16: now also IC7.IO16; no longer IC11.IO16
- net STM_IO17: now also IC7.IO17; no longer IC11.IO17
- net STM_IO20: now also IC7.IO20; no longer IC11.IO20
- net STM_TX: now also CON5.TX, IC7.IO9; no longer CON4.TX, IC11.IO9
- net SWCLK: now also CON5.SWCLK, IC7.SWCLK; no longer CON4.SWCLK, IC11.SWCLK
- net SWDIO: now also CON5.SWDIO, IC7.SWDIO; no longer CON4.SWDIO, IC11.SWDIO
- net V+: now also C58.1, C60.1, C61.1, D4.A, FB4.1, FB9.2, IC8.IN, Q1.C, Q2.C; no longer C73.1, C75.1, C76.1, FB5.2, IC12.IN, IC3.IN, IC7.IN
- net VIN+: now also CON3.V+, FB9.1; no longer FB5.1, TP5.1
Other:
- moved on the sheet: C10, C11, C12, C13, C14, C15, C16, C17, C18, C19, C20, C21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

Commit message: インダクタ変更
Parts:
- removed D5: PWR, my_rcl:LED-SMD1608
- removed L3, L4: 15uH, my_rcl:L-5
- added C65: 0.1u, my_rcl:C-1608
- added C66: 22u, my_rcl:C-2012
- added Q3: NPN, my_ic:NPN-SOT223
- added R27, R28: 1k, my_rcl:R-3216-3
- C26, C27: device my_rcl:C-2012 -> my_rcl:C-3225-2
- C46: value 100p -> DNP; device my_rcl:C-1608-2 -> my_rcl:C-1608
- C48: value 0.1u -> 100p; device my_rcl:C-5W -> my_rcl:C-1608-2
- C50: value 0.47uF -> 0.1u
- C52: value 470u -> 0.47uF; device my_rcl:CPOLE5-10 -> my_rcl:C-5W
- C53: value 470u -> DNP; device my_rcl:CPOLE5-10 -> my_rcl:C-1608
- C54: value DNP -> 470u; device my_rcl:C-1608-2 -> my_rcl:CPOLE5-10
- C56: value 1000u -> DNP; device my_rcl:CPOLE5-13 -> my_rcl:C-1608-2
- C57: value 0.1u -> 470u; device my_rcl:C-1608 -> my_rcl:CPOLE5-10
- C58: value 0.1u -> 1000u; device my_rcl:C-1608 -> my_rcl:CPOLE5-13
- C59: value DNP -> 0.1u
- C60: value 1000u -> 0.1u; device my_rcl:CPOLE5-10 -> my_rcl:C-1608
- C61: value 1000u -> DNP; device my_rcl:CPOLE5-10 -> my_rcl:C-1608
- C62: value 220u -> 1000u; device my_rcl:CPOLE2.5-8 -> my_rcl:CPOLE5-10
- C63: value 0.1u -> 1000u; device my_rcl:C-1608 -> my_rcl:CPOLE5-10
- C64: value 22u -> 220u; device my_rcl:C-2012 -> my_rcl:CPOLE2.5-8
- D4: value 5.6mA -> PWR; device my_rcl:CRD-SMD -> my_rcl:LED-SMD1608
- L1, L2: value 15uH -> 10uH; device my_rcl:L-5 -> my_rcl:L-DUAL-CSD1013
- Q1: value NPN -> JFET; device my_ic:NPN2SC3325 -> my_ic:JFET-N
- Q2: device my_ic:NPN-SOT223 -> my_ic:NPN2SC3325
- R16, R17, R19, R20: device my_rcl:R-2012 -> my_rcl:R-3216-3
Connections:
- net +12V: now also C54.1, C57.1, C58.1, Q3.E, R27.2, R28.2; no longer C52.1, C56.1, Q2.E
- net +3V3: now also C59.1, C66.1, D4.A; no longer C57.1, C64.1, D5.A
- net +5V: now also C64.1, C65.1; no longer C62.1, C63.1
- net AMP_OUTN_L: now also L1G$1.1; no longer L1.2
- net AMP_OUTN_R: now also C55.2, L2G$1.2; no longer C54.2, L3.1
- net AMP_OUTP_L: now also L1G$2.2; no longer L2.1
- net AMP_OUTP_R: now also C56.1, L2G$2.1; no longer C55.1, L4.2
- net GND: now also C47.1, C48.2, C49.1, C50.2, C52.1, C54.2, C55.1, C65.2, C66.2, R27.1, R28.1; no longer C46.1, C47.2, C48.1, C49.2, C50.1, C52.2, C53.2, C54.1, C55.2
- net N$16: now also Q2.E, Q3.B; no longer Q1.E, Q2.B
- net N$20: now also C46.2, C53.2
- net N$23: now also C46.1, Q1.G, Q1.S, Q2.B; no longer D4.K, Q1.B
- net N$30: now also C49.2; no longer C48.2
- net N$31: now also C50.1; no longer C49.1
- net N$36: now also D4.K; no longer D5.K
- net N$72: now also C61.1; no longer C59.1
- net SP_OUTN_L: now also L1G$1.2; no longer L1.1
- net SP_OUTN_R: now also C47.2, C51.2, L2G$1.1; no longer C46.2, C50.2, L3.2
- net SP_OUTP_L: now also L1G$2.1; no longer L2.2
- net SP_OUTP_R: now also C48.1, C52.2, L2G$2.2; no longer C47.1, C51.2, L4.1
- net V+: now also C62.1, C63.1, Q1.D, Q3.C; no longer C58.1, C61.1, D4.A, Q1.C
Other:
- moved on the sheet: C46, C47, C48, C49, C50, C51, C55, C59, C62, L2G$1, Q2
