File: USB_Amp.sch (EAGLE design)
At the start: 142 parts, among them CON1 USB-C, CON2 PROG, CON3 DC IN, CON4 VOLUEME, CON5 SWD, IC1 3.3V, IC2 PIC32MZEF, IC3 SSM3582, IC4 +5V, IC5 1.8V, IC6 TL431, IC7 STM32G031F, IC8 +5V, IC9 3.3V, Q1 JFET, Q2 NPN, Q3 NPN, X1 24.576MHz, X2 22.5792MHz, X3 12MHz

Commit message: 発注
Parts:
- added C67: DNP, my_rcl:C-1608
- added C68: 1000u, my_rcl:CPOLE5-10
- added C69: 220u, my_rcl:CPOLE2.5-8
- added C70: 0.1u, my_rcl:C-1608
- added C71: 22u, my_rcl:C-2012
- added IC10: STM32G031F, my_ic:STM32G031F
- added IC11: +5V, my_ic:78X-3
- added IC12: 3.3V, my_ic:TLV740
- added R29, R30, R31, R32, R33: 10k, my_rcl:R-1608
- added R34, R35: 1k, my_rcl:R-3216
- C14, C15: value 22p -> 0.1u
- C16, C19: value 0.22u -> 0.1u
- C17, C18: value 0.22u -> 22p
- C20, C21: value 10n -> 0.1u; device my_rcl:C-1005 -> my_rcl:C-1608
- C23: value 0.1u -> 1u
- C24, C25: value 0.1u -> 1u; device my_rcl:C-1005 -> my_rcl:C-1608
- C26: value 10u -> 1u; device my_rcl:C-3225-2 -> my_rcl:C-1608
- C27: value 10u -> 0.1u; device my_rcl:C-3225-2 -> my_rcl:C-1005
- C28: value 100p -> 0.1u; device my_rcl:C-1608-2 -> my_rcl:C-1005
- C29: value 100p -> 1u
- C3: value 10u -> 0.1u; device my_rcl:C-2012 -> my_rcl:C-1608
- C30: value 0.1u -> 1u; device my_rcl:C-1608 -> my_rcl:C-1608-2
- C31: value 0.1u -> 10u; device my_rcl:C-1608 -> my_rcl:C-3225-3
- C32: value 100p -> 10u; device my_rcl:C-1608-2 -> my_rcl:C-3225-3
- C33: value 100p -> 0.1u; device my_rcl:C-1608-2 -> my_rcl:C-1608
- C34, C49, C50: device my_rcl:C-5W -> my_rcl:C-1608
- C35: value 0.1u -> 100p; device my_rcl:C-5W -> my_rcl:C-1608-2
- C36, C37, C51, C52: value 0.47uF -> 100p; device my_rcl:C-5W -> my_rcl:C-1608-2
- C38: value 47u -> 100p; device my_rcl:CPOLE2.5-5 -> my_rcl:C-1608-2
- C39: device my_rcl:C-1608 -> my_rcl:C-5W2
- C40: value 10u -> 0.1u; device my_rcl:C-2012 -> my_rcl:C-5W2
- C41, C42: value DNP -> 0.1u; device my_rcl:C-1608-2 -> my_rcl:C-1608
- C43: value 10u -> 0.47uF; device my_rcl:C-2012 -> my_rcl:C-5W
- C44: value 100p -> 0.47uF; device my_rcl:C-1608-2 -> my_rcl:C-5W
- C45: value 100p -> 22u; device my_rcl:C-1608-2 -> my_rcl:C-3225
- C46: value DNP -> 22u; device my_rcl:C-1608 -> my_rcl:C-3225
- C47, C48: value 100p -> 10u; device my_rcl:C-1608-2 -> my_rcl:C-2012
- C5, C9: value 0.1u -> 10u; device my_rcl:C-1608 -> my_rcl:C-2012
- C53: value DNP -> 100p; device my_rcl:C-1608 -> my_rcl:C-1608-2
- C54: value 470u -> 100p; device my_rcl:CPOLE5-10 -> my_rcl:C-1608-2
- C55: device my_rcl:C-1608-2 -> my_rcl:C-1608
- C56: value DNP -> 0.1u; device my_rcl:C-1608-2 -> my_rcl:C-5W2
- C57: value 470u -> 0.1u; device my_rcl:CPOLE5-10 -> my_rcl:C-5W2
- C58: value 1000u -> 0.47uF; device my_rcl:CPOLE5-13 -> my_rcl:C-5W
- C59: value 0.1u -> 0.47uF; device my_rcl:C-1608 -> my_rcl:C-5W
- C60: value 0.1u -> DNP
- C61: value DNP -> 470u; device my_rcl:C-1608 -> my_rcl:CPOLE5-10
- C62: value 1000u -> 470u
- C63: device my_rcl:CPOLE5-10 -> my_rcl:CPOLE5-13
- C64: value 220u -> 0.1u; device my_rcl:CPOLE2.5-8 -> my_rcl:C-1608
- C66: value 22u -> 1000u; device my_rcl:C-2012 -> my_rcl:CPOLE5-10
- C7: value 22u -> 0.1u; device my_rcl:C-3225 -> my_rcl:C-1608
- C8: value 0.1u -> 22u; device my_rcl:C-1608 -> my_rcl:C-3225
- IC2: value PIC32MZEF -> 1.8V; device my_ic:PIC32MZEF -> my_ic:TLV740
- IC3: value SSM3582 -> 7WZ07; device my_ic:SSM3582 -> my_ic:TC7WZ07FK
- IC4: value +5V -> PIC32MZEF; device my_ic:78X-3 -> my_ic:PIC32MZEF
- IC5: value 1.8V -> TAS2770; device my_ic:NJM12888 -> my_ic:TAS2770
- IC6: value TL431 -> TAS2770; device my_ic:TL431-SMD -> my_ic:TAS2770
- IC7: value STM32G031F -> 1.8V; device my_ic:STM32G031F -> my_ic:NJM12888
- IC8: value +5V -> 1.8V; device my_ic:78X-3 -> my_ic:NJM12888
- IC9: value 3.3V -> TL431; device my_ic:TLV740 -> my_ic:TL431-SMD
- R11: value DATA -> 10k; device my_rcl:R-1608J -> my_rcl:R-1608
- R12: value SCK -> 10k; device my_rcl:R-1608J -> my_rcl:R-1608
- R13: value LRCLK -> 1k; device my_rcl:R-1608J -> my_rcl:R-1608
- R14: value DATA -> 1k; device my_rcl:R-1608J -> my_rcl:R-1608
- R15: value SCK -> 1k; device my_rcl:R-1608J -> my_rcl:R-1608
- R16: value 10 -> 1k; device my_rcl:R-3216-3 -> my_rcl:R-1608
- R17: value 10 -> ADDR; device my_rcl:R-3216-3 -> my_rcl:R-1608
- R18: value 1k -> ADDR
- R21: value 3.6k -> 10; device my_rcl:R-1608 -> my_rcl:R-3216-3
- R22: value 1k -> 10; device my_rcl:R-1608 -> my_rcl:R-3216-3
- R23, R25: value 10k -> 1k
- R24: value 100k -> 3.6k
- R27: value 1k -> 100k; device my_rcl:R-3216-3 -> my_rcl:R-1608
- R28: value 1k -> 10k; device my_rcl:R-3216-3 -> my_rcl:R-1608
- R8: value 10k -> DATA; device my_rcl:R-1608 -> my_rcl:R-1608J
- R9: value 10k -> SCK; device my_rcl:R-1608 -> my_rcl:R-1608J
- TP3: value R_P -> R_N
- TP4: value R_N -> R_P
Connections:
- removed net AMP_AVDD: C23.1, C38.1, C40.1, IC3.AVDD, IC4.OUT
- removed net AMP_DVDD: C22.1, C43.1, IC3.DVDD, IC5.VOUT
- removed net N$40: IC2.RD1, IC2.T1CK, R12.1
- removed net N$41: IC2.RD2, R11.1
- removed net N$43: IC2.RD4, R10.1
- new net +1V8: C16.1, C9.1, IC2.OUT, IC3G$4.V+
- new net AMP_AVDD_L: C45.1, C47.1, C49.1, IC5.AVDD, IC5.IOVDD, IC7.VOUT
- new net AMP_AVDD_R: C46.1, C48.1, C50.1, IC6.AVDD, IC6.IOVDD, IC8.VOUT
- new net AMP_SDZ: IC5.SDZ, IC6.SDZ, R32.2, R33.1
- new net I2S_DATA_PIC: IC3G$1.IN, IC4.RD2
- new net I2S_LRCLK_PIC: IC3G$2.IN, IC4.RD4
- new net I2S_SCK_PIC: IC3G$3.IN, IC4.RD1, IC4.T1CK
- new net N$25: C26.2, IC6.AREG
- new net N$26: IC6.MODE, R18.2
- new net N$27: C24.1, IC6.DREG
- new net N$28: IC6.VSNS_N, R16.1
- new net N$29: IC6.VSNS_P, R14.2
- new net N$32: IC10.IO3, R32.1
- new net N$33: IC3G$1.OUT, R8.2
- new net N$34: IC3G$3.OUT, R9.2
- new net N$35: IC3G$2.OUT, R10.2
- new net N$37: C42.1, IC8.BYPASS
- new net N$38: C34.1, FB4.2, IC8.CONTROL, IC8.VIN
- new net N$6: C19.1, IC5.BST_P
- net +12V: now also C28.1, C29.1, C30.1, C31.1, C32.1, C60.1, C61.1, C62.1, C63.1, IC5.PVDD, IC6.PVDD, R23.2, R24.2, R34.2, R35.2; no longer C20.1, C21.1, C24.1, C25.1, C26.1, C53.1, C54.1, C57.1, C58.1, IC3.PVDD@1, IC3.PVDD@2, IC3.PVDD@3, IC3.PVDD@4, IC3.PVDD@5, IC3.PVDD@6, IC3.PVDD@7, IC3.PVDD@8, R18.2, R21.2, R27.2, R28.2
- net +3V3: now also C64.1, C71.1, IC10.VDD, IC12.OUT, R28.2, R30.2; no longer C59.1, C66.1, IC7.VDD, IC9.OUT, R25.2, R26.2
- net +3V3D: now also C14.1, C15.1, C5.1, IC4.AVDD, IC4.VBUS3V3, IC4.VDD@1, IC4.VDD@2, IC4.VDD@4, IC4.VDD@5, IC4.VDD@6; no longer C4.1, C7.1, C9.1, IC2.AVDD, IC2.VBUS3V3, IC2.VDD@1, IC2.VDD@2, IC2.VDD@4, IC2.VDD@5, IC2.VDD@6
- net +5V: now also C3.1, C69.1, C70.1, FB4.1, IC11.OUT, IC12.EN, IC12.IN, IC2.EN, IC2.IN; no longer C64.1, C65.1, IC8.OUT, IC9.EN, IC9.IN
- net AMP_OUTN_L: now also C20.1, IC5.OUT_N, R15.2; no longer C18.1, C41.2, IC3.OUTL-@1, IC3.OUTL-@2
- net AMP_OUTN_R: now also C22.1, FB8.1, IC6.OUT_N, L2G$2.1, R16.2; no longer C19.2, C55.2, FB7.2, IC3.OUTR-@1, IC3.OUTR-@2, L2G$1.2
- net AMP_OUTP_L: now also C19.2, IC5.OUT_P, R13.1; no longer C16.1, C42.1, IC3.OUTL+@1, IC3.OUTL+@2
- net AMP_OUTP_R: now also C21.2, FB7.2, IC6.OUT_P, L2G$1.2, R14.1; no longer C17.2, C56.1, FB8.1, IC3.OUTR+@1, IC3.OUTR+@2, L2G$2.1
- net EN_44.1K: now also IC4.RB14, R12.2; no longer IC2.RB14, R9.2
- net EN_48K: now also IC4.RB13, R11.2; no longer IC2.RB13, R8.2
- net EN_DDC: now also IC10.IO8; no longer IC7.IO8
- net GND: now also C16.2, C17.2, C18.2, C25.1, C26.1, C28.2, C32.2, C34.2, C35.1, C36.2, C39.1, C41.2, C43.1, C46.2, C47.2, C49.2, C52.2, C53.1, C56.1, C58.1, C59.1, C67.2, C68.2, C69.2, C70.2, C71.2, IC10.VSS, IC11.GND, IC12.GND, IC2.GND, IC3G$4.V-, IC4.AVSS, IC4.VSS@1, IC4.VSS@2, IC4.VSS@3, IC4.VSS@4, IC4.VSS@5, IC4.VSS@6, IC5.GND@1, IC5.GND@2, IC5.GND@3, IC5.PGND, IC6.GND@1, IC6.GND@2, IC6.GND@3, IC6.PGND, IC7.GND, R11.1, R12.1, R17.1, R18.1, R25.1, R26.1, R29.1, R31.1, R33.2, R34.1, R35.1; no longer C20.2, C21.2, C22.2, C25.2, C26.2, C28.1, C32.1, C34.1, C35.2, C36.1, C39.2, C41.1, C43.2, C47.1, C49.1, C52.1, C55.1, C56.2, C58.2, C59.2, C60.2, IC2.AVSS, IC2.VSS@1, IC2.VSS@2, IC2.VSS@3, IC2.VSS@4, IC2.VSS@5, IC2.VSS@6, IC3.ADDR0, IC3.ADDR1, IC3.AGND, IC3.AVDD_EN, IC3.DVDD_EN, IC3.HT, IC3.PGND@1, IC3.PGND@2, IC3.PGND@3, IC3.PGND@4, IC3.PGND@5, IC3.PGND@6, IC3.PGND@7, IC3.PGND@8, IC4.GND, IC5.GND, IC6.GND, IC7.VSS, R22.1, R23.1, R24.1, R28.1, R8.1, R9.1
- net I2C_SCL: now also IC10.IO1, IC5.SCL, IC6.SCL, R28.1, R29.2; no longer IC3.SCL, IC7.IO1, R25.1
- net I2C_SDA: now also IC10.IO2, IC5.SDA, IC6.SDA, R30.1, R31.2; no longer IC3.SDA, IC7.IO2, R26.1
- net I2S_DATA: now also IC5.SDIN, IC6.SDIN, R8.1; no longer R11.2, R14.1
- net I2S_LRCLK: now also IC5.FSYNC, IC6.FSYNC, R10.1; no longer R10.2, R13.1
- net I2S_SCK: now also IC5.SBLK, IC6.SBLK, R9.1; no longer R12.2, R15.1
- net LED0: now also IC4.RE6; no longer IC2.RE6
- net LED1: now also IC4.RE7; no longer IC2.RE7
- net MCLK: now also IC4.RB9; no longer IC2.RB9
- net MCLR: now also IC4.!MCLR; no longer IC2.!MCLR
- net N$10: now also C25.2, IC5.AREG; no longer IC3.FSYNC, R13.2
- net N$11: now also C20.2, IC5.BST_N; no longer IC3.SDATA, R14.2
- net N$12: now also IC5.MODE, R17.2; no longer C18.2, IC3.BSTL-
- net N$13: now also C23.1, IC5.DREG; no longer C16.2, IC3.BSTL+
- net N$14: now also IC5.VSNS_N, R15.1; no longer IC3.BCLK, R15.2
- net N$15: now also C41.1, IC7.BYPASS; no longer C39.1, IC5.BYPASS
- net N$16: now also R23.1; no longer R18.1
- net N$17: now also IC5.VSNS_P, R13.2; no longer C17.1, IC3.BSTR+
- net N$18: now also C21.1, IC6.BST_P; no longer C19.1, IC3.BSTR-
- net N$19: now also C33.1, IC7.CONTROL, IC7.VIN; no longer C30.1, IC5.CONTROL, IC5.VIN
- net N$20: now also C55.2, C60.2, IC9.REF, R24.1, R25.2; no longer C46.2, C53.2, IC6.REF, R21.1, R22.2
- net N$21: now also C39.2, R19.2; no longer C34.2, R16.2
- net N$22: now also C40.1, R20.1; no longer C35.1, R17.1
- net N$23: now also C55.1, IC9.OUT; no longer C46.1, IC6.OUT
- net N$24: now also C22.2, IC6.BST_N; no longer C31.1, FB4.2, IC4.IN
- net N$30: now also C56.2, R21.2; no longer C49.2, R19.2
- net N$31: now also C57.1, R22.1; no longer C50.1, R20.1
- net N$36: now also R26.2; no longer R23.2
- net N$5: now also C17.1, IC4.OSC1; no longer C14.1, IC2.OSC1
- net N$7: now also C18.1, IC4.OSC2; no longer C15.1, IC2.OSC2
- net N$72: now also C67.1, IC10.IO11, R27.2; no longer C61.1, IC7.IO11, R24.2
- net PGEC: now also IC4.PGEC1; no longer IC2.PGEC1
- net PGED: now also IC4.PGED1; no longer IC2.PGED1
- net PIC_COM1: now also IC10.IO12, IC4.RE2; no longer IC2.RE2, IC7.IO12
- net PIC_COM2: now also IC10.IO13, IC4.RE4; no longer IC2.RE4, IC7.IO13
- net PIC_COM3: now also IC10.IO14, IC4.RE3; no longer IC2.RE3, IC7.IO14
- net SP_OUTN_L: now also C35.2, C37.2, C43.2, R19.1; no longer C28.2, C32.2, C36.2, R16.1
- net SP_OUTN_R: now also C52.1, C54.1, C59.2, FB8.2, L2G$2.2, R22.2, TP3.1; no longer C44.2, C47.2, C51.2, FB7.1, L2G$1.1, R19.1, TP4.1
- net SP_OUTP_L: now also C36.1, C38.1, C44.2, R20.2; no longer C29.1, C33.1, C37.2, R17.2
- net SP_OUTP_R: now also C51.2, C53.2, C58.2, FB7.1, L2G$1.1, R21.1, TP4.1; no longer C45.1, C48.1, C52.2, FB8.2, L2G$2.2, R20.2, TP3.1
- net STM_IO16: now also IC10.IO16; no longer IC7.IO16
- net STM_IO17: now also IC10.IO17; no longer IC7.IO17
- net STM_IO20: now also IC10.IO20; no longer IC7.IO20
- net STM_TX: now also IC10.IO9; no longer IC7.IO9
- net SWCLK: now also IC10.SWCLK; no longer IC7.SWCLK
- net SWDIO: now also IC10.SWDIO; no longer IC7.SWDIO
- net UART_TX: now also IC4.RE5; no longer IC2.RE5
- net USB_D+: now also IC4.D+; no longer IC2.D+
- net USB_D-: now also IC4.D-; no longer IC2.D-
- net USB_VBUS: now also IC4.VBUS; no longer IC2.VBUS
- net V+: now also C65.1, C66.1, C68.1, IC11.IN; no longer C60.1, C62.1, C63.1, FB4.1, IC8.IN
- net XVCC: now also C4.1, C7.1; no longer C3.1, C5.1
Other:
- moved on the sheet: C10, C11, C12, C13, C14, C15, C16, C17, C18, C19, C20, C21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

Commit message: 修正
Parts:
- IC12: value 3.3V -> 2.5V
- R28, R30, R32: value 10k -> 5.1k
Connections:
- net +3V3 renamed +2V5
