File: USB_Amp.sch (EAGLE design)
At the start: 169 parts, among them CON1 USB-C-2OZ, CON2 PROG, CON3 PWR IN, CON5 SWD, CON6 USB-C-2OZ, IC1 3.3V, IC2 PIC32MZEF, IC3 TAS6422, IC4 3.3V, IC5 3.3V, IC6 TL431, IC7 STM32G030F, IC8 7805, IC9 CH221, Q1 NPN, Q2 NPN, Q3 PNP, Q4 PNP, X1 24.576MHz, X3 12MHz

Commit message: MCLK配線修正
Connections:
- net EN_DDC: now also IC7.PA1; no longer IC7.IO8
- net I2C_SCL: now also IC7.PB7/8; no longer IC7.IO1
- net I2C_SDA: now also IC7.PB9; no longer IC7.IO2
- net LED0: now also IC7.PC15; no longer IC7.IO3
- net N$39: now also IC7.PA11; no longer IC7.IO16
- net N$42: now also IC7.PA12; no longer IC7.IO17
- net N$72: now also IC7.PA4; no longer IC7.IO11
- net PIC_COM1: now also IC7.PA8/B0-2; no longer IC7.IO15
- net PIC_COM2: now also IC7.PA7; no longer IC7.IO14
- net PIC_COM3: now also IC7.PA6; no longer IC7.IO13
- net PIC_MCLK: now also IC2.RF1; no longer IC2.RE0
- net STM_TX: now also IC7.PA2; no longer IC7.IO9
Changed lines of the file:
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@@
 <net name="I2C_SCL" class="0">
 <segment>
-<pinref part="IC7" gate="G$1" pin="IO1"/>
+<pinref part="IC7" gate="G$1" pin="PB7/8"/>
 <wire x1="523.24" y1="66.04" x2="515.62" y2="66.04" width="0.1524" layer="91"/>
 <label x="513.08" y="66.04" size="1.27" layer="95" rot="R180" xref="yes"/>
@@
 <net name="I2C_SDA" class="0">
 <segment>
-<pinref part="IC7" gate="G$1" pin="IO2"/>
+<pinref part="IC7" gate="G$1" pin="PB9"/>
 <wire x1="523.24" y1="63.5" x2="520.7" y2="63.5" width="0.1524" layer="91"/>
 <label x="513.08" y="63.5" size="1.27" layer="95" rot="R180" xref="yes"/>
@@
 <pinref part="CON5" gate="G$1" pin="TX"/>
 <wire x1="574.04" y1="53.34" x2="586.74" y2="53.34" width="0.1524" layer="91"/>
-<pinref part="IC7" gate="G$1" pin="IO9"/>
+<pinref part="IC7" gate="G$1" pin="PA2"/>
 <wire x1="523.24" y1="45.72" x2="520.7" y2="45.72" width="0.1524" layer="91"/>
 <wire x1="520.7" y1="45.72" x2="520.7" y2="33.02" width="0.1524" layer="91"/>
@@
 <wire x1="515.62" y1="35.56" x2="556.26" y2="35.56" width="0.1524" layer="91"/>
 <wire x1="556.26" y1="35.56" x2="556.26" y2="43.18" width="0.1524" layer="91"/>
-<pinref part="IC7" gate="G$1" pin="IO11"/>
+<pinref part="IC7" gate="G$1" pin="PA4"/>
 <wire x1="556.26" y1="43.18" x2="553.72" y2="43.18" width="0.1524" layer="91"/>
 <pinref part="R24" gate="G$1" pin="2"/>
@@
 <net name="EN_DDC" class="0">
 <segment>
-<pinref part="IC7" gate="G$1" pin="IO8"/>
+<pinref part="IC7" gate="G$1" pin="PA1"/>
 <wire x1="523.24" y1="48.26" x2="520.7" y2="48.26" width="0.1524" layer="91"/>
 <label x="520.7" y="48.26" size="1.27" layer="95" rot="R180" xref="yes"/>
@@
 </segment>
 <segment>
-<pinref part="IC7" gate="G$1" pin="IO15"/>
+<pinref part="IC7" gate="G$1" pin="PA8/B0-2"/>
 <wire x1="553.72" y1="53.34" x2="556.26" y2="53.34" width="0.1524" layer="91"/>
 <label x="556.26" y="53.34" size="1.27" layer="95" xref="yes"/>
@@
 </segment>
 <segment>
-<pinref part="IC7" gate="G$1" pin="IO13"/>
+<pinref part="IC7" gate="G$1" pin="PA6"/>
 <wire x1="553.72" y1="48.26" x2="556.26" y2="48.26" width="0.1524" layer="91"/>
 <label x="556.26" y="48.26" size="1.27" layer="95" xref="yes"/>
@@
 </segment>
 <segment>
-<pinref part="IC7" gate="G$1" pin="IO14"/>
+<pinref part="IC7" gate="G$1" pin="PA7"/>
 <wire x1="553.72" y1="50.8" x2="556.26" y2="50.8" width="0.1524" layer="91"/>
 <label x="556.26" y="50.8" size="1.27" layer="95" xref="yes"/>
@@
 </segment>
 <segment>
-<pinref part="IC2" gate="G$1" pin="RE0"/>
-<wire x1="93.98" y1="132.08" x2="93.98" y2="134.62" width="0.1524" layer="91"/>
-<label x="93.98" y="134.62" size="1.27" layer="95" rot="R90" xref="yes"/>
+<wire x1="96.52" y1="132.08" x2="96.52" y2="134.62" width="0.1524" layer="91"/>
+<label x="96.52" y="134.62" size="1.27" layer="95" rot="R90" xref="yes"/>
+<pinref part="IC2" gate="G$1" pin="RF1"/>
 </segment>
 </net>
@@
 <segment>
 <pinref part="R35" gate="G$1" pin="2"/>
-<pinref part="IC7" gate="G$1" pin="IO16"/>
+<pinref part="IC7" gate="G$1" pin="PA11"/>
 <wire x1="556.26" y1="55.88" x2="553.72" y2="55.88" width="0.1524" layer="91"/>
 </segment>
@@
 <segment>
 <pinref part="R34" gate="G$1" pin="2"/>
-<pinref part="IC7" gate="G$1" pin="IO17"/>
+<pinref part="IC7" gate="G$1" pin="PA12"/>
 <wire x1="556.26" y1="58.42" x2="553.72" y2="58.42" width="0.1524" layer="91"/>
 </segment>
@@
 <net name="LED0" class="0">
 <segment>
-<pinref part="IC7" gate="G$1" pin="IO3"/>
+<pinref part="IC7" gate="G$1" pin="PC15"/>
 <wire x1="523.24" y1="60.96" x2="520.7" y2="60.96" width="0.1524" layer="91"/>
 <label x="520.7" y="60.96" size="1.27" layer="95" rot="R180" xref="yes"/>

Commit message: ver5.1
Parts:
- added R42: 10k, my_rcl:R-1608
- added R43: 1.5k, my_rcl:R-1608
- added TP11, TP6: G, my_connector:TESTPIN
- R18: value 1k -> 360
- R30: value 100k -> 200k
- R38, R39, R40, R41: value 22 -> 10
Connections:
- net N$10 renamed AMP_GVDD
- net N$11 renamed AMP_AVDD
- net N$12 renamed AMP_AVSS
- net N$13 renamed AMP_AREF
- net N$15 renamed AMP_VCOM
- net N$18 renamed AMP_VREG
- new net V+_ADC: IC7.PA5, R42.1, R43.1
- net +3V3: now also R17G$1.3, R17G$2.3; no longer R17G$1.1, R17G$2.1
- net GND: now also R17G$1.1, R17G$2.1, R43.2, TP11.1, TP6.1; no longer R17G$1.3, R17G$2.3
- net V+: now also R42.2
Other:
- moved on the sheet: CON5, R17G$1, R17G$2

Commit message: 微修正
Parts:
- C16, C17, C18, C19: device my_rcl:C-1608 -> my_rcl:C-1608-3
- C24, C25, C26, C40: value 0.1u -> 0.01u; device my_rcl:C-3225-3 -> my_rcl:C-3216-3
- R13, R14, R19, R20: device my_rcl:R-3216-3 -> my_rcl:R-2012-2
Connections:
- net +3V3D: now also IC2.VUSB3V3; no longer IC2.VBUS3V3

Commit message: TAS6424対応
Parts:
- removed D3: LED1, my_rcl:LED-SMD1608
- removed D8: LED2, my_rcl:LED-SMD1608
- removed R11: DATA, my_rcl:R-1005
- removed R12: SCK, my_rcl:R-1005
- removed R36, R37: 3.3k, my_rcl:R-1608
- added C82, C83, C85: 0.1u, my_rcl:C-1608
- added C84: 2.2u, my_rcl:C-1608
- added D1: PLY, my_rcl:LED-SMD1608
- added IC10: ISO7762, my_ic:ISO6762-SSOP
- added Q5: PNP, my_ic:PNP2SA1313
- C14, C15: device my_rcl:C-1608 -> my_rcl:C-1005
- C74, C75: device my_rcl:C-3216 -> my_rcl:C-3225
- D2, D5: device my_rcl:LED-SMD1608 -> my_rcl:LED-2.5
- R10: value LRCLK -> 3.3k; device my_rcl:R-1005 -> my_rcl:R-1608
- R23, R7: value 3.3k -> 1.5k
- R6: value 10k -> 100; device my_rcl:R-1608 -> my_rcl:R-ARRAY
Connections:
- removed net EN_DDC: IC1.EN, IC7.PA1, R6.1
- removed net LED2: IC2.RD11, R37.2
- removed net N$40: IC2.RD1, IC2.T1CK, R12.1
- removed net N$41: IC2.RD2, R11.1
- removed net N$43: IC2.RD4, R10.1
- removed net N$44: D8.A, R37.1
- removed net PIC_COM2: IC2.RD9, IC7.PA7
- removed net PIC_COM3: IC2.RF5, IC7.PA6
- new net AMP_GVDD2: C84.1, IC3.GVDD2
- new net DGND: C1.2, C10.2, C11.2, C12.2, C13.2, C14.2, C15.2, C2.2, C4.2, C6.2, C7.2, C8.2, C82.2, C9.2, CON1.GND, CON1.XT, CON2.GND, D1.K, IC1.GND, IC10.GND1, IC2.AVSS, IC2.VSS@1, IC2.VSS@2, IC2.VSS@3, IC2.VSS@4, IC2.VSS@5, IC2.VSS@6, Q5.C, R2.1, R4.1, TP9.1, X3.GND
- new net I2S_MCLK2: IC10.IN5, R15.2
- new net N$10: IC10.OUT1, R6G$2.1
- new net N$11: IC10.OUT2, R6G$3.1
- new net N$12: IC10.OUT3, R6G$4.1
- new net PIC_DATA: IC10.IN3, IC2.RD2
- new net PIC_DDC_EN: IC10.OUT6, Q5.B
- new net PIC_LRCLK: IC10.IN4, IC2.RD4
- new net PIC_SCK: IC10.IN2, IC2.RD1, IC2.T1CK
- new net STM_COM1: IC10.OUT4, IC7.PA7
- new net STM_DDC_EN: IC10.IN6, IC7.PA8/B0-2
- net +3V3: now also C83.1, IC10.VCC2
- net +3V3D: now also C82.1, IC10.VCC1
- net GND: now also C83.2, C84.2, C85.2, IC10.GND2, IC3.GND@10, IC3.GND@11, R6G$1.1, R6G$1.2; no longer C1.2, C10.2, C11.2, C12.2, C13.2, C14.2, C15.2, C2.2, C4.2, C6.2, C7.2, C8.2, C9.2, CON1.GND, CON1.XT, CON2.GND, D3.K, D8.K, IC1.GND, IC2.AVSS, IC2.VSS@1, IC2.VSS@2, IC2.VSS@3, IC2.VSS@4, IC2.VSS@5, IC2.VSS@6, R2.1, R4.1, R6.2, TP9.1, X3.GND
- net I2S_DATA: now also R6G$3.2; no longer R11.2
- net I2S_LRCLK: now also IC7.PA0, R6G$2.2; no longer R10.2
- net I2S_SCK: now also R6G$4.2; no longer R12.2
- net LED1: now also IC2.RF5, R10.2; no longer IC2.RD0, R36.2
- net MCLR: now also Q5.E
- net N$4: now also IC1.EN
- net N$9: now also D1.A, R10.1; no longer D3.A, R36.1
- net PIC_COM1: now also IC10.IN1; no longer IC7.PA8/B0-2
- net PIC_MCLK: now also IC10.OUT5; no longer R15.2
- net PVDD: now also C85.1, IC3.PVDD@6, IC3.PVDD@7
Other:
- moved on the sheet: C1, C2, C34, C4, C41, C42, C45, C46, C47, FB1, IC1, R1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

Commit message: CH1/4に変更
Parts:
- added C86, C87: 10n, my_rcl:C-1005
- added C88: 4.7u, my_rcl:C-3225
- added C89, C90: 0.1u, my_rcl:C-1608
- added C91: 10u, my_rcl:CPOL2012
- added TP12, TP13: G, my_connector:TESTPIN
- added TP14: GND, my_connector:TESTPIN-MID
- added TP15: PVDD, my_connector:TESTPIN-MID
- C3: value 10u -> 2.2u
- C39: device my_rcl:C-3216 -> my_rcl:CPOL3216
- C62: value 1u -> 0.1u
- C65: value 0.1u -> 10n
- C85: value 0.1u -> 1u; device my_rcl:C-1608 -> my_rcl:C-2012
- CON1: value USB-C-2OZ -> AUDIO_IN
- IC3: value TAS6422 -> TAS6424; device my_ic:TAS6422 -> my_ic:TAS6424
- R15, R9: value 39 -> 51; device my_rcl:R-1608 -> my_rcl:R-1005
Connections:
- removed net AMP_GVDD: C20.1, IC3.GVDD
- removed net AMP_GVDD2: C84.1, IC3.GVDD2
- removed net N$17: C17.2, IC3.BST_2M
- removed net N$19: C16.1, IC3.BST_2P
- new net AMP_GVDD12: C84.1, IC3.GVDD12
- new net AMP_GVDD34: C20.1, IC3.GVDD34
- new net N$13: C17.2, IC3.BST_4M
- new net N$15: C16.1, IC3.BST_4P
- net AMP_OUTN_R: now also IC3.OUT_4M; no longer IC3.OUT_2M
- net AMP_OUTP_R: now also IC3.OUT_4P; no longer IC3.OUT_2P
- net GND: now also C86.2, C87.2, C88.2, C89.2, C90.2, C91.2, R6G$4.1, R6G$4.2, TP12.1, TP13.1, TP14.1; no longer IC3.TEST, R6G$1.1, R6G$1.2
- net I2S_DATA: now also IC3.SDIN1, IC3.SDIN2, R6G$2.2; no longer IC3.SDIN, R6G$3.2
- net I2S_LRCLK: now also R6G$3.2; no longer R6G$2.2
- net I2S_SCK: now also R6G$1.2; no longer R6G$4.2
- net N$10: now also IC10.OUT2, R6G$1.1; no longer IC10.OUT1, R6G$2.1
- net N$11: now also IC10.OUT3, R6G$2.1; no longer IC10.OUT2, R6G$3.1
- net N$12: now also IC10.OUT4, R6G$3.1; no longer IC10.OUT3, R6G$4.1
- net PVDD: now also C86.1, C87.1, C88.1, C89.1, C90.1, TP15.1
- net STM_COM1: now also IC10.OUT1; no longer IC10.OUT4
- net XVCC: now also C91.1
Other:
- moved on the sheet: C16, C17, C42, C45, C46, C48, C49, C50, C55, C57, C58, C60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
