File: USB_Amp.sch (EAGLE design)
At the start: 141 parts, among them CON1 USB-C-2OZ, CON2 PROG, CON3 PWR IN, CON4 VOLUEME, CON5 SWD, CON6 USB-C-2OZ, IC1 3.3V, IC10 AK1110, IC2 PIC32MZEF, IC3 SSM3582, IC4 1.8V, IC5 TAR5SB33, IC6 TL431, IC7 STM32G030F, IC8 7808, IC9 CH221, Q1 NPN, Q2 NPN, X1 24.576MHz, X2 22.5792MHz, X3 12MHz

Commit message: こんな感じ
Parts:
- removed CON4: VOLUEME, my_connector:VOL_CON
- removed D3: LED1, my_rcl:LED-SMD1608
- removed D4: 5.6mA, my_rcl:CRD-SMD
- added C62, C66, C82, C83: 0.1u, my_rcl:C-1608
- added C65: 2.2u, my_rcl:C-2012
- added C67, C68, C72, C73, C77, C78, C79: 0.1u, my_rcl:C-1005
- added C69: 10u, my_rcl:C-2012
- added C70, C71, C74: 10u, my_rcl:CPOL2012
- added C75: 10u, my_rcl:C-3216
- added C76: 1n, my_rcl:C-1608
- added D6: 1mA, my_rcl:CRD-SMD
- added FB3: FB, my_rcl:FB-1608FB
- added IC11: ISO7762, my_ic:ISO6762-SSOP
- added IC12, IC15, IC16: 74LVC1G79, my_ic:74LVC1G79
- added IC13: TC7WU04FU, my_ic:TC7WU04FU
- added IC14: TAR5SB33, my_ic:TAR5SB33
- added Q3, Q4, Q5: PNP, my_ic:PNP2SA1313
- added R34: MCLKB, my_rcl:R-1005
- added R35: 5.1, my_rcl:R-2012H
- added R42: 10k, my_rcl:R-1608
- added R43: 1.5k, my_rcl:R-1608
- added TP5: G, my_connector:TESTPIN
- C14, C15, C63: device my_rcl:C-1608 -> my_rcl:C-1005
- C24, C25: value 0.1u -> 10n
- C26, C27: value 10u -> 1u
- C3: device my_rcl:C-2012 -> my_rcl:C-3225
- C35, C40: device my_rcl:C-3216 -> my_rcl:C-5W2
- C39: value 10u -> 4.7u
- C5: value 0.1u -> 10u; device my_rcl:C-1608 -> my_rcl:C-3225
- C7: value 22u -> 1u; device my_rcl:C-3225 -> my_rcl:C-1608
- CON1: value USB-C-2OZ -> AUDIO_IN
- D1: value SBD -> PLY; device my_rcl:SBD-E -> my_rcl:LED-SMD1608
- D2, D5: device my_rcl:LED-SMD1608 -> my_rcl:LED-2.5
- FB1: value VBUS -> FB; device my_rcl:FB -> my_rcl:FB-1608FB
- FB12: device my_rcl:FB-1608FB -> my_rcl:FB-2012-FB
- FB2: value (none) -> FB; device my_rcl:FB -> my_rcl:FB-1608FB
- IC6: device my_ic:TL431-TO252 -> my_ic:TL431-SC59
- IC8: device my_ic:78X-3 -> my_ic:78X-SOP
- L2: value (none) -> 7uH
- R1: value 10k -> 5.1
- R10: value LRCLK -> 3.3k
- R11: value DATA -> 50k; device my_rcl:R-1608 -> my_rcl:R-VAL2
- R12: value SCK -> MCLK; device my_rcl:R-1608 -> my_rcl:R-1005
- R15: value SCK -> 10k; device my_rcl:R-1005 -> my_rcl:R-1608
- R29: device my_rcl:R-1608 -> my_rcl:R-2012
- R3: value 10k -> 100
- R6: value 1k -> 100; device my_rcl:R-1608 -> my_rcl:R-ARRAY
- R7: value 1k -> 51; device my_rcl:R-1608 -> my_rcl:R-1005
- R8: value 10k -> SCK; device my_rcl:R-1608 -> my_rcl:R-1005
- R9: value 10k -> 51; device my_rcl:R-1608 -> my_rcl:R-1005
- X1: value 24.576MHz -> 22.5792MHz
- X2: value 22.5792MHz -> 24.576MHz
Connections:
- removed net EN_44.1K: IC2.RB14, R9.2, X2.EN
- removed net EN_48K: IC2.RB13, R8.2, X1.EN
- removed net EN_DDC: IC7.PA1, R1.1, R3.2
- removed net MCLK: IC2.RB9, X1.OUT, X2.OUT
- removed net N$72: CON4.VOL, IC7.PA4, R24.2, R28.1
- removed net PIC_COM1: IC2.RE2, IC7.PA5
- removed net PIC_COM2: IC2.RE4, IC7.PA6
- removed net PIC_COM3: IC2.RE3, IC7.PA7
- new net +3V3A: C67.1, C68.1, C69.1, C72.1, C73.1, FB2.2, IC12.VDD, IC13G$4.V+, IC15.VDD, IC16.VDD
- new net DGND: C1.2, C10.2, C11.2, C12.2, C13.2, C14.2, C15.2, C2.2, C4.2, C6.2, C7.2, C8.2, C82.2, C9.2, CON1.GND, CON1.XT, CON2.GND, D1.K, IC1.GND, IC11.GND1, IC2.AVSS, IC2.VSS@1, IC2.VSS@2, IC2.VSS@3, IC2.VSS@4, IC2.VSS@5, IC2.VSS@6, Q5.C, R2.1, R4.1, TP5.1, X3.GND
- new net I2S_DATA_BUF: IC3.SDATA, R13.2
- new net I2S_EN_441K: IC11.OUT1, IC13G$1.IN, IC7.PA12, X1.EN
- new net I2S_EN_48K: IC13G$1.OUT, X2.EN
- new net I2S_LRCLK_BUF: IC3.FSYNC, R14.2
- new net I2S_MCLK: IC12.CP, IC15.CP, IC16.CP, R9.2
- new net I2S_MCLK2: IC13G$3.IN, R7.2
- new net I2S_MCLK_BUF: R12.2, R34.2, R6G$4.2
- new net I2S_SCK_BUF: IC3.BCLK, R8.2
- new net MCLK_OSC: R7.1, R9.1, X1.OUT, X2.OUT
- new net N$22: IC11.OUT3, R6G$2.1
- new net N$24: IC11.OUT4, R6G$3.1
- new net N$25: C38.1, IC6.OUT, Q1.B, Q3.C
- new net N$28: Q3.E, Q4.B, R3.1
- new net N$37: IC13G$2.IN, IC13G$3.OUT, R34.1
- new net N$38: D6.A, Q3.B, Q4.C
- new net N$39: IC13G$2.OUT, R12.1
- new net N$42: FB12.2, R35.1
- new net PIC_DATA: IC11.IN3, IC2.RD2
- new net PIC_DDC_EN: IC11.OUT6, Q5.B
- new net PIC_EN441K: IC11.IN1, IC2.RD10
- new net PIC_LRCLK: IC11.IN4, IC2.RD4
- new net PIC_MCLK: IC11.OUT5, IC2.RF1
- new net PIC_SCK: IC11.IN2, IC2.RD1, IC2.T1CK
- new net STM_DDC_EN: IC11.IN6, IC7.PA11
- new net V+_ADC: IC7.PA5, R42.1, R43.1
- new net VOL_ADC: C76.1, IC7.PA4, R11G$1.2, R11G$2.2, R24.2, R28.1
- net +12V: now also C3.1, C5.1, C63.1, C77.1, C78.1, C79.1
- net +3V3: now also C83.1, IC11.VCC2, R11G$1.3, R11G$2.3; no longer CON4.VCC
- net +3V3D: now also C6.1, C82.1, IC11.VCC1; no longer FB2.1
- net +8V: now also C75.1, FB3.1; no longer C63.1
- net GND: now also C62.2, C65.2, C66.2, C67.2, C68.2, C69.2, C70.2, C71.2, C72.2, C73.2, C74.2, C75.2, C76.2, C77.2, C78.2, C79.2, C83.2, D6.K, IC11.GND2, IC12.VSS, IC13G$4.V-, IC14.GND, IC15.VSS, IC16.VSS, R11G$1.1, R11G$2.1, R15.1, R43.2; no longer C1.2, C10.2, C11.2, C12.2, C13.2, C14.2, C15.2, C2.2, C4.2, C6.2, C7.2, C8.2, C9.2, CON1.GND, CON1.XT, CON2.GND, CON4.GND, D2.K, D3.K, IC1.GND, IC2.AVSS, IC2.VSS@1, IC2.VSS@2, IC2.VSS@3, IC2.VSS@4, IC2.VSS@5, IC2.VSS@6, R2.1, R3.1, R4.1, R8.1, R9.1, X3.GND
- net I2S_DATA: now also IC15.D, R6G$2.2; no longer R11.2, R14.1
- net I2S_LRCLK: now also IC16.D, IC7.PA0, R6G$3.2; no longer R10.2, R13.1
- net I2S_SCK: now also IC12.D, R6G$1.2; no longer R12.2, R15.1
- net LED0: now also D2.A, IC7.PA1; no longer IC2.RE6, R6.2
- net LED1: now also IC2.RF5, R10.2; no longer IC2.RE7, R7.2
- net MCLR: now also Q5.E
- net N$10: now also IC12.Q, R8.1; no longer IC3.FSYNC, R13.2
- net N$11: now also IC15.Q, R13.1; no longer IC3.SDATA, R14.2
- net N$14: now also IC16.Q, R14.1; no longer IC3.BCLK, R15.2
- net N$23: now also C71.1, IC14.BYPASS; no longer C38.1, D4.K, IC6.OUT, Q1.B
- net N$29: now also R35.2; no longer FB12.2
- net N$3: now also FB1.2, R1.1; no longer CON1.VBUS, FB1.1
- net N$31: now also IC9.CC1; no longer IC9.CC2
- net N$32: now also IC9.CC2; no longer IC9.CC1
- net N$4: now also C1.1, C2.1, IC1.IN; no longer D1.A
- net N$40: now also IC11.IN5, R6G$4.1; no longer IC2.RD1, IC2.T1CK, R12.1
- net N$41: now also D2.K, R15.2; no longer IC2.RD2, R11.1
- net N$43: now also C74.1, FB3.2, IC14.CONTROL, IC14.VIN; no longer IC2.RD4, R10.1
- net N$8: now also IC11.OUT2, R6G$1.1; no longer D2.A, R6.1
- net N$9: now also D1.A, R10.1; no longer D3.A, R7.1
- net USB_VBUS: now also CON1.VBUS, FB1.1; no longer C1.1, C2.1, D1.K, FB1.2, IC1.IN
- net V+: now also Q4.E, R3.2, R42.2; no longer D4.A
- net XVCC: now also C62.1, C65.1, C66.1, C70.1, FB2.1, IC14.VOUT; no longer C3.1, C5.1, C6.1, FB2.2
Other:
- moved on the sheet: C1, C10, C11, C12, C13, C14, C15, C2, C21, C24, C25, C26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

Commit message: OK?
Parts:
- removed D6: 1mA, my_rcl:CRD-SMD
- removed R42: 10k, my_rcl:R-1608
- added C80: 0.1u, my_rcl:C-1608
- added C81: 10u, my_rcl:C-3216
- added C84: 4.7u, my_rcl:C-2012
- added D4: LED0, my_rcl:LED-2.5
- added R37: 1k, my_rcl:R-2012
- C13: value 0.1u -> 1u
- C16: value 0.22u -> 10u; device my_rcl:C-1608 -> my_rcl:CPOL2012
- C19: value 0.22u -> 2.2u; device my_rcl:C-1608 -> my_rcl:CPOL2012
- C20: value 10n -> 10u; device my_rcl:C-1005 -> my_rcl:CPOL2012
- C21: value 10n -> 0.22u; device my_rcl:C-1005 -> my_rcl:C-1608
- C22: value 0.1u -> 0.22u
- C23: value 0.1u -> 10u; device my_rcl:C-1608 -> my_rcl:C-2012
- C24: value 10n -> 2.2u; device my_rcl:C-1005 -> my_rcl:C-2012
- C26: value 1u -> 10n; device my_rcl:C-2012 -> my_rcl:C-1005
- C27: value 1u -> 0.1u; device my_rcl:C-2012 -> my_rcl:C-1608
- C28: value 0.47u -> 0.1u; device my_rcl:C-5W -> my_rcl:C-1608
- C29: value 1n -> 10n; device my_rcl:C-2012 -> my_rcl:C-1005
- C3: value 10u -> 0.1u; device my_rcl:C-3225 -> my_rcl:C-1608
- C30: value 10u -> 10n; device my_rcl:C-2012 -> my_rcl:C-1005
- C32: value 100p -> 0.1u
- C33, C41: value 100p -> 0.1u; device my_rcl:C-1608 -> my_rcl:C-1005
- C34, C45: value 1n -> 0.1u; device my_rcl:C-2012 -> my_rcl:C-1005
- C35: value 10n -> 0.1u; device my_rcl:C-5W2 -> my_rcl:C-1005
- C36, C37: value 10u -> 0.1u; device my_rcl:C-2012 -> my_rcl:C-1005
- C38: value DNP -> 0.1u; device my_rcl:C-1608 -> my_rcl:C-1005
- C39: value 4.7u -> 1u; device my_rcl:C-3216 -> my_rcl:C-2012
- C4: value 10u -> 0.1u; device my_rcl:C-2012 -> my_rcl:C-1608
- C40: value 10n -> 1u; device my_rcl:C-5W2 -> my_rcl:C-2012
- C42: value 10u -> DNP; device my_rcl:C-2012 -> my_rcl:C-1608
- C43: device my_rcl:C-2012 -> my_rcl:C-3225
- C44: value 47u -> 10u; device my_rcl:CPOLE2.5-5 -> my_rcl:C-3225
- C46: value 10n -> 10u; device my_rcl:C-3216 -> my_rcl:C-3225
- C47: value 100p -> 10u; device my_rcl:C-1608 -> my_rcl:C-3225
- C48: value 1n -> 4.7u; device my_rcl:C-2012 -> my_rcl:C-3216
- C49: value 1u -> 16V 680u; device my_rcl:C-1608 -> my_rcl:CPOLE5-10
- C5: device my_rcl:C-3225 -> my_rcl:C-2012
- C50: value 0.1u -> 16V 680u; device my_rcl:C-1608 -> my_rcl:CPOLE5-10
- C51: value 100u -> 100p; device my_rcl:CPOLE2.5-6.5 -> my_rcl:C-1608
- C52: value 470u -> 0.22u; device my_rcl:CPOLE5-10 -> my_rcl:C-5W
- C53: value 470u -> 100p; device my_rcl:CPOLE5-10 -> my_rcl:C-1608
- C54: value 0.1u -> 16V 2200u; device my_rcl:C-1608 -> my_rcl:CPOLE5-13
- C55: value 10n -> 1n; device my_rcl:C-3216 -> my_rcl:C-2012
- C56: value 2200u -> 1n; device my_rcl:CPOLE5-13 -> my_rcl:C-2012
- C57, C58: value 0.1u -> 10n; device my_rcl:C-1608 -> my_rcl:C-5W2
- C59: value 0.47u -> 47u; device my_rcl:C-5W -> my_rcl:CPOLE2.5-5
- C60: value 1000u -> 10u; device my_rcl:CPOLE5-10 -> my_rcl:C-2012
- C61: value 1000u -> 4.7u; device my_rcl:CPOLE5-10 -> my_rcl:C-2012
- C62: value 0.1u -> 100u; device my_rcl:C-1608 -> my_rcl:CPOLE2.5-6.5
- C63: device my_rcl:C-1005 -> my_rcl:C-1608
- C64: value 22u -> 100p; device my_rcl:C-2012 -> my_rcl:C-1608
- C65: value 2.2u -> 0.22u; device my_rcl:C-2012 -> my_rcl:C-5W
- C66: value 0.1u -> 100p
- C67, C68: value 0.1u -> 1n; device my_rcl:C-1005 -> my_rcl:C-2012
- C7: value 1u -> 0.1u
- C70, C71: value 10u -> 10n; device my_rcl:CPOL2012 -> my_rcl:C-5W2
- C72, C73: value 0.1u -> 10u; device my_rcl:C-1005 -> my_rcl:C-2012
- C74: value 10u -> 0.1u; device my_rcl:CPOL2012 -> my_rcl:C-1608
- C75: value 10u -> 0.1u; device my_rcl:C-3216 -> my_rcl:C-1608
- C76: value 1n -> 25V 1000u; device my_rcl:C-1608 -> my_rcl:CPOLE5-10
- C77: value 0.1u -> 1n; device my_rcl:C-1005 -> my_rcl:C-1608
- C78: value 0.1u -> 25V 1000u; device my_rcl:C-1005 -> my_rcl:CPOLE5-10
- C79: value 0.1u -> 1u; device my_rcl:C-1005 -> my_rcl:C-1608
- C83: value 0.1u -> 22u; device my_rcl:C-1608 -> my_rcl:C-2012
- D2: value LED0 -> 1mA; device my_rcl:LED-2.5 -> my_rcl:CRD-SMD
- IC1: value 3.3V -> ISO7762; device my_ic:TLV740 -> my_ic:ISO6762-SSOP
- IC10: value AK1110 -> 74LVC1G79; device my_ic:AK1110 -> my_ic:74LVC1G79
- IC11: value ISO7762 -> 1.8V; device my_ic:ISO6762-SSOP -> my_ic:TLV740
- IC12: value 74LVC1G79 -> AK1110; device my_ic:74LVC1G79 -> my_ic:AK1110
- IC13: value TC7WU04FU -> STM32G030F; device my_ic:TC7WU04FU -> my_ic:STM32G030F
- IC14: value TAR5SB33 -> CH221; device my_ic:TAR5SB33 -> my_ic:CH221
- IC15: value 74LVC1G79 -> 7808; device my_ic:74LVC1G79 -> my_ic:78X-SOP
- IC16: value 74LVC1G79 -> TAR5SB33; device my_ic:74LVC1G79 -> my_ic:TAR5SB33
- IC2: value PIC32MZEF -> 3.3V; device my_ic:PIC32MZEF -> my_ic:TLV740
- IC3: value SSM3582 -> PIC32MZEF; device my_ic:SSM3582 -> my_ic:PIC32MZEF
- IC4: value 1.8V -> TAR5SB33; device my_ic:TLV740 -> my_ic:TAR5SB33
- IC5: value TAR5SB33 -> SSM3582; device my_ic:TAR5SB33 -> my_ic:SSM3582
- IC6: value TL431 -> TC7WU04FU; device my_ic:TL431-SC59 -> my_ic:TC7WU04FU
- IC7: value STM32G030F -> TL431; device my_ic:STM32G030F -> my_ic:TL431-SC59
- IC8: value 7808 -> 74LVC1G79; device my_ic:78X-SOP -> my_ic:74LVC1G79
- IC9: value CH221 -> 74LVC1G79; device my_ic:CH221 -> my_ic:74LVC1G79
- Q1: value NPN -> PNP; device my_ic:NPN2SC3325 -> my_ic:PNP2SA1313
- Q2: value NPN -> PNP; device my_ic:NPN-SOT223 -> my_ic:PNP2SA1313
- Q4: value PNP -> NPN; device my_ic:PNP2SA1313 -> my_ic:NPN2SC3325
- Q5: value PNP -> NPN; device my_ic:PNP2SA1313 -> my_ic:NPN-SOT223
- R1: value 5.1 -> 3.3k
- R10: value 3.3k -> 51; device my_rcl:R-1608 -> my_rcl:R-1005
- R11: value 50k -> 51; device my_rcl:R-VAL2 -> my_rcl:R-1005
- R12: value MCLK -> 39.2k; device my_rcl:R-1005 -> my_rcl:R-1608
- R13: value LRCLK -> 10k; device my_rcl:R-1005 -> my_rcl:R-1608
- R14: value DATA -> 1k; device my_rcl:R-1005 -> my_rcl:R-3216
- R15, R23: value 10k -> 51; device my_rcl:R-1608 -> my_rcl:R-2012
- R17: value 51 -> MCLK; device my_rcl:R-2012 -> my_rcl:R-1005
- R18: value 1k -> MCLKB; device my_rcl:R-1608 -> my_rcl:R-1005
- R19: value 51 -> SCK; device my_rcl:R-2012 -> my_rcl:R-1005
- R20: value 51 -> LRCLK; device my_rcl:R-2012 -> my_rcl:R-1005
- R21: value 3.6k -> DATA; device my_rcl:R-1608 -> my_rcl:R-1005
- R22: value 1k -> 5.1; device my_rcl:R-1608 -> my_rcl:R-2012H
- R24: value 100k -> 51; device my_rcl:R-1608 -> my_rcl:R-2012
- R27: value 1k -> 50k; device my_rcl:R-1608 -> my_rcl:R-VAL2
- R29: value 1k -> 100k; device my_rcl:R-2012 -> my_rcl:R-1608
- R3: value 100 -> 5.1k
- R30: value 100k -> 10k
- R31: value 5.1k -> 10k
- R33: value 1k -> 5.1k; device my_rcl:R-3216 -> my_rcl:R-1608
- R34: value MCLKB -> 100k; device my_rcl:R-1005 -> my_rcl:R-1608
- R35: value 5.1 -> 10k; device my_rcl:R-2012H -> my_rcl:R-1608
- R4: value 5.1k -> 5.1
- R7: value 51 -> 100; device my_rcl:R-1005 -> my_rcl:R-1608
- R8: value SCK -> 1k; device my_rcl:R-1005 -> my_rcl:R-1608
- R9: value 51 -> 1k; device my_rcl:R-1005 -> my_rcl:R-1608
- X1: value 22.5792MHz -> 12MHz; device my_rcl:OSC-KC3225 -> my_rcl:CRYSTAL2
- X2: value 24.576MHz -> 22.5792MHz
- X3: value 12MHz -> 24.576MHz; device my_rcl:CRYSTAL2 -> my_rcl:OSC-KC3225
- renumbered CON6 to CON4, D5 to D3, FB12 to FB4, FB13 to FB6, FB9 to FB5, R43 to R36
Connections:
- removed net I2S_EN_441K: IC11.OUT1, IC13G$1.IN, IC7.PA12, X1.EN
- removed net I2S_EN_48K: IC13G$1.OUT, X2.EN
- removed net N$40: IC11.IN5, R6G$4.1
- new net EN_441K: IC1.OUT1, IC13.PA12, IC6G$1.IN, X2.EN
- new net EN_48K: IC6G$1.OUT, X3.EN
- net +12V: now also C29.1, C30.1, C33.1, C34.1, C36.1, C37.1, C40.1, C43.1, C44.1, C46.1, C47.1, C48.1, C49.1, C50.1, C54.1, IC5.PVDD@1, IC5.PVDD@2, IC5.PVDD@3, IC5.PVDD@4, IC5.PVDD@5, IC5.PVDD@6, IC5.PVDD@7, IC5.PVDD@8, Q5.E, R12.2, R14.2, R8.2; no longer C20.1, C21.1, C24.1, C27.1, C3.1, C5.1, C52.1, C53.1, C56.1, C63.1, C77.1, C78.1, C79.1, IC3.PVDD@1, IC3.PVDD@2, IC3.PVDD@3, IC3.PVDD@4, IC3.PVDD@5, IC3.PVDD@6, IC3.PVDD@7, IC3.PVDD@8, Q2.E, R18.2, R21.2, R33.2
- net +3V3: now also C4.1, C74.1, IC1.VCC2, IC13.VDD, IC16.VOUT, R27G$1.3, R27G$2.3, R30.2, R31.2; no longer C57.1, C64.1, IC11.VCC2, IC5.VOUT, IC7.VDD, R11G$1.3, R11G$2.3, R25.2, R26.2
- net +3V3A: now also C23.1, C35.1, C38.1, C41.1, C45.1, FB3.2, IC10.VDD, IC6G$4.V+, IC8.VDD, IC9.VDD; no longer C67.1, C68.1, C69.1, C72.1, C73.1, FB2.2, IC12.VDD, IC13G$4.V+, IC15.VDD, IC16.VDD
- net +3V3D: now also C3.1, C5.1, IC1.VCC1, IC2.OUT, IC3.AVDD, IC3.VDD@1, IC3.VDD@2, IC3.VDD@4, IC3.VDD@5, IC3.VDD@6, IC3.VUSB3V3; no longer C4.1, C82.1, IC1.OUT, IC11.VCC1, IC2.AVDD, IC2.VDD@1, IC2.VDD@2, IC2.VDD@4, IC2.VDD@5, IC2.VDD@6, IC2.VUSB3V3
- net +8V: now also C81.1, FB2.1, IC15.OUT, IC16.CONTROL, IC16.VIN; no longer C75.1, FB3.1, IC5.CONTROL, IC5.VIN, IC8.OUT
- net AMP_+5V: now also C61.1, C84.1, IC11.EN, IC11.IN, IC12.VOUT1; no longer C30.1, IC10.VOUT1, IC4.EN, IC4.IN
- net AMP_AVDD: now also C28.1, C59.1, C60.1, IC12.VOUT2, IC5.AVDD; no longer C23.1, C42.1, C44.1, IC10.VOUT2, IC3.AVDD
- net AMP_DVDD: now also C27.1, C69.1, IC11.OUT, IC5.DVDD; no longer C22.1, C43.1, IC3.DVDD, IC4.OUT
- net AMP_OUTN_L: now also C21.1, IC5.OUTL-@1, IC5.OUTL-@2; no longer C18.1, IC3.OUTL-@1, IC3.OUTL-@2
- net AMP_OUTN_R: now also C22.2, IC5.OUTR-@1, IC5.OUTR-@2; no longer C19.2, IC3.OUTR-@1, IC3.OUTR-@2
- net AMP_OUTP_L: now also C17.1, IC5.OUTL+@1, IC5.OUTL+@2; no longer C16.1, IC3.OUTL+@1, IC3.OUTL+@2
- net AMP_OUTP_R: now also C18.2, IC5.OUTR+@1, IC5.OUTR+@2; no longer C17.2, IC3.OUTR+@1, IC3.OUTR+@2
- net DGND: now also C3.2, C5.2, IC1.GND1, IC2.GND, IC3.AVSS, IC3.VSS@1, IC3.VSS@2, IC3.VSS@3, IC3.VSS@4, IC3.VSS@5, IC3.VSS@6, Q1.C, R3.1, X1.GND; no longer C4.2, C82.2, IC1.GND, IC11.GND1, IC2.AVSS, IC2.VSS@1, IC2.VSS@2, IC2.VSS@3, IC2.VSS@4, IC2.VSS@5, IC2.VSS@6, Q5.C, R4.1, X3.GND
- net GND: now also C16.2, C19.2, C28.2, C29.2, C33.2, C38.2, C39.2, C4.2, C40.2, C47.2, C51.1, C57.1, C59.2, C64.1, C67.1, C70.1, C80.2, C81.2, C82.2, C84.2, D2.K, IC1.GND2, IC10.VSS, IC11.GND, IC12.GND1, IC12.GND2, IC12.GND_REG, IC12.HT, IC13.VSS, IC15.GND, IC16.GND, IC5.ADDR0, IC5.ADDR1, IC5.AGND, IC5.AVDD_EN, IC5.DVDD_EN, IC5.HT, IC5.PGND@1, IC5.PGND@2, IC5.PGND@3, IC5.PGND@4, IC5.PGND@5, IC5.PGND@6, IC5.PGND@7, IC5.PGND@8, IC6G$4.V-, IC7.GND, IC8.VSS, IC9.VSS, R13.1, R14.1, R25.1, R26.1, R27G$1.1, R27G$2.1, R29.1, R33.2, R6G$1.1, R6G$1.2, X3.GND; no longer C21.2, C22.2, C29.1, C3.2, C33.1, C40.1, C42.2, C47.1, C48.1, C5.2, C51.2, C52.2, C57.2, C64.2, C65.2, C67.2, C70.2, D6.K, IC10.GND1, IC10.GND2, IC10.GND_REG, IC10.HT, IC11.GND2, IC12.VSS, IC13G$4.V-, IC15.VSS, IC16.VSS, IC3.ADDR0, IC3.ADDR1, IC3.AGND, IC3.AVDD_EN, IC3.DVDD_EN, IC3.HT, IC3.PGND@1, IC3.PGND@2, IC3.PGND@3, IC3.PGND@4, IC3.PGND@5, IC3.PGND@6, IC3.PGND@7, IC3.PGND@8, IC5.GND, IC6.GND, IC7.VSS, IC8.GND, IC9.GND, R11G$1.1, R11G$2.1, R15.1, R22.1, R23.1, R24.1, R31.2, R33.1, X1.GND
- net I2C_SCL: now also IC13.PB7/8, IC5.SCL, R30.1; no longer IC3.SCL, IC7.PB7/8, R25.1
- net I2C_SDA: now also IC13.PB9, IC5.SDA, R31.1; no longer IC3.SDA, IC7.PB9, R26.1
- net I2S_DATA: now also IC9.D, R6G$3.2; no longer IC15.D, R6G$2.2
- net I2S_DATA_BUF: now also IC5.SDATA, R20.2; no longer IC3.SDATA, R13.2
- net I2S_LRCLK: now also IC10.D, IC13.PA0, R6G$4.2; no longer IC16.D, IC7.PA0, R6G$3.2
- net I2S_LRCLK_BUF: now also IC5.FSYNC, R21.2; no longer IC3.FSYNC, R14.2
- net I2S_MCLK: now also IC10.CP, IC8.CP, IC9.CP, R10.2; no longer IC12.CP, IC15.CP, IC16.CP, R9.2
- net I2S_MCLK2: now also IC6G$3.IN, R11.2; no longer IC13G$3.IN, R7.2
- net I2S_MCLK_BUF: now also IC1.IN5, R17.2, R18.2; no longer R12.2, R34.2, R6G$4.2
- net I2S_SCK: now also IC8.D, R6G$2.2; no longer IC12.D, R6G$1.2
- net I2S_SCK_BUF: now also IC5.BCLK, R19.2; no longer IC3.BCLK, R8.2
- net LED0: now also D4.A, IC13.PA1; no longer D2.A, IC7.PA1
- net LED1: now also IC3.RF5, R1.2; no longer IC2.RF5, R10.2
- net MCLK_OSC: now also R10.1, R11.1, X3.OUT; no longer R7.1, R9.1, X1.OUT
- net MCLR: now also IC3.!MCLR, Q1.E; no longer IC2.!MCLR, Q5.E
- net N$10: now also IC8.Q, R19.1; no longer IC12.Q, R8.1
- net N$11: now also IC9.Q, R20.1; no longer IC15.Q, R13.1
- net N$12: now also C21.2, IC5.BSTL-; no longer C18.2, IC3.BSTL-
- net N$13: now also C17.2, IC5.BSTL+; no longer C16.2, IC3.BSTL+
- net N$14: now also IC10.Q, R21.1; no longer IC16.Q, R14.1
- net N$15: now also C58.1, R16.1; no longer C35.1, R17.1
- net N$16: now also Q4.E, Q5.B, R8.1; no longer Q1.E, Q2.B, R18.1
- net N$17: now also C18.1, IC5.BSTR+; no longer C17.1, IC3.BSTR+
- net N$18: now also C22.1, IC5.BSTR-; no longer C19.1, IC3.BSTR-
- net N$19: now also C71.1, R24.1; no longer C46.1, R19.1
- net N$2: now also R3.2; no longer R4.2
- net N$20: now also C42.2, IC7.REF, R9.1; no longer C38.2, IC6.REF, R27.1
- net N$21: now also C70.2, R23.2; no longer C55.2, R20.2
- net N$22: now also IC1.OUT3, R6G$3.1; no longer IC11.OUT3, R6G$2.1
- net N$23: now also C19.1, IC4.BYPASS; no longer C71.1, IC14.BYPASS
- net N$24: now also IC1.OUT4, R6G$4.1; no longer IC11.OUT4, R6G$3.1
- net N$25: now also C42.1, IC7.OUT, Q4.B; no longer C38.1, IC6.OUT, Q1.B
- net N$26: now also C73.1, IC12.NP1; no longer C37.1, IC10.NP1
- net N$27: now also C72.1, IC12.NP2; no longer C36.1, IC10.NP2
- net N$28: now also Q2.B, R7.1; no longer Q4.B, R3.1
- net N$29: now also C62.1, C63.1, IC12.EN, IC12.VIN1, IC12.VIN2, R22.2; no longer C31.1, C51.1, IC10.EN, IC10.VIN1, IC10.VIN2, R35.2
- net N$3: now also R4.1; no longer R1.1
- net N$30: now also C48.2, R12.1, R13.2, R9.2; no longer C39.2, R21.1, R22.2, R27.2
- net N$31: now also IC14.CC1, R32.1; no longer IC9.CC1, R31.1
- net N$32: now also IC14.CC2, R33.1; no longer IC9.CC2, R32.1
- net N$33: now also C79.1, IC14.VDD, R34.2, R37.1; no longer C49.1, IC9.VDD, R29.1, R30.2
- net N$34: now also IC14.CFG, R34.1; no longer IC9.CFG, R30.1
- net N$35: now also C82.1, IC16.BYPASS; no longer C54.1, IC5.BYPASS
- net N$36: now also R25.2; no longer R23.2
- net N$37: now also IC6G$2.IN, IC6G$3.OUT, R18.1; no longer IC13G$2.IN, IC13G$3.OUT, R34.1
- net N$38: now also D2.A, Q2.C; no longer D6.A, Q4.C
- net N$39: now also IC6G$2.OUT, R17.1; no longer IC13G$2.OUT, R12.1
- net N$4: now also IC2.EN, IC2.IN, R4.2; no longer IC1.EN, IC1.IN, R1.2
- net N$41: now also D4.K, R26.2; no longer D2.K, R15.2
- net N$42: now also R22.1; no longer R35.1
- net N$43: now also C16.1, FB2.2, IC4.CONTROL, IC4.VIN; no longer C74.1, FB3.2, IC14.CONTROL, IC14.VIN
- net N$5: now also IC3.OSC1, X1.2; no longer IC2.OSC1, X3.2
- net N$6: now also C57.2, R15.2; no longer C40.2, R16.2
- net N$7: now also IC3.OSC2, X1.1; no longer IC2.OSC2, X3.1
- net N$8: now also IC1.OUT2, R6G$2.1; no longer IC11.OUT2, R6G$1.1
- net N$9: now also R1.1; no longer R10.1
- net PGEC: now also IC3.PGEC1; no longer IC2.PGEC1
- net PGED: now also IC3.PGED1; no longer IC2.PGED1
- net PIC_DATA: now also IC1.IN3, IC3.RD2; no longer IC11.IN3, IC2.RD2
- net PIC_DDC_EN: now also IC1.OUT6, Q1.B; no longer IC11.OUT6, Q5.B
- net PIC_EN441K: now also IC1.IN1, IC3.RD10; no longer IC11.IN1, IC2.RD10
- net PIC_LRCLK: now also IC1.IN4, IC3.RD4; no longer IC11.IN4, IC2.RD4
- net PIC_MCLK: now also IC1.OUT5, IC3.RF1; no longer IC11.OUT5, IC2.RF1
- net PIC_SCK: now also IC1.IN2, IC3.RD1, IC3.T1CK; no longer IC11.IN2, IC2.RD1, IC2.T1CK
- net SPK_OUTN_L: now also C52.2, C53.1, C56.1, R16.2; no longer C28.2, C32.1, C34.1, R17.2
- net SPK_OUTN_R: now also C65.2, C66.1, C68.1, R24.2; no longer C41.1, C45.1, C59.2, R19.2
- net SPK_OUTP_L: now also C51.2, C52.1, C55.2, R15.1; no longer C28.1, C29.2, C33.2, R16.1
- net SPK_OUTP_R: now also C64.2, C65.1, C67.2, R23.1; no longer C47.2, C48.2, C59.1, R20.1
- net STM_DDC_EN: now also IC1.IN6, IC13.PA11; no longer IC11.IN6, IC7.PA11
- net STM_TX: now also IC13.PA2; no longer IC7.PA2
- net SWCLK: now also IC13.SWCLK; no longer IC7.SWCLK
- net SWDIO: now also IC13.SWDIO; no longer IC7.SWDIO
- net UART_TX: now also IC3.RE5; no longer IC2.RE5
- net USB_D+: now also IC3.D+; no longer IC2.D+
- net USB_D-: now also IC3.D-; no longer IC2.D-
- net USB_VBUS: now also IC3.VBUS; no longer IC2.VBUS
- net V+: now also C75.1, C76.1, C78.1, C80.1, IC15.IN, Q2.E, Q4.C, Q5.C, R35.2, R7.2; no longer C50.1, C58.1, C60.1, C61.1, IC8.IN, Q1.C, Q2.C, Q4.E, R3.2, R42.2
- net V+_ADC: now also IC13.PA5, R35.1; no longer IC7.PA5, R42.1
- net VINC_+: now also R37.2; no longer R29.2
- net VOL_ADC: now also C77.1, IC13.PA4, R27G$1.2, R27G$2.2, R29.2; no longer C76.1, IC7.PA4, R11G$1.2, R11G$2.2, R24.2
- net XVCC: now also C20.1, C24.1, C31.1, C32.1, FB3.1, IC4.VOUT, X3.VCC; no longer C62.1, C65.1, C66.1, C70.1, FB2.1, IC14.VOUT, X1.VCC
Other:
- note added: "Clock"
- moved on the sheet: C10, C11, C12, C13, C17, C18, C21, C22, C23, C24, C25, C26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

Commit message: v4.2 発注
Parts:
- added C85, C86, C87, C88: 100p, my_rcl:C-1608
- added R38, R39, R40, R41: 10, my_rcl:R-1608
- added TP11, TP12, TP13, TP14, TP15, TP16, TP17, TP18, TP6: G, my_connector:TESTPIN
- C4: device my_rcl:C-1608 -> my_rcl:C-1005
- DR2: value HOLE-3.2 -> HOLE-3.2C; device my_connector:HOLE-3.2 -> my_connector:HOLE-3.2C
- IC6: value TC7WU04FU -> 3G04
- R22: value 5.1 -> 2.2
- R25, R26: value 10k -> 3.3k
- TP5: value G -> DG
Connections:
- new net N$40: C86.1, R39.1
- new net N$44: C87.1, R40.1
- new net N$45: C85.1, R38.1
- new net N$46: C88.1, R41.1
- net AMP_OUTN_L: now also R38.2
- net AMP_OUTN_R: now also R40.2
- net AMP_OUTP_L: now also R39.2
- net AMP_OUTP_R: now also R41.2
- net GND: now also C85.2, C86.2, C87.2, C88.2, DR2.HT, TP11.1, TP12.1, TP13.1, TP14.1, TP15.1, TP16.1, TP17.1, TP18.1, TP6.1

Commit message: 微修正
Parts:
- added TP19, TP20: L_P, my_connector:TESTPIN-MID
- added TP21, TP22: R_N, my_connector:TESTPIN-MID
- L1, L2: value 7uH -> 7uH-UA8013
- R20: value LRCLK -> DATA
- R21: value DATA -> LRCLK
Connections:
- net SPK_OUTN_L: now also TP19.1
- net SPK_OUTN_R: now also TP22.1
- net SPK_OUTP_L: now also TP20.1
- net SPK_OUTP_R: now also TP21.1
Changed lines of the file:
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@@
 <part name="SUPPLY98" library="my_supply" deviceset="GND" device=""/>
 <part name="P+3" library="my_supply" deviceset="+12V" device=""/>
-<part name="L2" library="my_rcl" deviceset="L-DUAL" device="" value="7uH"/>
+<part name="L2" library="my_rcl" deviceset="L-DUAL" device="" value="7uH-UA8013"/>
 <part name="C52" library="my_rcl" deviceset="C" device="-5W" value="0.22u"/>
-<part name="L1" library="my_rcl" deviceset="L-DUAL" device="" value="7uH"/>
+<part name="L1" library="my_rcl" deviceset="L-DUAL" device="" value="7uH-UA8013"/>
 <part name="C55" library="my_rcl" deviceset="C" device="-2012" value="1n"/>
 <part name="C56" library="my_rcl" deviceset="C" device="-2012" value="1n"/>
@@
 <part name="SUPPLY134" library="my_supply" deviceset="GND" device=""/>
 <part name="R19" library="my_rcl" deviceset="R" device="-1005" value="SCK"/>
-<part name="R20" library="my_rcl" deviceset="R" device="-1005" value="LRCLK"/>
-<part name="R21" library="my_rcl" deviceset="R" device="-1005" value="DATA"/>
+<part name="R20" library="my_rcl" deviceset="R" device="-1005" value="DATA"/>
+<part name="R21" library="my_rcl" deviceset="R" device="-1005" value="LRCLK"/>
 <part name="IC8" library="my_ic" deviceset="74LVC1G79" device=""/>
 <part name="IC9" library="my_ic" deviceset="74LVC1G79" device=""/>
@@
 <part name="SUPPLY170" library="my_supply" deviceset="GND" device=""/>
 <part name="SUPPLY171" library="my_supply" deviceset="GND" device=""/>
+<part name="TP19" library="my_connector" deviceset="TESTPIN" device="-MID" value="L_P"/>
+<part name="TP20" library="my_connector" deviceset="TESTPIN" device="-MID" value="L_P"/>
+<part name="TP21" library="my_connector" deviceset="TESTPIN" device="-MID" value="R_N"/>
+<part name="TP22" library="my_connector" deviceset="TESTPIN" device="-MID" value="R_N"/>
 </parts>
 <sheets>
@@
 </instance>
 <instance part="L2" gate="G$1" x="401.32" y="132.08" smashed="yes" rot="R90">
-<attribute name="NAME" x="406.4" y="130.81" size="1.778" layer="95" rot="R180"/>
-<attribute name="VALUE" x="406.4" y="135.89" size="1.778" layer="96" rot="R180"/>
+<attribute name="NAME" x="396.24" y="134.62" size="1.778" layer="95"/>
+<attribute name="VALUE" x="393.7" y="129.54" size="1.778" layer="96"/>
 </instance>
 <instance part="C52" gate="G$1" x="340.36" y="125.73" smashed="yes">
@@
 </instance>
 <instance part="L1" gate="G$1" x="332.74" y="119.38" smashed="yes" rot="R90">
-<attribute name="NAME" x="337.82" y="118.11" size="1.778" layer="95" rot="R180"/>
-<attribute name="VALUE" x="337.82" y="123.19" size="1.778" layer="96" rot="R180"/>
+<attribute name="NAME" x="327.66" y="116.84" size="1.778" layer="95"/>
+<attribute name="VALUE" x="325.12" y="121.92" size="1.778" layer="96"/>
 </instance>
 <instance part="L1" gate="G$2" x="332.74" y="132.08" smashed="yes" rot="R270">
 <attribute name="NAME" x="327.66" y="133.35" size="1.778" layer="95"/>
-<attribute name="VALUE" x="327.66" y="128.27" size="1.778" layer="96"/>
+<attribute name="VALUE" x="325.12" y="128.27" size="1.778" layer="96"/>
 </instance>
 <instance part="C55" gate="G$1" x="347.98" y="137.16" smashed="yes">
@@
 </instance>
 <instance part="L2" gate="G$2" x="401.32" y="119.38" smashed="yes" rot="R270">
-<attribute name="NAME" x="396.24" y="120.65" size="1.778" layer="95"/>
-<attribute name="VALUE" x="396.24" y="115.57" size="1.778" layer="96"/>
+<attribute name="NAME" x="396.24" y="115.57" size="1.778" layer="95"/>
+<attribute name="VALUE" x="393.7" y="120.65" size="1.778" layer="96"/>
 </instance>
 <instance part="C66" gate="G$1" x="408.94" y="114.3" smashed="yes">
@@
 <instance part="SUPPLY170" gate="GND" x="223.52" y="43.18" smashed="yes" rot="R90"/>
 <instance part="SUPPLY171" gate="GND" x="223.52" y="38.1" smashed="yes" rot="R90"/>
+<instance part="TP19" gate="G$1" x="363.22" y="123.19" smashed="yes" rot="R270">
+<attribute name="VALUE" x="367.665" y="122.555" size="1.778" layer="95"/>
+</instance>
+<instance part="TP20" gate="G$1" x="363.22" y="128.27" smashed="yes" rot="R270">
+<attribute name="VALUE" x="367.665" y="127.635" size="1.778" layer="95"/>
+</instance>
+<instance part="TP21" gate="G$1" x="431.8" y="128.27" smashed="yes" rot="R270">
+<attribute name="VALUE" x="436.245" y="127.635" size="1.778" layer="95"/>
+</instance>
+<instance part="TP22" gate="G$1" x="431.8" y="123.19" smashed="yes" rot="R270">
+<attribute name="VALUE" x="436.245" y="122.555" size="1.778" layer="95"/>
+</instance>
 </instances>
 <busses>
@@
 <wire x1="358.14" y1="134.62" x2="358.14" y2="132.08" width="0.1524" layer="91"/>
 <junction x="358.14" y="132.08"/>
+<pinref part="TP20" gate="G$1" pin="1"/>
+<wire x1="360.68" y1="128.27" x2="358.14" y2="128.27" width="0.1524" layer="91"/>
+<wire x1="358.14" y1="128.27" x2="358.14" y2="132.08" width="0.1524" layer="91"/>
 </segment>
 </net>
@@
 <wire x1="358.14" y1="116.84" x2="358.14" y2="119.38" width="0.1524" layer="91"/>
 <junction x="358.14" y="119.38"/>
+<pinref part="TP19" gate="G$1" pin="1"/>
+<wire x1="358.14" y1="119.38" x2="358.14" y2="123.19" width="0.1524" layer="91"/>
+<wire x1="358.14" y1="123.19" x2="360.68" y2="123.19" width="0.1524" layer="91"/>
 </segment>
 </net>
@@
 <pinref part="C65" gate="G$1" pin="1"/>
 <wire x1="408.94" y1="128.27" x2="408.94" y2="132.08" width="0.1524" layer="91"/>
+<pinref part="TP21" gate="G$1" pin="1"/>
+<wire x1="429.26" y1="128.27" x2="426.72" y2="128.27" width="0.1524" layer="91"/>
+<wire x1="426.72" y1="128.27" x2="426.72" y2="132.08" width="0.1524" layer="91"/>
 </segment>
 </net>
@@
 <pinref part="C65" gate="G$1" pin="2"/>
 <wire x1="408.94" y1="123.19" x2="408.94" y2="119.38" width="0.1524" layer="91"/>
-</segment>
-</net>
+<pinref part="TP22" gate="G$1" pin="1"/>
+<wire x1="426.72" y1="119.38" x2="426.72" y2="123.19" width="0.1524" layer="91"/>
+<wire x1="426.72" y1="123.19" x2="429.26" y2="123.19" width="0.1524" layer="91"/>
+</segment>
+</net>

Commit message: v4.3
Parts:
- added D5, D6, D7, D8: SBD, my_rcl:DIODE-323
- added R42, R43: THJ, my_rcl:R-3216-2
Connections:
- net AMP_OUTN_L: now also D5.K
- net AMP_OUTN_R: now also D8.K
- net AMP_OUTP_L: now also D6.K
- net AMP_OUTP_R: now also D7.K
- net DGND: now also R42.1, R43.1
- net GND: now also D5.A, D6.A, D7.A, D8.A, R42.2, R43.2
Other:
- moved on the sheet: C42, C48, C49, C50, C54, D2, IC7, Q2, Q3, Q4, Q5, R12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
